Commit message: update urdf

File: eklavya_description/urdf/eklavya.urdf (robot description, URDF)
Before this commit: robot eklavya, 24 links, 24 joints
Links:
- added link front_wheel_link, mass 0.01; collision sphere radius=0.018; visual sphere radius=0.018
- added link gyro_link, mass 0.001
- added link left_cliff_sensor_link, mass 0.01
- added link leftfront_cliff_sensor_link, mass 0.01
- added link plate_0_link, mass 0.01; collision box size=0.233502 0.314845 0.006401; visual mesh filename=package://eklavya_description/meshes/plate_0_logo.dae
- added link plate_1_link, mass 0.1; collision box size=0.314856 0.314856 0.006401; visual mesh filename=package://eklavya_description/meshes/plate_1_logo.dae
- added link plate_2_link, mass 0.01; collision box size=0.314856 0.314856 0.006401; visual mesh filename=package://eklavya_description/meshes/plate_1_logo.dae
- added link rear_wheel_link, mass 0.001; collision sphere radius=0.015; visual sphere radius=0.015
- added link right_cliff_sensor_link, mass 0.01
- added link rightfront_cliff_sensor_link, mass 0.01
- added link wall_sensor_link, mass 0.01
- link base_footprint: mass None -> 0.0001
Joints:
- added joint base_footprint_joint: type fixed, parent base_footprint, child base_link, origin xyz=0 0 0.017 rpy=0 0 0
- added joint base_left_cliff_sensor_joint: type fixed, parent base_link, child left_cliff_sensor_link, origin xyz=0.07 0.14 0.01 rpy=0 1.57079 0
- added joint base_leftfront_cliff_sensor_joint: type fixed, parent base_link, child leftfront_cliff_sensor_link, origin xyz=0.15 0.04 0.01 rpy=0 1.57079 0
- added joint base_right_cliff_sensor_joint: type fixed, parent base_link, child right_cliff_sensor_link, origin xyz=0.07 -0.14 0.01 rpy=0 1.57079 0
- added joint base_rightfront_cliff_sensor_joint: type fixed, parent base_link, child rightfront_cliff_sensor_link, origin xyz=0.15 -0.04 0.01 rpy=0 1.57079 0
- added joint base_wall_sensor_joint: type fixed, parent base_link, child wall_sensor_link, origin xyz=0.09 -0.120 0.042 rpy=0 0 -1.0
- added joint gyro_joint: type fixed, parent base_link, child gyro_link, origin xyz=0 0 0.04 rpy=0 0 0, axis 0 1 0
- added joint plate_0_joint: type fixed, parent base_link, child plate_0_link, origin xyz=-0.04334 0  0.06775704 rpy=0 0 0
- added joint plate_1_joint: type fixed, parent plate_0_link, child plate_1_link, origin xyz=0.04068 0 0.05715 rpy=0 0 0
- added joint plate_2_joint: type fixed, parent plate_1_link, child plate_2_link, origin xyz=0 0 0.0572008 rpy=0 0 0

File: eklavya_description/urdf/eklavya_body.urdf.xacro (robot description, xacro)
@@ -12,5 +12,4 @@
   <!-- base_footprint is a fictitious link(frame) that is on the ground right below base_link origin, navigation stack depends on this frame -->
   <link name="base_footprint">
-<!--
     <inertial>
       <mass value="0.0001" />
@@ -20,5 +19,4 @@
               izz="0.0001" />
     </inertial>
--->
     <visual>
       <origin xyz="0 0 0" rpy="0 0 0" />
@@ -45,5 +43,5 @@
       <origin xyz=" 0 0 0.0308" rpy="0 0 0" />
       <geometry>
-        <mesh filename="package://eklvya_description/meshes/create_body.dae"/>
+        <mesh filename="package://eklavya_description/meshes/create_body.dae"/>
       </geometry>
     </visual>
@@ -55,5 +53,4 @@
     </collision>
   </link>
-<!--
   <link name="wall_sensor_link">
     <inertial>
@@ -126,5 +123,4 @@
     <child link="rightfront_cliff_sensor_link" />
   </joint>
--->
   <link name="left_wheel_link">
     <inertial>
@@ -179,5 +175,5 @@
     <axis xyz="0 1 0"/>
   </joint>
-<!--  <link name="rear_wheel_link">
+ <link name="rear_wheel_link">
     <inertial>
       <origin xyz="0 0 0"/>
@@ -199,5 +195,4 @@
     </collision>
   </link>
--->
   <!-- fixed because there's no transmission -->
   <joint name="rear_castor_joint" type="fixed">
@@ -207,5 +202,5 @@
     <axis xyz="0 1 0"/>
   </joint>
-<!--  <link name="front_wheel_link">
+ <link name="front_wheel_link">
     <inertial>
       <origin xyz="0 0 0" />
@@ -227,5 +222,4 @@
     </collision>
   </link>
--->
   <!-- fixed because there's no transmission -->
   <joint name="front_castor_joint" type="fixed">
@@ -239,5 +233,5 @@
   <eklavya_spacer parent="base_link" number="2" x_loc="-0.07239" y_loc="-0.1114679" z_loc="0.062992"/>
   <eklavya_spacer parent="base_link" number="3" x_loc="-0.07239" y_loc="0.1114679" z_loc="0.062992"/>
-<!--  <joint name="gyro_joint" type="fixed">
+ <joint name="gyro_joint" type="fixed">
     <axis xyz="0 1 0" />
     <origin xyz="0 0 0.04" rpy="0 0 0" />
@@ -251,5 +245,5 @@
       <inertia ixx="0.0001" ixy="0" ixz="0" iyy="0.000001" iyz="0" izz="0.0001" />
     </inertial>
-  </link>-->
+  </link>
   <joint name="laser_joint" type="fixed">
     <origin xyz="-0.065 0 0.075" rpy="0 0 0" />
@@ -272,5 +266,4 @@
     </inertial>
   </link>
-<!--
   <joint name="plate_0_joint" type="fixed">
     <origin xyz="-0.04334 0  0.06775704" rpy="0 0 0" />
@@ -299,10 +292,8 @@
     </collision>
   </link>
--->
   <eklavya_standoff_2in parent="base_link" number="0" x_loc="0.0676402" y_loc="0.1314196" z_loc="0.0709803"/>
   <eklavya_standoff_2in parent="base_link" number="1" x_loc="0.0676402" y_loc="-0.1314196" z_loc="0.0709803"/>
   <eklavya_standoff_2in parent="base_link" number="2" x_loc="-0.052832" y_loc="-0.1314196" z_loc="0.0709803"/>
   <eklavya_standoff_2in parent="base_link" number="3" x_loc="-0.052832" y_loc="0.1314196" z_loc="0.0709803"/>
-<!--
   <joint name="plate_1_joint" type="fixed">
     <origin xyz="0.04068 0 0.05715" rpy="0 0 0" />
@@ -331,10 +322,8 @@
     </collision>
   </link>
--->
   <eklavya_standoff_2in parent="standoff_2in_0_link" number="4" x_loc="0" y_loc="0" z_loc="0.05715"/>
   <eklavya_standoff_2in parent="standoff_2in_1_link" number="5" x_loc="0" y_loc="0" z_loc="0.05715"/>
   <eklavya_standoff_2in parent="standoff_2in_2_link" number="6" x_loc="0" y_loc="0" z_loc="0.05715"/>
   <eklavya_standoff_2in parent="standoff_2in_3_link" number="7" x_loc="0" y_loc="0" z_loc="0.05715"/>
-<!--
   <joint name="plate_2_joint" type="fixed">
     <origin xyz="0 0 0.0572008" rpy="0 0 0" />
@@ -363,5 +352,4 @@
     </collision>
   </link>
--->
   <eklavya_standoff_kinect parent="plate_2_link" number="0" x_loc="-0.1024382" y_loc="0.098" z_loc="0.0032004"/>
   <eklavya_standoff_kinect parent="plate_2_link" number="1" x_loc="-0.1024382" y_loc="-0.098" z_loc="0.0032004"/>

Commit message: updated_model.

File: eklavya_description/urdf/eklavya.urdf (robot description, URDF)
Before this commit: robot eklavya, 35 links, 34 joints
Links:
- removed link base_footprint
- removed link front_wheel_link
- removed link gyro_link
- removed link laser
- removed link left_cliff_sensor_link
- removed link left_wheel_link
- removed link leftfront_cliff_sensor_link
- removed link plate_0_link
- removed link plate_1_link
- removed link plate_2_link
- removed link plate_3_link
- removed link rear_wheel_link
- removed link right_cliff_sensor_link
- removed link right_wheel_link
- removed link rightfront_cliff_sensor_link
- removed link spacer_0_link
- removed link spacer_1_link
- removed link spacer_2_link
- removed link spacer_3_link
- removed link standoff_2in_0_link
- removed link standoff_2in_1_link
- removed link standoff_2in_2_link
- removed link standoff_2in_3_link
- removed link standoff_2in_4_link
- removed link standoff_2in_5_link
- removed link standoff_2in_6_link
- removed link standoff_2in_7_link
- removed link standoff_8in_0_link
- removed link standoff_8in_1_link
- removed link standoff_8in_2_link
- removed link standoff_8in_3_link
- removed link standoff_kinect_0_link
- removed link standoff_kinect_1_link
- removed link wall_sensor_link
- added link left_wheel, mass 0.0001; collision cylinder length=0.06 radius=.1; visual cylinder length=0.06 radius=.1
- added link right_wheel, mass 0.0001; collision cylinder length=0.06 radius=.1; visual cylinder length=0.06 radius=.1
- link base_link: mass 2 -> 0.0001; geometry collision box size=.55 .55 .55; visual box size=.55 .55 .55
Joints:
- removed joint base_footprint_joint
- removed joint base_left_cliff_sensor_joint
- removed joint base_leftfront_cliff_sensor_joint
- removed joint base_right_cliff_sensor_joint
- removed joint base_rightfront_cliff_sensor_joint
- removed joint base_wall_sensor_joint
- removed joint front_castor_joint
- removed joint gyro_joint
- removed joint laser_joint
- removed joint left_wheel_joint
- removed joint plate_0_joint
- removed joint plate_1_joint
- removed joint plate_2_joint
- removed joint plate_3_joint
- removed joint rear_castor_joint
- removed joint right_wheel_joint
- removed joint spacer_0_joint
- removed joint spacer_1_joint
- removed joint spacer_2_joint
- removed joint spacer_3_joint
- removed joint standoff_2in_0_joint
- removed joint standoff_2in_1_joint
- removed joint standoff_2in_2_joint
- removed joint standoff_2in_3_joint
- removed joint standoff_2in_4_joint
- removed joint standoff_2in_5_joint
- removed joint standoff_2in_6_joint
- removed joint standoff_2in_7_joint
- removed joint standoff_8in_0_joint
- removed joint standoff_8in_1_joint
- removed joint standoff_8in_2_joint
- removed joint standoff_8in_3_joint
- removed joint standoff_kinect_0_joint
- removed joint standoff_kinect_1_joint
- added joint left_wheel_hinge: type revolute, parent base_link, child left_wheel, axis 0 1 0, limit effort=30 velocity=1.0
- added joint right_wheel_hinge: type revolute, parent base_link, child right_wheel, axis 0 1 0, limit effort=30 velocity=1.0

File: eklavya_description/urdf/eklavya.urdf.xacro (robot description, xacro)
@@ -5,5 +5,5 @@
        xmlns:interface="http://playerstage.sourceforge.net/gazebo/xmlschema/#interface"
        xmlns:xacro="http://ros.org/wiki/xacro">
-  <include filename="$(find eklavya_description)/urdf/eklavya_hardware.urdf.xacro" />
+  <!--<include filename="$(find eklavya_description)/urdf/eklavya_hardware.urdf.xacro" />-->
   <include filename="$(find eklavya_description)/urdf/eklavya_body.urdf.xacro" />
  <!-- <include filename="$(find eklavya_description)/urdf/eklavya_calibration.xacro" />

File: eklavya_description/urdf/eklavya_body.urdf.xacro (robot description, xacro)
@@ -6,382 +6,194 @@
   <property name="base_x" value="0.33" />
   <property name="base_y" value="0.33" />
-  <xacro:macro name="eklavya_body">
-    <material name="Green">
-      <color rgba="0.0 0.8 0.0 1.0"/>
-    </material>
-  <!-- base_footprint is a fictitious link(frame) that is on the ground right below base_link origin, navigation stack depends on this frame -->
-  <link name="base_footprint">
+ <xacro:macro name="eklavya_body">
+    <!--  INSERT YOU MODEL HERE -->
+  <link name='base_link'>
+    <pose>0 0 .375 0 0 3.14</pose>
     <inertial>
       <mass value="0.0001" />
-      <origin xyz="0 0 0" />
       <inertia ixx="0.0001" ixy="0.0" ixz="0.0"
               iyy="0.0001" iyz="0.0"
               izz="0.0001" />
     </inertial>
-    <visual>
-      <origin xyz="0 0 0" rpy="0 0 0" />
-      <geometry>
-        <box size="0.001 0.001 0.001" />
-      </geometry>
-      <material name="Green" />
-    </visual>
-    <collision>
-      <origin xyz="0 0 0.017" rpy="0 0 0" />
-      <geometry>
-       <box size="0.001 0.001 0.001" />
-      </geometry>
-    </collision>
-  </link>
-  <link name="base_link">
+    <collision name='collision'>
+      <geometry>
+        <box size=".55 .55 .55"/>
+      </geometry>
+    </collision>
+    <visual name='visual'>
+      <geometry>
+        <box size=".55 .55 .55"/>
+      </geometry>
+      <material name="red">
+        <color rgba=".8 0 0 1"/>
+      </material>
+    </visual>
+  </link>
+  <!--Top of base_link support-->
+  <!--<link name="sc1">
+    <collision name='sc1'>
+      <pose>0.26 0.26 0.575 0 0 0</pose>
+      <geometry>
+        <box size=".03 .03 .6"/>
+      </geometry>
+    </collision>
+    <visual name='sv1'>
+      <pose>0.26 0.26 0.575 0 0 0</pose>
+      <geometry>
+        <box size=".03 .03 .6"/>
+      </geometry>
+    </visual>
+  </link>
+  <link name="sc2">
+    <collision name='sc2'>
+      <pose>-0.26 0.26 0.575 0 0 0</pose>
+      <geometry>
+        <box size=".03 .03 .6"/>
+      </geometry>
+    </collision>
+    <visual name='sv2'>
+      <pose>-0.26 0.26 0.575 0 0 0</pose>
+      <geometry>
+        <box size=".03 .03 .6"/>
+      </geometry>
+    </visual>
+  </link>
+  <link name="sc3">
+    <collision name='sc3'>
+      <pose>0 0.26 0.89 0 0 0</pose>
+      <geometry>
+        <box size=".55 .03 .03"/>
+      </geometry>
+    </collision>
+    <visual name='sv3'>
+      <pose>0 0.26 0.89 0 0 0</pose>
+      <geometry>
+        <box size=".55 .03 .03"/>
+      </geometry>
+    </visual>
+  </link>
+  <link name="castor_support">
+ --> <!--Castor Support-->
+<!--    <collision name='extrusion_collision'>
+      <pose>0 0.375 -0.275 0 0 0</pose>
+      <geometry>
+        <box size=".1 .2 .02"/>
+      </geometry>
+    </collision>
+    <visual name='extrusion_visual'>
+      <pose>0 0.375 -0.275 0 0 0</pose>
+      <geometry>
+        <box size=".1 .2 .02"/>
+      </geometry>
+    </visual>
+  </link>
+  <link name="castor">
+  --><!--Castor-->
+<!-- 	<collision name='caster_collision'>
+      <pose>0 0.375 -0.325 0 0 0</pose>
+      <geometry>
+        <sphere radius=".05"/>
+      </geometry>
+      <surface>
+        <friction>
+          <ode>
+            <mu>0</mu>
+            <mu2>0</mu2>
+            <slip1>1.0</slip1>
+            <slip2>1.0</slip2>
+          </ode>
+        </friction>
+      </surface>
+    </collision>
+    <visual name='caster_visual'>
+      <pose>0 0.375 -0.325 0 0 0</pose>
+      <geometry>
+        <sphere radius=".05"/>
+      </geometry>
+    </visual>
+  </link>
+  -->
+  <!--Left_Wheel-->
+  <link name="left_wheel">
+    <pose>0.278 0.275 0.1 1.5707 0 1.5707</pose>
     <inertial>
-      <mass value="2" />
-      <origin xyz="0 0 0.0" />
-      <inertia ixx="0.01" ixy="0.0" ixz="0.0"
-        iyy="0.01" iyz="0.0" izz="0.5" />
+      <mass value="0.0001" />
+      <inertia ixx="0.0001" ixy="0.0" ixz="0.0"
+              iyy="0.0001" iyz="0.0"
+              izz="0.0001" />
     </inertial>
-    <visual>
-      <origin xyz=" 0 0 0.0308" rpy="0 0 0" />
-      <geometry>
-        <mesh filename="package://eklavya_description/meshes/create_body.dae"/>
-      </geometry>
-    </visual>
-    <collision>
-      <origin xyz="0.0 0.0 0.0308" rpy="0 0 0" />
-      <geometry>
-        <cylinder length="0.0611632" radius="0.016495"/>
-      </geometry>
-    </collision>
-  </link>
-  <link name="wall_sensor_link">
+    <collision name='left_wheel_collision'>
+      <geometry>
+        <cylinder radius=".1" length="0.06"/>
+      </geometry>
+      <surface>
+        <friction>
+          <ode>
+            <mu>0</mu>
+            <mu2>0</mu2>
+            <slip1>1.0</slip1>
+            <slip2>1.0</slip2>
+          </ode>
+        </friction>
+      </surface>
+    </collision>
+    <visual name='left_wheel_visual'>
+      <geometry>
+        <cylinder radius=".1" length="0.06"/>
+      </geometry>
+      <material name="red">
+        <color rgba=".8 0 0 1"/>
+      </material>
+    </visual>
+  </link>
+  <!--Right_Wheel-->
+  <link name="right_wheel">
+    <pose>-0.278 0.275 0.1 1.5707 0 1.5707</pose>
     <inertial>
-      <mass value="0.01" />
-      <origin xyz="0 0 0"/>
-      <inertia ixx="0.001" ixy="0.0" ixz="0.0"
-        iyy="0.001" iyz="0.0" izz="0.001" />
+      <mass value="0.0001" />
+      <inertia ixx="0.0001" ixy="0.0" ixz="0.0"
+              iyy="0.0001" iyz="0.0"
+              izz="0.0001" />
     </inertial>
-  </link>
-  <link name="left_cliff_sensor_link">
-    <inertial>
-      <mass value="0.01" />
-      <origin xyz="0 0 0"/>
-      <inertia ixx="0.001" ixy="0.0" ixz="0.0"
-        iyy="0.001" iyz="0.0" izz="0.001" />
-    </inertial>
-  </link>
-  <link name="right_cliff_sensor_link">
-    <inertial>
-      <mass value="0.01" />
-      <origin xyz="0 0 0"/>
-      <inertia ixx="0.001" ixy="0.0" ixz="0.0"
-        iyy="0.001" iyz="0.0" izz="0.001" />
-    </inertial>
-  </link>
-  <link name="leftfront_cliff_sensor_link">
-    <inertial>
-      <mass value="0.01" />
-      <origin xyz="0 0 0"/>
-      <inertia ixx="1.0" ixy="0.0" ixz="0.0"
-        iyy="0.01" iyz="0.0" izz="0.01" />
-    </inertial>
-  </link>
-  <link name="rightfront_cliff_sensor_link">
-    <inertial>
-      <mass value="0.01" />
-      <origin xyz="0 0 0"/>
-      <inertia ixx="0.001" ixy="0.0" ixz="0.0"
-        iyy="0.001" iyz="0.0" izz="0.001" />
-    </inertial>
-  </link>
-  <joint name="base_footprint_joint" type="fixed">
-    <origin xyz="0 0 0.017" rpy="0 0 0" />
-    <parent link="base_footprint"/>
-    <child link="base_link" />
+    <collision name='right_wheel_collision'>
+      <geometry>
+        <cylinder radius=".1" length="0.06"/>
+      </geometry>
+      <surface>
+        <friction>
+          <ode>
+            <mu>0</mu>
+            <mu2>0</mu2>
+            <slip1>1.0</slip1>
+            <slip2>1.0</slip2>
+          </ode>
+        </friction>
+      </surface>
+    </collision>
+    <visual name='right_wheel_visual'>
+      <geometry>
+        <cylinder radius=".1" length="0.06"/>
+      </geometry>
+      <material name="red">
+        <color rgba=".8 0 0 1"/>
+      </material>
+    </visual>
+  </link>
+  <!--Creating hinge joints for the wheels-->
+  <joint type="revolute" name="left_wheel_hinge">
+    <origin xyz="0 0.275" rpy="0.1 0 0 0"/>
+    <child link="left_wheel"/>
+    <parent link="base_link"/>
+    <axis xyz="0 1 0"/>
+    <limit effort="30" velocity="1.0"/> <!--lower="-2.2" upper="0.7"-->
   </joint>
-  <joint name="base_wall_sensor_joint" type="fixed">
-    <origin xyz="0.09 -0.120 0.042" rpy="0 0 -1.0" />
+  <joint type="revolute" name="right_wheel_hinge">
+    <origin xyz="0 0.275 0.1" rpy="0 0 0"/>
+    <child link="right_wheel"/>
     <parent link="base_link"/>
-    <child link="wall_sensor_link" />
+    <axis xyz="0 1 0"/>
+    <limit effort="30" velocity="1.0"/> <!--lower="-2.2" upper="0.7"-->
   </joint>
-  <joint name="base_left_cliff_sensor_joint" type="fixed">
-    <origin xyz="0.07 0.14 0.01" rpy="0 1.57079 0" />
-    <parent link="base_link"/>
-    <child link="left_cliff_sensor_link" />
-  </joint>
-  <joint name="base_right_cliff_sensor_joint" type="fixed">
-    <origin xyz="0.07 -0.14 0.01" rpy="0 1.57079 0" />
-    <parent link="base_link"/>
-    <child link="right_cliff_sensor_link" />
-  </joint>
-  <joint name="base_leftfront_cliff_sensor_joint" type="fixed">
-    <origin xyz="0.15 0.04 0.01" rpy="0 1.57079 0" />
-    <parent link="base_link"/>
-    <child link="leftfront_cliff_sensor_link" />
-  </joint>
-  <joint name="base_rightfront_cliff_sensor_joint" type="fixed">
-    <origin xyz="0.15 -0.04 0.01" rpy="0 1.57079 0" />
-    <parent link="base_link"/>
-    <child link="rightfront_cliff_sensor_link" />
-  </joint>
-  <link name="left_wheel_link">
-    <inertial>
-      <origin xyz="0 0 0"/>
-      <mass value="0.01" />
-      <inertia ixx="0.001" ixy="0.0" ixz="0.0"
-        iyy="0.001" iyz="0.0" izz="0.001" />
-    </inertial>
-    <visual>
-      <origin xyz="0 0 0" rpy="0 1.5707 1.5707" />
-      <geometry>
-        <cylinder radius="0.033" length = "0.023"/>
-      </geometry>
-    </visual>
-    <collision>
-      <origin xyz="0 0 0" rpy="0 1.5707 1.5707" />
-      <geometry>
-        <cylinder radius="0.033" length = "0.023"/>
-      </geometry>
-    </collision>
-  </link>
-  <joint name="left_wheel_joint" type="continuous">
-    <origin xyz="0 0.13 0.015" rpy="0 0 0"/>
-    <parent link="base_link"/>
-    <child link="left_wheel_link"/>
-    <axis xyz="0 1 0"/>
-  </joint>
-  <link name="right_wheel_link">
-    <inertial>
-      <origin xyz="0 0 0"/>
-      <mass value="0.01" />
-      <inertia ixx="0.001" ixy="0.0" ixz="0.0"
-        iyy="0.001" iyz="0.0" izz="0.001" />
-    </inertial>
-    <visual>
-      <origin xyz="0 0 0" rpy="0 1.5707 1.5707" />
-      <geometry>
-        <cylinder radius="0.033" length = "0.023"/>
-      </geometry>
-    </visual>
-    <collision>
-      <origin xyz="0 0 0" rpy="0 1.5707 1.5707" />
-      <geometry>
-        <cylinder radius="0.033" length = "0.023"/>
-      </geometry>
-    </collision>
-  </link>
-  <joint name="right_wheel_joint" type="continuous">
-    <origin xyz="0 -0.13 0.015" rpy="0 0 0"/>
-    <parent link="base_link"/>
-    <child link="right_wheel_link"/>
-    <axis xyz="0 1 0"/>
-  </joint>
- <link name="rear_wheel_link">
-    <inertial>
-      <origin xyz="0 0 0"/>
-      <mass value="0.001" />
-      <inertia ixx="0.0001" ixy="0.0" ixz="0.0"
-        iyy="0.0001" iyz="0.0" izz="0.0001" />
-    </inertial>
-    <visual>
-      <origin xyz="0 0 0" rpy="0 1.5707 1.5707"/>
-      <geometry>
-        <sphere radius="0.015" />
-      </geometry>
-    </visual>
-    <collision>
-      <origin xyz="0 0 0" rpy="0 1.5707 1.5707" />
-      <geometry>
-        <sphere radius="0.015" />
-      </geometry>
-    </collision>
-  </link>
-  <!-- fixed because there's no transmission -->
-  <joint name="rear_castor_joint" type="fixed">
-    <origin xyz="-0.13 0 0.0" rpy="0 0 0"/>
-    <parent link="base_link"/>
-    <child link="rear_wheel_link"/>
-    <axis xyz="0 1 0"/>
-  </joint>
- <link name="front_wheel_link">
-    <inertial>
-      <origin xyz="0 0 0" />
-      <mass value="0.01" />
-      <inertia ixx="0.001" ixy="0.0" ixz="0.0"
-        iyy="0.001" iyz="0.0" izz="0.001" />
-    </inertial>
-    <visual>
-      <origin xyz="0 0 0" rpy="0 1.5707 1.5707"/>
-      <geometry>
-        <sphere radius="0.018" />
-      </geometry>
-    </visual>
-    <collision>
-      <origin xyz="0 0 0" rpy="0 1.5707 1.5707" />
-      <geometry>
-        <sphere radius="0.018" />
-      </geometry>
-    </collision>
-  </link>
-  <!-- fixed because there's no transmission -->
-  <joint name="front_castor_joint" type="fixed">
-    <origin xyz="0.13 0 0.0" rpy="0 0 0"/>
-    <parent link="base_link"/>
-    <child link="front_wheel_link"/>
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