Commit message: more slam to be tested

File: eklavya_description/urdf/eklavya_hardware.xacro (robot description, xacro)
@@ -25,5 +25,6 @@
           <box size=".03 .03 ${length}"/>
         </geometry>
-        <material name="White"/>
+        <!--<material name="White"/>-->
+        <material name="GunMetalBrushedAluminum"/>
       </visual>
     </link>
