Commit message: Tanmay's Update

File: eklavya_description/urdf/eklavya_calibration.xacro (robot description, xacro)
@@ -1,10 +1,10 @@
 <?xml version="1.0"?>
 <robot>
-  <property name="eklavya_calib_cam_x" value="${-0.0844382+0.36}" />
+  <property name="eklavya_calib_cam_x" value="${-0.0844382+0.36-0.55}" />
   <property name="eklavya_calib_cam_y" value="${0+ 0}" />
-  <property name="eklavya_calib_cam_z" value="${0.05+0.55}" />
+  <property name="eklavya_calib_cam_z" value="${0.05+0.55-0.18}" />
   <property name="eklavya_calib_cam_rr" value="0" />
   <property name="eklavya_calib_cam_rp" value="0" />
-  <property name="eklavya_calib_cam_ry" value="0" />
+  <property name="eklavya_calib_cam_ry" value="3.1415926535897932384626" />
   <property name="eklavya_camera_parent_name" value="base_link" />
 </robot>

File: eklavya_description/urdf/eklavya_hardware.xacro (robot description, xacro)
@@ -32,5 +32,5 @@
  <macro name="castor_support" params="suffix parent">
 	<joint type="fixed" name="${parent}_castor_support_${suffix}_joint">
-	  <origin rpy="0 0 0" xyz="${base_x_size/2+0.1} 0 ${0.02/2}"/>
+	  <origin rpy="0 0 0" xyz="${base_x_size/2} 0 0.058"/>
       <parent link="${parent}"/>
       <child link="${parent}_castor_support_${suffix}_link"/>
@@ -44,10 +44,10 @@
       <collision name='extrusion_collision'>
         <geometry>
-          <box size=".2 .1 .02"/>
+          <box size="0 0 0"/>
         </geometry>
       </collision>
       <visual name='extrusion_visual'>
         <geometry>
-          <box size=".2 .1 .02"/>
+          <box size="0 0 0"/>
         </geometry>
         <material name="GunMetalBrushedAluminum"/>
@@ -57,5 +57,5 @@
  <macro name="caster_support_hinge" params="suffix parent">
 	<joint name="${parent}_caster_support_hinge_${suffix}_joint" type="continuous">
-      <origin rpy="0 0 0" xyz="${base_x_size/2+0.1} 0 ${0.02-0.02}"/>
+      <origin rpy="0 0 0" xyz="${base_x_size/2} 0 0.058"/>
       <parent link="${parent}" />
       <child link="${parent}_caster_support_hinge_${suffix}_link"/>
@@ -88,5 +88,5 @@
 <macro name="caster_wheel" params="suffix parent">
 	  <joint name="${parent}_caster_wheel_${suffix}_joint" type="continuous">
-      <origin rpy="0 0 0" xyz="${-0.036} 0 ${-0.0818}" />
+      <origin rpy="0 0 0" xyz="0.066 0 -0.085" />
       <parent link="${parent}_caster_support_hinge_${suffix}_link" />
       <child link="${parent}_caster_wheel_${suffix}_link" />

File: eklavya_description/urdf/eklavya_kinect.urdf.xacro (robot description, xacro)
@@ -49,5 +49,5 @@
     </inertial>
     <visual>
-      <origin xyz=" 0 0 0 " rpy="0 0 0" />
+      <origin xyz="0 0 0 " rpy="0 0 0" />
       <geometry>
         <mesh filename="package://eklavya_description/meshes/kinect.dae"/>

File: eklavya_description/urdf/eklavya_wheel.xacro (robot description, xacro)
@@ -7,6 +7,8 @@
 	<property name="wheel_y_com" value="0.00000000" /> <!-- com : center of mass -->
 	<property name="wheel_z_com" value="0.00019000" /> <!-- com : center of mass -->
-	<property name="wheel_x_size" value="0.30550000" />
-	<property name="wheel_y_size" value="0.30550000" />
+	<!--property name="wheel_x_size" value="0.30550000" /-->
+	<!--property name="wheel_y_size" value="0.30550000" /-->
+	<property name="wheel_x_size" value="0.22" />
+	<property name="wheel_y_size" value="0.22" />
 	<property name="wheel_z_size" value="0.11430000" />
 	<property name="wheel_mass" value="2.63657000" /> <!-- in kg-->
@@ -17,7 +19,7 @@
 	<property name="wheel_iyz_com_cs" value="0.00000000" /> <!-- at center of mass aligned with coordinate system, kg*m^2-->
 	<property name="wheel_izz_com_cs" value="0.04410576" /> <!-- at center of mass aligned with coordinate system, kg*m^2-->
-	<property name="base_x_origin_to_wheel_origin" value="0.20" />
-	<property name="base_y_origin_to_wheel_origin" value="0.350" />
-	<property name="base_z_origin_to_wheel_origin" value="-0.0262508" />
+	<property name="base_x_origin_to_wheel_origin" value="0.15" />
+	<property name="base_y_origin_to_wheel_origin" value="0.225" />
+	<property name="base_z_origin_to_wheel_origin" value="0" />
   <macro name="eklavya_wheel" params="suffix parent *origin">
     <joint name="${parent}_${suffix}_wheel_joint" type="continuous">
@@ -39,5 +41,5 @@
       <visual>
         <eklavya_wheel_mesh suffix="${suffix}" />
-		<!--<material name="DarkGray" />-->
+		<material name="Red" />
       </visual>
       <collision>

File: eklavya_description/urdf/gazebo2.urdf.xacro (robot description, xacro)
@@ -25,5 +25,5 @@
 	  <insert_block name="origin" />
      <geometry>
-    <!--<mesh filename="package://eklavya_description/meshes/rmp50-base-link.dae" scale="0.0254 0.0254 0.0254"/> -->
+    <!-- mesh filename="package://eklavya_description/meshes/rmp50-base-link.dae" scale="0.0254 0.0254 0.0254"/ -->
     <mesh filename="package://eklavya_description/meshes/body.dae" />
   	<!-- <insert_block name="box" /> -->
@@ -34,5 +34,6 @@
     <origin xyz="0 0 0" rpy="0 0 0" />
     <geometry>
-      <mesh filename="package://eklavya_description/meshes/rmp50-castor-wheel.dae" scale="0.0220 0.0220 0.0220"/>
+      <!--mesh filename="package://eklavya_description/meshes/rmp50-castor-wheel.dae"/-->
+      <mesh filename="package://eklavya_description/meshes/castorWheel.dae" scale="2 2 2"/>
     </geometry>
   </macro>
@@ -46,9 +47,10 @@
     <origin xyz="0 0 0" rpy="0 0 0" />
     <geometry>
-      <mesh filename="package://eklavya_description/meshes/rmp50-castor-link.dae" scale="0.0220 0.0220 0.0220"/>
+      <!--mesh filename="package://eklavya_description/meshes/rmp50-castor-link.dae" scale="0.0220 0.0220 0.0220"/-->
+      <mesh filename="package://eklavya_description/meshes/wheelhub.dae"/> <!-- scale="0.0220 0.0220 0.0220"-->
     </geometry>
   </macro>
   <macro name="eklavya_wheel_mesh" params="suffix">
-    <origin xyz="0 0 0" rpy="0 0 0" />
+    <origin xyz="0 0 0" rpy="0 0 1.570796327" />
     <geometry>
      <!-- <mesh filename="package://eklavya_description/meshes/rmp50-${suffix}-wheel.dae" scale="0.0150 0.0150 0.0150"/>-->
