Commit message: ek2

File: eklavya_description/urdf/eklavya_body2.urdf.xacro (robot description, xacro)
@@ -23,5 +23,5 @@
     <property name="base_izz_com_cs" value="2.02955229" />
   <!-- Macro for eklavya body. Including Gazebo extensions, but does not include Kinect -->
-  <include filename="$(find eklavya_description)/urdf/gazebo.urdf.xacro"/>
+  <include filename="$(find eklavya_description)/urdf/gazebo2.urdf.xacro"/>
   <include filename="$(find eklavya_description)/urdf/materials.urdf.xacro"/>
   <include filename="$(find eklavya_description)/urdf/eklavya_hardware.xacro"/>
@@ -78,6 +78,6 @@
       <visual>
         <eklavya_base_link_mesh>
-          <origin xyz="0 0 ${base_x_size/2}" rpy="0 0 0" />
-           <!--  <origin xyz="-0.33 0 0.69" rpy="0 0 0" /> -->
+           <!--<origin xyz="0 0 ${base_x_size/2}" rpy="0 0 0" />-->
+            <origin xyz="-0.33 0 0.69" rpy="0 0 0" />
            <box size = "${base_x_size} ${base_y_size} ${base_z_size}"/>
         </eklavya_base_link_mesh>
@@ -93,17 +93,18 @@
     <gazebo_eklavya_base_link_surface />
 	 <!-- WHEEL macros -->
-    <eklavya_wheel suffix="left" parent="base_link">
+   <!-- <eklavya_wheel suffix="left" parent="base_link">
       <origin xyz="${ -1*base_x_origin_to_wheel_origin} ${base_y_origin_to_wheel_origin} ${ -1*base_z_origin_to_wheel_origin}" rpy="${M_PI} 0 0" />
     </eklavya_wheel>
     <eklavya_wheel suffix="right" parent="base_link">
       <origin xyz="${ -1*base_x_origin_to_wheel_origin} ${-1*base_y_origin_to_wheel_origin} ${ -1*base_z_origin_to_wheel_origin}" rpy="0 0 0" />
-    </eklavya_wheel>
+    </eklavya_wheel>  -->
     <!-- Castor -->
-    <castor_support suffix="front" parent="base_link" />
+  <!--  <castor_support suffix="front" parent="base_link" />
 	<caster_support_hinge suffix="front" parent="base_link" />
     <caster_wheel suffix="front" parent="base_link" />
+	-->
      <!-- DECORATIONS -->
      <!-- Bars -->
-	 <eklavya_support_bar suffix="left" parent="base_link" length="0.6">
+	<!--  <eklavya_support_bar suffix="left" parent="base_link" length="0.6">
       <origin rpy="0 0 0" xyz="${base_x_size/2-0.03/2} ${(base_y_size/2-0.03/2)} ${base_z_size+0.6/2}"/>
 	</eklavya_support_bar>
@@ -113,22 +114,22 @@
 	<eklavya_support_bar suffix="top" parent="base_link" length="0.55">
 		<origin rpy="${M_PI/2} 0 0"  xyz="${base_x_size/2-0.03/2} 0 ${base_z_size+0.6+0.03/2}"/>
-	</eklavya_support_bar>
+	</eklavya_support_bar>   -->
 	<!-- Controllers -->
    <!-- <gazebo_eklavya_simple_drive_plugin />    -->
-    <gazebo_eklavya_drive_plugin_diffdrive /><!-- cmd_vel movement -->
-    <gazebo_eklavya_p3d_plugin /> <!-- Ground Truth-->
-     <eklavya_controllers_common />
+  <!--   <gazebo_eklavya_drive_plugin_diffdrive /> --> <!-- cmd_vel movement -->
+  <!--   <gazebo_eklavya_p3d_plugin />--> <!-- Ground Truth-->
+  <!--    <eklavya_controllers_common />   -->
     <!-- Simulation sensors -->
-	<hokuyo_urg name="hokuyo_laser" parent="base_link" >
+	<!-- <hokuyo_urg name="hokuyo_laser" parent="base_link" >
       <origin rpy="0 0 0" xyz="${base_x_size/2+0.05} 0  0.021"/>
-    </hokuyo_urg>
-    <!-- <sick_lms100_200 name="sick_laser" parent="base_link" >
+    </hokuyo_urg> -->
+  <!--   <sick_lms100_200 name="sick_laser" parent="base_link" >
       <origin rpy="0 0 0" xyz="${base_x_size/2+0.12} 0  0.080"/>
     </sick_lms100_200>   -->
-	 <microstrain_imu name="eklavya_sim_imu" parent="base_link" imu_topic="imu/data" update_rate="30" stdevNoise="0.0017">
+	<!--  <microstrain_imu name="eklavya_sim_imu" parent="base_link" imu_topic="imu/data" update_rate="30" stdevNoise="0.0017">
 		 <origin rpy="0 0 0" xyz="${base_x_size/2-0.03/2} ${base_y_size/4} ${base_z_size}"/>
-	</microstrain_imu>
+	</microstrain_imu>  -->
     <!-- Kinect frames and mounting (includes simulation) -->
-    <eklavya_kinect/>
+    <!-- <eklavya_kinect/>  -->
   </xacro:macro>
 </robot>

File: eklavya_description/urdf/eklavya_kinect.urdf.xacro (robot description, xacro)
@@ -5,5 +5,5 @@
        xmlns:interface="http://playerstage.sourceforge.net/gazebo/xmlschema/#interface">
   <property name="M_PI" value="3.14159"/>
-  <include filename="$(find eklavya_description)/urdf/gazebo.urdf.xacro"/>
+  <!-- <include filename="$(find eklavya_description)/urdf/gazebo.urdf.xacro"/> -->
   <include filename="$(find eklavya_description)/urdf/eklavya_calibration.xacro" />
 <xacro:macro name="eklavya_sim_kinect">

Commit message: Tanmay's Update + IMU + Controller

File: eklavya_description/urdf/eklavya_body2.urdf.xacro (robot description, xacro)
@@ -6,7 +6,7 @@
     <!-- Main Body-base-->
     <!-- Location of com : center of mass -->
-    <property name="base_x_com" value="-0.04748000" />
-    <property name="base_y_com" value="-0.00000000" />
-    <property name="base_z_com" value="0.09947000" />
+    <property name="base_x_com" value="0" />
+    <property name="base_y_com" value="0" />
+    <property name="base_z_com" value="0" />
     <!-- Size of the base-->
     <property name="base_x_size" value="0.55000000" />
@@ -37,7 +37,7 @@
     <link name="base_footprint">
       <visual>
-        <origin xyz="0 0 0.0" rpy="0 0 0" />
+        <origin xyz="0 0 0" rpy="0 0 0" />
         <geometry>
-          <box size="0.001 0.001 0.001" />
+          <box size="0.1 0.1 0.01" />
         </geometry>
       </visual>
@@ -79,12 +79,11 @@
         <eklavya_base_link_mesh>
            <!--<origin xyz="0 0 ${base_x_size/2}" rpy="0 0 0" />-->
-            <origin xyz="-0.33 0 0.69" rpy="0 0 0" />
-           <box size = "${base_x_size} ${base_y_size} ${base_z_size}"/>
+            <origin xyz="0 0 0" rpy="0 0 0" />
+           <box size = "0.001 0.001 0.001"/>
         </eklavya_base_link_mesh>
       </visual>
       <collision>
         <eklavya_base_link_mesh>
-	   <origin xyz="0 0 0" rpy="0 0 0" />
-            <!-- <origin xyz="0 0 ${base_x_size/2 }" rpy="0 0 0 " /> -->
+            <origin xyz="0 0 0" rpy="0 0 0" />
            <box size = "${base_x_size} ${base_y_size} ${base_z_size}"/> <!--making it slightly bigger in x and z direction-->
         </eklavya_base_link_mesh>
@@ -93,43 +92,33 @@
     <gazebo_eklavya_base_link_surface />
 	 <!-- WHEEL macros -->
-   <!-- <eklavya_wheel suffix="left" parent="base_link">
+   <eklavya_wheel suffix="left" parent="base_link">
       <origin xyz="${ -1*base_x_origin_to_wheel_origin} ${base_y_origin_to_wheel_origin} ${ -1*base_z_origin_to_wheel_origin}" rpy="${M_PI} 0 0" />
     </eklavya_wheel>
     <eklavya_wheel suffix="right" parent="base_link">
       <origin xyz="${ -1*base_x_origin_to_wheel_origin} ${-1*base_y_origin_to_wheel_origin} ${ -1*base_z_origin_to_wheel_origin}" rpy="0 0 0" />
-    </eklavya_wheel>  -->
+    </eklavya_wheel>
     <!-- Castor -->
-  <!--  <castor_support suffix="front" parent="base_link" />
+    <castor_support suffix="front" parent="base_link" />
 	<caster_support_hinge suffix="front" parent="base_link" />
     <caster_wheel suffix="front" parent="base_link" />
-	-->
-     <!-- DECORATIONS -->
-     <!-- Bars -->
-	<!--  <eklavya_support_bar suffix="left" parent="base_link" length="0.6">
-      <origin rpy="0 0 0" xyz="${base_x_size/2-0.03/2} ${(base_y_size/2-0.03/2)} ${base_z_size+0.6/2}"/>
-	</eklavya_support_bar>
-	<eklavya_support_bar suffix="right" parent="base_link" length="0.6">
-     <origin rpy="0 0 0" xyz="${base_x_size/2-0.03/2} ${-1*(base_y_size/2+-0.03/2)} ${base_z_size+0.6/2}"/>
-	</eklavya_support_bar>
-	<eklavya_support_bar suffix="top" parent="base_link" length="0.55">
-		<origin rpy="${M_PI/2} 0 0"  xyz="${base_x_size/2-0.03/2} 0 ${base_z_size+0.6+0.03/2}"/>
-	</eklavya_support_bar>   -->
-	<!-- Controllers -->
+<!-- Controllers -->
    <!-- <gazebo_eklavya_simple_drive_plugin />    -->
-  <!--   <gazebo_eklavya_drive_plugin_diffdrive /> --> <!-- cmd_vel movement -->
-  <!--   <gazebo_eklavya_p3d_plugin />--> <!-- Ground Truth-->
-  <!--    <eklavya_controllers_common />   -->
+    <gazebo_eklavya_drive_plugin_diffdrive /><!-- cmd_vel movement -->
+    <gazebo_eklavya_p3d_plugin /> <!-- Ground Truth-->
+     <eklavya_controllers_common />
     <!-- Simulation sensors -->
-	<!-- <hokuyo_urg name="hokuyo_laser" parent="base_link" >
-      <origin rpy="0 0 0" xyz="${base_x_size/2+0.05} 0  0.021"/>
-    </hokuyo_urg> -->
+    <hokuyo_urg name="hokuyo_laser" parent="base_link" >
+      <origin rpy="0 0 0" xyz="${-base_x_size/2} 0  0.23"/>
+    </hokuyo_urg>
   <!--   <sick_lms100_200 name="sick_laser" parent="base_link" >
       <origin rpy="0 0 0" xyz="${base_x_size/2+0.12} 0  0.080"/>
     </sick_lms100_200>   -->
-	<!--  <microstrain_imu name="eklavya_sim_imu" parent="base_link" imu_topic="imu/data" update_rate="30" stdevNoise="0.0017">
-		 <origin rpy="0 0 0" xyz="${base_x_size/2-0.03/2} ${base_y_size/4} ${base_z_size}"/>
-	</microstrain_imu>  -->
+	 <microstrain_imu name="eklavya_sim_imu" parent="base_link" imu_topic="imu/data" update_rate="30" stdevNoise="0.0017">
+		 <origin rpy="0 0 0" xyz="0 0 0"/>
+	</microstrain_imu>
     <!-- Kinect frames and mounting (includes simulation) -->
-    <!-- <eklavya_kinect/>  -->
+    <eklavya_kinect>
+	  <!--origin rpy="0 0 ${M_PI/2}" xyz="${-base_x_size/2-0.05} 0  0.6"/-->
+	</eklavya_kinect>
   </xacro:macro>
 </robot>

Commit message: without Controller

File: eklavya_description/urdf/eklavya_body2.urdf.xacro (robot description, xacro)
@@ -102,16 +102,16 @@
 	<caster_support_hinge suffix="front" parent="base_link" />
     <caster_wheel suffix="front" parent="base_link" />
-<!-- Controllers -->
-   <!-- <gazebo_eklavya_simple_drive_plugin />    -->
-    <gazebo_eklavya_drive_plugin_diffdrive /><!-- cmd_vel movement -->
-    <gazebo_eklavya_p3d_plugin /> <!-- Ground Truth-->
-     <eklavya_controllers_common />
+	<!-- Controllers -->
+	<!-- <gazebo_eklavya_simple_drive_plugin />    -->
+	<!--  <gazebo_eklavya_drive_plugin_diffdrive /> --><!-- cmd_vel movement -->
+	<gazebo_eklavya_p3d_plugin /> <!-- Ground Truth-->
+	<eklavya_controllers_common />
     <!-- Simulation sensors -->
     <hokuyo_urg name="hokuyo_laser" parent="base_link" >
-      <origin rpy="0 0 0" xyz="${-base_x_size/2} 0  0.23"/>
+      <origin rpy="0 0 ${M_PI}" xyz="${-base_x_size/2} 0  0.33"/>
     </hokuyo_urg>
-  <!--   <sick_lms100_200 name="sick_laser" parent="base_link" >
-      <origin rpy="0 0 0" xyz="${base_x_size/2+0.12} 0  0.080"/>
-    </sick_lms100_200>   -->
+	<!--<sick_lms100_200 name="sick_laser" parent="base_link" >
+		<origin rpy="0 0 0" xyz="${base_x_size/2+0.12} 0  0.080"/>
+	</sick_lms100_200>   -->
 	 <microstrain_imu name="eklavya_sim_imu" parent="base_link" imu_topic="imu/data" update_rate="30" stdevNoise="0.0017">
 		 <origin rpy="0 0 0" xyz="0 0 0"/>
