Commit message: semi_fixed

File: eklavya_description/urdf/eklavya_body.urdf.xacro (robot description, xacro)
@@ -1,13 +1,10 @@
 <?xml version="1.0"?>
 <robot name="eklavya_hardware" xmlns:xacro="http://ros.org/wiki/xacro">
-  <property name="M_PI" value="3.14159"/>
   <!-- Macro for eklavya body. Including Gazebo extensions, but does not include Kinect -->
   <!--<include filename="$(find eklavya_description)/urdf/gazebo.urdf.xacro"/>-->
-  <property name="base_x" value="0.33" />
-  <property name="base_y" value="0.33" />
  <xacro:macro name="eklavya_body">
     <!--  INSERT YOU MODEL HERE -->
   <link name='base_link'>
-    <pose>0 0 .375 0 0 3.14</pose>
+    <origin rpy="0 0 3.14" xyz="0 0 .375"/>
     <inertial>
       <mass value="0.0001" />
@@ -116,5 +113,5 @@
   <!--Left_Wheel-->
   <link name="left_wheel">
-    <pose>0.278 0.275 0.1 1.5707 0 1.5707</pose>
+     <origin rpy="1.5707 0 1.5707" xyz="0 1.275 0.1"/>
     <inertial>
       <mass value="0.0001" />
@@ -142,6 +139,6 @@
         <cylinder radius=".1" length="0.06"/>
       </geometry>
-      <material name="red">
-        <color rgba=".8 0 0 1"/>
+      <material name="green">
+        <color rgba="0 .8 0 1"/>
       </material>
     </visual>
@@ -149,5 +146,5 @@
   <!--Right_Wheel-->
   <link name="right_wheel">
-    <pose>-0.278 0.275 0.1 1.5707 0 1.5707</pose>
+    <origin rpy="1.5707 0 1.5707" xyz="0 0.275 0.1"/>
     <inertial>
       <mass value="0.0001" />
@@ -175,6 +172,6 @@
         <cylinder radius=".1" length="0.06"/>
       </geometry>
-      <material name="red">
-        <color rgba=".8 0 0 1"/>
+      <material name="blue">
+        <color rgba="0 0 .8 1"/>
       </material>
     </visual>
@@ -182,16 +179,16 @@
   <!--Creating hinge joints for the wheels-->
   <joint type="revolute" name="left_wheel_hinge">
-    <origin xyz="0 0.275" rpy="0.1 0 0 0"/>
+    <origin xyz="0.278 0.275 0.1 " rpy="0 0 0"/>
     <child link="left_wheel"/>
     <parent link="base_link"/>
     <axis xyz="0 1 0"/>
-    <limit effort="30" velocity="1.0"/> <!--lower="-2.2" upper="0.7"-->
+    <limit effort="30" velocity="1.0" lower="-2.2" upper="0.7" />
   </joint>
   <joint type="revolute" name="right_wheel_hinge">
-    <origin xyz="0 0.275 0.1" rpy="0 0 0"/>
+    <origin xyz="-0.278 0.275 0.1" rpy="0 0 0"/>
     <child link="right_wheel"/>
     <parent link="base_link"/>
     <axis xyz="0 1 0"/>
-    <limit effort="30" velocity="1.0"/> <!--lower="-2.2" upper="0.7"-->
+    <limit effort="30" velocity="1.0" lower="-2.2" upper="0.7" />
   </joint>
   <!--  INSERT YOU MODEL HERE -->

Commit message: 

File: eklavya_description/urdf/eklavya_body.urdf.xacro (robot description, xacro)
@@ -2,5 +2,5 @@
 <robot name="eklavya_hardware" xmlns:xacro="http://ros.org/wiki/xacro">
   <!-- Macro for eklavya body. Including Gazebo extensions, but does not include Kinect -->
-  <!--<include filename="$(find eklavya_description)/urdf/gazebo.urdf.xacro"/>-->
+  <include filename="$(find eklavya_description)/urdf/gazebo.urdf.xacro"/>
  <xacro:macro name="eklavya_body">
     <!--  INSERT YOU MODEL HERE -->
@@ -179,20 +179,20 @@
   <!--Creating hinge joints for the wheels-->
   <joint type="revolute" name="left_wheel_hinge">
-    <origin xyz="0.278 0.275 0.1 " rpy="0 0 0"/>
+    <origin xyz="0.278 0.275 0.1 " rpy="1.5707 0 1.5707"/>
     <child link="left_wheel"/>
     <parent link="base_link"/>
-    <axis xyz="0 1 0"/>
+    <axis xyz="0 0 1"/>
     <limit effort="30" velocity="1.0" lower="-2.2" upper="0.7" />
   </joint>
   <joint type="revolute" name="right_wheel_hinge">
-    <origin xyz="-0.278 0.275 0.1" rpy="0 0 0"/>
+    <origin xyz="-0.278 0.275 0.1" rpy="1.5707 0 1.5707"/>
     <child link="right_wheel"/>
     <parent link="base_link"/>
-    <axis xyz="0 1 0"/>
+    <axis xyz="0 0 1"/>
     <limit effort="30" velocity="1.0" lower="-2.2" upper="0.7" />
   </joint>
   <!--  INSERT YOU MODEL HERE -->
   <!-- Simulation sensors -->
-  <!--  <eklavya_sim_imu/>
+    <!--<eklavya_sim_imu/>
   <eklavya_sim_laser/>
 <eklavya_sim_create/>

Commit message: visible in Gazebo with changes like <mass value="2.0001" />       <inertia ixx="0.01" ixy="0.0" ixz="0.0" iyy="0.01" iyz="0.0" izz="0.5"/>

File: eklavya_description/urdf/eklavya_body.urdf.xacro (robot description, xacro)
@@ -5,11 +5,36 @@
  <xacro:macro name="eklavya_body">
     <!--  INSERT YOU MODEL HERE -->
-  <link name='base_link'>
-    <origin rpy="0 0 3.14" xyz="0 0 .375"/>
+  <material name="Green">
+    <color rgba="0.0 0.8 0.0 1.0"/>
+  </material>
+  <link name="base_footprint">
+    <!--
     <inertial>
       <mass value="0.0001" />
+      <origin xyz="0 0 0" />
       <inertia ixx="0.0001" ixy="0.0" ixz="0.0"
               iyy="0.0001" iyz="0.0"
               izz="0.0001" />
+    </inertial>
+-->
+    <visual>
+      <origin rpy="0 0 0" xyz="0 0 0"/>
+      <geometry>
+        <box size="0.001 0.001 0.001"/>
+      </geometry>
+      <material name="Green"/>
+    </visual>
+    <collision>
+      <origin rpy="0 0 0" xyz="0 0 0.017"/>
+      <geometry>
+        <box size="0.001 0.001 0.001"/>
+      </geometry>
+    </collision>
+  </link>
+  <link name='base_link'>
+   <origin rpy="0 0 3.14" xyz="0 0 .375"/>
+    <inertial>
+      <mass value="2.0001" />
+      <inertia ixx="0.01" ixy="0.0" ixz="0.0" iyy="0.01" iyz="0.0" izz="0.5"/>
     </inertial>
     <collision name='collision'>
@@ -115,8 +140,6 @@
      <origin rpy="1.5707 0 1.5707" xyz="0 1.275 0.1"/>
     <inertial>
-      <mass value="0.0001" />
-      <inertia ixx="0.0001" ixy="0.0" ixz="0.0"
-              iyy="0.0001" iyz="0.0"
-              izz="0.0001" />
+      <mass value="0.2001" />
+      <inertia ixx="0.01" ixy="0.0" ixz="0.0" iyy="0.01" iyz="0.0" izz="0.5"/>
     </inertial>
     <collision name='left_wheel_collision'>
@@ -148,8 +171,6 @@
     <origin rpy="1.5707 0 1.5707" xyz="0 0.275 0.1"/>
     <inertial>
-      <mass value="0.0001" />
-      <inertia ixx="0.0001" ixy="0.0" ixz="0.0"
-              iyy="0.0001" iyz="0.0"
-              izz="0.0001" />
+      <mass value="0.2001" />
+      <inertia ixx="0.01" ixy="0.0" ixz="0.0" iyy="0.01" iyz="0.0" izz="0.5"/>
     </inertial>
     <collision name='right_wheel_collision'>
@@ -177,18 +198,21 @@
     </visual>
   </link>
+  <joint name="base_footprint_joint" type="fixed">
+    <origin rpy="0 0 0" xyz="0 0 0.017"/>
+    <parent link="base_footprint"/>
+    <child link="base_link"/>
+  </joint>
   <!--Creating hinge joints for the wheels-->
-  <joint type="revolute" name="left_wheel_hinge">
+  <joint type="continuous" name="left_wheel_hinge">
     <origin xyz="0.278 0.275 0.1 " rpy="1.5707 0 1.5707"/>
     <child link="left_wheel"/>
     <parent link="base_link"/>
     <axis xyz="0 0 1"/>
-    <limit effort="30" velocity="1.0" lower="-2.2" upper="0.7" />
   </joint>
-  <joint type="revolute" name="right_wheel_hinge">
+  <joint type="continuous" name="right_wheel_hinge">
     <origin xyz="-0.278 0.275 0.1" rpy="1.5707 0 1.5707"/>
     <child link="right_wheel"/>
     <parent link="base_link"/>
     <axis xyz="0 0 1"/>
-    <limit effort="30" velocity="1.0" lower="-2.2" upper="0.7" />
   </joint>
   <!--  INSERT YOU MODEL HERE -->

Commit message: 

File: eklavya_description/urdf/eklavya_body.urdf.xacro (robot description, xacro)
@@ -3,9 +3,7 @@
   <!-- Macro for eklavya body. Including Gazebo extensions, but does not include Kinect -->
   <include filename="$(find eklavya_description)/urdf/gazebo.urdf.xacro"/>
+  <include filename="$(find eklavya_description)/urdf/materials.urdf.xacro"/>
  <xacro:macro name="eklavya_body">
     <!--  INSERT YOU MODEL HERE -->
-  <material name="Green">
-    <color rgba="0.0 0.8 0.0 1.0"/>
-  </material>
   <link name="base_footprint">
     <!--
@@ -23,5 +21,5 @@
         <box size="0.001 0.001 0.001"/>
       </geometry>
-      <material name="Green"/>
+      <material name="Red"/>
     </visual>
     <collision>
@@ -47,7 +45,5 @@
         <box size=".55 .55 .55"/>
       </geometry>
-      <material name="red">
-        <color rgba=".8 0 0 1"/>
-      </material>
+      <material name="Blue"/>
     </visual>
   </link>
@@ -147,14 +143,4 @@
         <cylinder radius=".1" length="0.06"/>
       </geometry>
-      <surface>
-        <friction>
-          <ode>
-            <mu>0</mu>
-            <mu2>0</mu2>
-            <slip1>1.0</slip1>
-            <slip2>1.0</slip2>
-          </ode>
-        </friction>
-      </surface>
     </collision>
     <visual name='left_wheel_visual'>
@@ -162,7 +148,5 @@
         <cylinder radius=".1" length="0.06"/>
       </geometry>
-      <material name="green">
-        <color rgba="0 .8 0 1"/>
-      </material>
+      <material name="Green"/>
     </visual>
   </link>
@@ -178,14 +162,4 @@
         <cylinder radius=".1" length="0.06"/>
       </geometry>
-      <surface>
-        <friction>
-          <ode>
-            <mu>0</mu>
-            <mu2>0</mu2>
-            <slip1>1.0</slip1>
-            <slip2>1.0</slip2>
-          </ode>
-        </friction>
-      </surface>
     </collision>
     <visual name='right_wheel_visual'>
@@ -193,7 +167,5 @@
         <cylinder radius=".1" length="0.06"/>
       </geometry>
-      <material name="blue">
-        <color rgba="0 0 .8 1"/>
-      </material>
+     <material name="Blue"/>
     </visual>
   </link>

Commit message: texture working in rviz

File: eklavya_description/urdf/eklavya_body.urdf.xacro (robot description, xacro)
@@ -21,5 +21,5 @@
         <box size="0.001 0.001 0.001"/>
       </geometry>
-      <material name="Red"/>
+      <material name="Green"/>
     </visual>
     <collision>
@@ -45,5 +45,5 @@
         <box size=".55 .55 .55"/>
       </geometry>
-      <material name="Blue"/>
+      <material name="GunMetalBrushedAluminum"/>
     </visual>
   </link>

Commit message: not working wheel xacro (segbot_file called)

File: eklavya_description/urdf/eklavya_body.urdf.xacro (robot description, xacro)
@@ -4,4 +4,5 @@
   <include filename="$(find eklavya_description)/urdf/gazebo.urdf.xacro"/>
   <include filename="$(find eklavya_description)/urdf/materials.urdf.xacro"/>
+  <include filename="$(find eklavya_description)/urdf/eklavya_wheel.xacro"/>
   <xacro:macro name="eklavya_body">
     <!--  INSERT YOU MODEL HERE -->
@@ -46,8 +47,16 @@
         <geometry>
           <box size=".55 .55 .55"/>
-        </geometry>
+         </geometry>
         <material name="GunMetalBrushedAluminum"/>
       </visual>
     </link>
+     <!-- left wheel -->
+    <eklavya_wheel suffix="left" parent="base_link">
+     <origin rpy="1.5707 0 1.5707" xyz="-.375 -.275 -0.2"/>
+    </eklavya_wheel>
+    <!-- right wheel -->
+    <eklavya_wheel suffix="right" parent="base_link">
+      <origin rpy="1.5707 0 1.5707" xyz=".375 -.275 -.2"/>
+    </eklavya_wheel>
     <!--Top of base_link supports-->
     <link name="base_link_support_1">
@@ -153,42 +162,45 @@
       </visual>
     </link>
-    <!--Link for Left_Wheel-->
-    <link name="left_wheel">
-      <origin rpy="0 1.5707 0" xyz="0 1.275 0.1"/>
-      <inertial>
-        <mass value="0.2001" />
-        <inertia ixx="0.01" ixy="0.0" ixz="0.0" iyy="0.01" iyz="0.0" izz="0.5"/>
-      </inertial>
-      <collision name='left_wheel_collision'>
-        <geometry>
-          <cylinder radius=".1" length="0.06"/>
-        </geometry>
-      </collision>
-      <visual name='left_wheel_visual'>
-        <geometry>
-          <cylinder radius=".1" length="0.06"/>
-        </geometry>
-        <material name="Grey"/>
-      </visual>
-    </link>
-    <!--Link for Right_Wheel-->
-    <link name="right_wheel">
-      <origin rpy="0 1.5707 0" xyz="0 0.275 0.1"/>
-      <inertial>
-        <mass value="0.2001" />
-        <inertia ixx="0.01" ixy="0.0" ixz="0.0" iyy="0.01" iyz="0.0" izz="0.5"/>
-      </inertial>
-      <collision name='right_wheel_collision'>
-        <geometry>
-          <cylinder radius=".1" length="0.06"/>
-        </geometry>
-      </collision>
-      <visual name='right_wheel_visual'>
-        <geometry>
-          <cylinder radius=".1" length="0.06"/>
-        </geometry>
-        <material name="Grey2"/>
-      </visual>
-    </link>
+    <!--Links for sensor integration-->
+    <!--IMU link-->
+   <!-- <link name="IMU_sensor_link">
+      <inertial>
+        <mass value="0.01" />
+        <origin xyz="0 0 0"/>
+        <inertia ixx="0.001" ixy="0.0" ixz="0.0"
+                  iyy="0.001" iyz="0.0" izz="0.001" />
+      </inertial>
+    </link>
+-->
+    <!--BumbleBee link-->
+   <!-- <link name="BumbleBee_sensor_link">
+      <inertial>
+        <mass value="0.01" />
+        <origin xyz="0 0 0"/>
+        <inertia ixx="0.001" ixy="0.0" ixz="0.0"
+                 iyy="0.001" iyz="0.0" izz="0.001" />
+      </inertial>
+    </link>
+ -->
+    <!--LIDAR link-->
+    <!--<link name="LIDAR_sensor_link">
+      <inertial>
+        <mass value="0.01" />
+        <origin xyz="0 0 0"/>
+        <inertia ixx="0.001" ixy="0.0" ixz="0.0"
+                 iyy="0.001" iyz="0.0" izz="0.001" />
+      </inertial>
+    </link>
+-->
+    <!--GPS link-->
+   <!-- <link name="GPS_sensor_link">
+      <inertial>
+        <mass value="0.01" />
+        <origin xyz="0 0 0"/>
+        <inertia ixx="0.001" ixy="0.0" ixz="0.0"
+                 iyy="0.001" iyz="0.0" izz="0.001" />
+      </inertial>
+    </link>
+-->
     <!--JOINTS-->
     <!--Joining base_link and dummy base-->
@@ -198,18 +210,4 @@
       <child link="base_link"/>
     </joint>
-    <!--Creating hinge joints for the LEFT wheel-->
-    <joint type="continuous" name="left_wheel_hinge">
-      <origin rpy="1.5707 0 1.5707" xyz="-.375 -.275 -0.2"/>
-      <child link="left_wheel"/>
-      <parent link="base_link"/>
-      <axis xyz="0 0 1"/>
-    </joint>
-    <!--Creating hinge joints for the RIGHT wheel-->
-    <joint type="continuous" name="right_wheel_hinge">
-      <origin rpy="1.5707 0 1.5707" xyz=".375 -.275 -.2"/>
-      <child link="right_wheel"/>
-      <parent link="base_link"/>
-      <axis xyz="0 0 1"/>
-    </joint>
     <!--Creating fixed joints for base link supports-->
     <joint type="fixed" name="base_link_support_1_joint">
@@ -240,5 +238,67 @@
       <child link="castor"/>
     </joint>
+    <!--Joint for IMU-->
+   <!-- <joint name="IMU_sensor_joint" type="fixed">
+      <origin xyz="0.26 0.26 0.275" rpy="0 0 -1.0" />
+      <parent link="base_link"/>
+      <child link="IMU_sensor_link" />
+    </joint>
+-->
+    <!--Joint for BumbleBee Sterio Camera-->
+   <!-- <joint name="BumbleBee_sensor_joint" type="fixed">
+      <origin rpy="0 0 0" xyz="0 0.26 0.89"/>
+      <parent link="base_link"/>
+      <child link="BumbleBee_sensor_link" />
+    </joint>
+-->
+    <!--Joint for LIDAR-->
+   <!-- <joint name="LIDAR_sensor_joint" type="fixed">
+      <origin xyz="0 0.375 -0.3" rpy="0 0 -1.0" />
+      <parent link="base_link"/>
+      <child link="LIDAR_sensor_link" />
+    </joint>
+-->
+    <!-- try  try try-->
+  <!--  <joint name="hokuyo_laser_box_joint" type="fixed">
+      <origin xyz="0 0 0" rpy="0 0 0"/>
+      <parent link="LIDAR_sensor_link"/>
+      <child link="hokuyo_laser_box_link"/>
+    </joint>
+    <link name="hokuyo_laser_box_link">
+      <inertial>
+        <mass value="0.01"/>
+        <origin xyz="0 0 0"/>
+        <inertia ixx="0.001" ixy="0.0" ixz="0.0" iyy="0.001" iyz="0.0" izz="0.001"/>
+      </inertial>
+      <visual>
+        <origin xyz="0 0 0" rpy="0 0 0"/>
+        <geometry>-->
+        <!-- box size="0.05 0.05 0.1" / -->
+        <!--<mesh filename="package://meshes/collada/hokuyo_urg.dae" scale="0.5 0.5 0.5"/>
+        </geometry>
+      </visual>
+      <collision>
+        <origin xyz="0 0 0" rpy="0 0 0"/>
+        <geometry>
+          <box size="0.05 0.05 0.1"/>
+        </geometry>
+      </collision>
+    </link>
+    <gazebo reference="hokuyo_laser_box_link">
+      <material>Gazebo/Magenta</material>
+      <turnGravityOff>false</turnGravityOff>
+    </gazebo>-->
+    <!-- try  try try-->
+    <!--Joint for GPS-->
+   <!-- <joint name="GPS_sensor_joint" type="fixed">
+      <origin xyz="-0.26 0.26 0.275" rpy="0 0 -1.0" />
+      <parent link="base_link"/>
+      <child link="GPS_sensor_link" />
+    </joint>
+-->
     <!--  INSERT YOU MODEL HERE -->
+    <hokuyo_urg name="hokuyo_laser" parent="base_link" >
+      <origin xyz="0 0.375 -0.3" rpy="0 1 0"/>
+    </hokuyo_urg>
     <!-- Simulation sensors -->
     <!--<eklavya_sim_imu/>

File: eklavya_description/urdf/eklavya_wheel.xacro (robot description, xacro)
@@ -4,5 +4,6 @@
   xmlns:controller="http://playerstage.sourceforge.net/gazebo/xmlschema/#controller"
   xmlns:interface="http://playerstage.sourceforge.net/gazebo/xmlschema/#interface">
-  <macro name="segbot_wheel" params="suffix parent *origin">
+  <include filename="$(find eklavya_description)/urdf/gazebo_segbot.xacro" />
+  <macro name="eklavya_wheel" params="suffix parent *origin">
     <joint name="${parent}_${suffix}_wheel_joint" type="continuous">
       <insert_block name="origin" />

Commit message: rviz

File: eklavya_description/urdf/eklavya_body.urdf.xacro (robot description, xacro)
@@ -53,9 +53,9 @@
      <!-- left wheel -->
     <eklavya_wheel suffix="left" parent="base_link">
-     <origin rpy="1.5707 0 1.5707" xyz="-.375 -.275 -0.2"/>
+     <origin rpy="0 -1 0" xyz="-.375 -.275 -0.2"/>
     </eklavya_wheel>
     <!-- right wheel -->
     <eklavya_wheel suffix="right" parent="base_link">
-      <origin rpy="1.5707 0 1.5707" xyz=".375 -.275 -.2"/>
+      <origin rpy="0 0 0" xyz=".375 -.275 -.2"/>
     </eklavya_wheel>
     <!--Top of base_link supports-->

File: eklavya_description/urdf/gazebo_segbot.xacro (robot description, xacro)
@@ -5,5 +5,5 @@
   xmlns:interface="http://playerstage.sourceforge.net/gazebo/xmlschema/#interface">
   <!-- Included URDF Files -->
-  <include filename="$(find segbot_description)/urdf/gazebo_segbot_common.xacro" />
+  <include filename="$(find eklavya_description)/urdf/gazebo_segbot_common.xacro" />
   <macro name="segbot_base_link_visual" >
     <segbot_base_link_mesh />

File: eklavya_description/urdf/gazebo_segbot_common.xacro (robot description, xacro)
@@ -23,5 +23,5 @@
     <origin xyz="0 0 0" rpy="0 0 0" />
     <geometry>
-      <mesh filename="package://segbot_description/meshes/rmp50-base-link.dae" scale="0.0254 0.0254 0.0254"/>
+      <mesh filename="package://eklavya_description/meshes/rmp50-base-link.dae" scale="0.0254 0.0254 0.0254"/>
     </geometry>
   </macro>
@@ -35,5 +35,5 @@
     <origin xyz="0 0 0" rpy="0 0 0" />
     <geometry>
-      <mesh filename="package://segbot_description/meshes/rmp50-castor-wheel.dae" scale="0.0254 0.0254 0.0254"/>
+      <mesh filename="package://eklavya_description/meshes/rmp50-castor-wheel.dae" scale="0.0254 0.0254 0.0254"/>
     </geometry>
   </macro>
@@ -47,5 +47,5 @@
     <origin xyz="0 0 0" rpy="0 0 0" />
     <geometry>
-      <mesh filename="package://segbot_description/meshes/rmp50-castor-link.dae" scale="0.0254 0.0254 0.0254"/>
+      <mesh filename="package://eklavya_description/meshes/rmp50-castor-link.dae" scale="0.0254 0.0254 0.0254"/>
     </geometry>
   </macro>

File: eklavya_description/urdf/gazebo_segbot_simple.xacro (robot description, xacro)
@@ -2,5 +2,5 @@
 <robot>
   <!-- Included URDF Files -->
-  <include filename="$(find segbot_description)/urdf/gazebo_common.xacro" />
+  <include filename="$(find eklavya_description)/urdf/gazebo_common.xacro" />
   <macro name="segbot_base_link_visual" >
     <segbot_base_link_mesh />

Commit message: rviz working

File: eklavya_description/urdf/eklavya_body.urdf.xacro (robot description, xacro)
@@ -53,9 +53,9 @@
      <!-- left wheel -->
     <eklavya_wheel suffix="left" parent="base_link">
-     <origin rpy="0 -1 0" xyz="-.375 -.275 -0.2"/>
+     <origin rpy="0 0 1.5707" xyz="-.375 -.275 -0.2"/>
     </eklavya_wheel>
     <!-- right wheel -->
     <eklavya_wheel suffix="right" parent="base_link">
-      <origin rpy="0 0 0" xyz=".375 -.275 -.2"/>
+      <origin rpy="0 0 1.5707" xyz=".375 -.275 -.2"/>
     </eklavya_wheel>
     <!--Top of base_link supports-->
