Commit message: making the model right

File: eklavya_description/urdf/eklavya_body.urdf.xacro (robot description, xacro)
@@ -3,121 +3,135 @@
   <!-- Macro for eklavya body. Including Gazebo extensions, but does not include Kinect -->
   <include filename="$(find eklavya_description)/urdf/gazebo.urdf.xacro"/>
+  <include filename="$(find eklavya_description)/urdf/gazebo_segbot.xacro" />
   <include filename="$(find eklavya_description)/urdf/materials.urdf.xacro"/>
   <include filename="$(find eklavya_description)/urdf/eklavya_wheel.xacro"/>
+  <include filename="$(find eklavya_description)/urdf/hokuyo_urg.xacro"/>
   <xacro:macro name="eklavya_body">
-    <!--  INSERT YOU MODEL HERE -->
     <!--Dummy base without INERTIA because base_link is not supposed to have inertia-->
     <link name="base_footprint">
+      <visual>
+        <origin xyz="0 0 0" rpy="0 0 0" />
+        <geometry>
+          <box size="0.001 0.001 0.001" />
+        </geometry>
+      </visual>
+    </link>
+    <joint name="base_footprint_joint" type="fixed">
+      <origin xyz="0.0 0 0.5" rpy="0 0 0" />
+      <parent link="base_footprint"/>
+      <child link="base_link" />
+    </joint>
+    <!-- Links and Joints (i.e., the robot) -->
+    <link name="base_link">
+      <inertial>
+        <mass value="0.01" />
+        <origin xyz="0 0 0" />
+        <inertia ixx="1.0" ixy="0.0" ixz="0.0"
+          iyy="1.0" iyz="0.0"
+          izz="1.0" />
+      </inertial>
+      <visual>
+        <eklavya_base_link_mesh />
+      </visual>
+      <collision>
+        <eklavya_base_link_mesh />
+      </collision>
+    </link>
+    <gazebo_eklavya_base_link_surface />
+    <joint name="base_center_of_mass_joint" type="fixed">
+      <origin xyz="-0.1 0 -0.075" rpy="0 0 0" />
+      <parent link="base_link"/>
+      <child link="base_center_of_mass_link" />
+    </joint>
+    <link name="base_center_of_mass_link">
+      <inertial>
+        <mass value="30" />
+        <origin xyz="0 0 0" />
+        <inertia ixx="1.0" ixy="0.0" ixz="0.0"
+          iyy="1.0" iyz="0.0"
+          izz="1.0" />
+      </inertial>
+    </link>
+    <eklavya_wheel suffix="left" parent="base_link">
+      <origin xyz="-0.2 0.335 -0.2239" rpy="0 0 0" />
+    </eklavya_wheel>
+    <eklavya_wheel suffix="right" parent="base_link">
+      <origin xyz="-0.2 -0.335 -0.2239" rpy="0 0 0" />
+    </eklavya_wheel>
+    <joint type="fixed" name="base_link_support_left_joint">
+      <origin rpy="0 0 0" xyz="0.26 0.26 0.575"/>
+      <parent link="base_link"/>
+      <child link="base_link_support_left"/>
+    </joint>
+    <link name="base_link_support_left">
+      <origin rpy="0 0 0" xyz="0 0 0"/>
+      <inertial>
+        <mass value="2.0001" />
+        <inertia ixx="1" ixy="0.0" ixz="0.0" iyy="1" iyz="0.0" izz="1"/>
+      </inertial>
+      <collision name='sc1'>
+        <geometry>
+          <box size=".03 .03 .6"/>
+        </geometry>
+      </collision>
+      <visual name='sv1'>
+        <geometry>
+          <box size=".03 .03 .6"/>
+        </geometry>
+        <material name="Black"/>
+      </visual>
+    </link>
+     <joint type="fixed" name="base_link_support_right_joint">
+      <origin rpy="0 0 0" xyz="0.26 -0.26 0.575"/>
+      <parent link="base_link"/>
+      <child link="base_link_support_right"/>
+    </joint>
+    <link name="base_link_support_right">
+      <origin rpy="0 0 0" xyz="0 0 0"/>
+      <inertial>
+        <mass value="2.0001" />
+        <inertia ixx="1" ixy="0.0" ixz="0.0" iyy="1" iyz="0.0" izz="1"/>
+      </inertial>
+      <collision name='sc2'>
+        <geometry>
+          <box size=".03 .03 .6"/>
+        </geometry>
+      </collision>
+      <visual name='sv2'>
+        <geometry>
+          <box size=".03 .03 .6"/>
+        </geometry>
+        <material name="White"/>
+      </visual>
+    </link>
+    <joint type="fixed" name="base_link_support_top_joint">
+      <origin rpy="0 0  ${M_PI/2}" xyz="0.26 0 0.89"/>
+      <parent link="base_link"/>
+      <child link="base_link_support_top"/>
+    </joint>
+    <link name="base_link_support_top">
+      <origin rpy="0 0 0" xyz="0 0 0"/>
+      <inertial>
+        <mass value="2.0001" />
+        <inertia ixx="1" ixy="0.0" ixz="0.0" iyy="1" iyz="0.0" izz="1"/>
+      </inertial>
+      <collision name='sc3'>
+        <geometry>
+          <box size=".55 .03 .03"/>
+        </geometry>
+      </collision>
+      <visual name='sv3'>
+        <geometry>
+          <box size=".55 .03 .03"/>
+        </geometry>
+        <material name="Red"/>
+      </visual>
+    </link>
     <!--
-    <inertial>
-      <mass value="0.0001" />
-      <origin xyz="0 0 0" />
-      <inertia ixx="0.0001" ixy="0.0" ixz="0.0"
-               iyy="0.0001" iyz="0.0"
-               izz="0.0001" />
-      </inertial>
-    -->
-      <visual>
-        <origin rpy="0 0 0" xyz="0 0 0"/>
-        <geometry>
-          <box size="0.001 0.001 0.001"/>
-        </geometry>
-        <material name="Green"/>
-      </visual>
-      <collision>
-        <origin rpy="0 0 0" xyz="0 0 0.017"/>
-        <geometry>
-          <box size="0.001 0.001 0.001"/>
-        </geometry>
-      </collision>
-    </link>
-    <!--Base link with inertial properties to join with other links of the model-->
-    <link name='base_link'>
-      <origin rpy="0 0 3.14" xyz="0 0 .375"/>
-      <inertial>
-        <mass value="2.0001" />
-        <inertia ixx="0.01" ixy="0.0" ixz="0.0" iyy="0.01" iyz="0.0" izz="0.5"/>
-      </inertial>
-      <collision name='collision'>
-        <geometry>
-          <box size=".55 .55 .55"/>
-        </geometry>
-      </collision>
-      <visual name='visual'>
-        <geometry>
-          <box size=".55 .55 .55"/>
-         </geometry>
-        <material name="GunMetalBrushedAluminum"/>
-      </visual>
-    </link>
-     <!-- left wheel -->
-    <eklavya_wheel suffix="left" parent="base_link">
-     <origin rpy="0 0 1.5707" xyz="-.375 -.275 -0.2"/>
-    </eklavya_wheel>
-    <!-- right wheel -->
-    <eklavya_wheel suffix="right" parent="base_link">
-      <origin rpy="0 0 1.5707" xyz=".375 -.275 -.2"/>
-    </eklavya_wheel>
-    <!--Top of base_link supports-->
-    <link name="base_link_support_1">
-      <origin rpy="0 0 0" xyz="0.26 0.26 0.575"/>
-      <inertial>
-        <mass value="2.0001" />
-        <inertia ixx="0.01" ixy="0.0" ixz="0.0" iyy="0.01" iyz="0.0" izz="0.5"/>
-      </inertial>
-      <collision name='sc1'>
-        <geometry>
-          <box size=".03 .03 .6"/>
-        </geometry>
-      </collision>
-      <visual name='sv1'>
-        <geometry>
-          <box size=".03 .03 .6"/>
-        </geometry>
-        <material name="Black"/>
-      </visual>
-    </link>
-    <link name="base_link_support_2">
-      <origin rpy="0 0 0" xyz="-0.26 0.26 0.575"/>
-      <inertial>
-        <mass value="2.0001" />
-        <inertia ixx="0.01" ixy="0.0" ixz="0.0" iyy="0.01" iyz="0.0" izz="0.5"/>
-      </inertial>
-      <collision name='sc2'>
-        <geometry>
-          <box size=".03 .03 .6"/>
-        </geometry>
-      </collision>
-      <visual name='sv2'>
-        <geometry>
-          <box size=".03 .03 .6"/>
-        </geometry>
-        <material name="White"/>
-      </visual>
-    </link>
-    <link name="base_link_support_3">
-      <origin rpy="0 0 0" xyz="0 0.26 0.89"/>
-      <inertial>
-        <mass value="2.0001" />
-        <inertia ixx="0.01" ixy="0.0" ixz="0.0" iyy="0.01" iyz="0.0" izz="0.5"/>
-      </inertial>
-      <collision name='sc3'>
-        <geometry>
-          <box size=".55 .03 .03"/>
-        </geometry>
-      </collision>
-      <visual name='sv3'>
-        <geometry>
-          <box size=".55 .03 .03"/>
-        </geometry>
-        <material name="Red"/>
-      </visual>
-    </link>
-    <!--Link for Castor Support-->
     <link name="castor_support">
       <origin rpy="0 0 0" xyz="0 0.375 -0.275"/>
       <inertial>
         <mass value="2.0001" />
-        <inertia ixx="0.01" ixy="0.0" ixz="0.0" iyy="0.01" iyz="0.0" izz="0.5"/>
+        <inertia ixx="1" ixy="0.0" ixz="0.0" iyy="1" iyz="0.0" izz="1"/>
       </inertial>
       <collision name='extrusion_collision'>
@@ -133,10 +147,14 @@
       </visual>
     </link>
-    <!--Link for Castor-->
+        <joint type="fixed" name="castor_support_joint">
+      <origin rpy="0 0 0" xyz="0 0.375 -0.275"/>
+      <parent link="base_link"/>
+      <child link="castor_support"/>
+    </joint>
     <link name="castor">
    	  <origin rpy="0 0 0" xyz="0 0.375 -0.325"/>
       <inertial>
         <mass value="2.0001" />
-        <inertia ixx="0.01" ixy="0.0" ixz="0.0" iyy="0.01" iyz="0.0" izz="0.5"/>
+        <inertia ixx="1" ixy="0.0" ixz="0.0" iyy="1" iyz="0.0" izz="1"/>
       </inertial>
       <collision name='caster_collision'>
@@ -162,4 +180,10 @@
       </visual>
     </link>
+     <joint type="fixed" name="castor_joint">
+      <origin rpy="0 0 0" xyz="0 0.375 -0.325"/>
+      <parent link="base_link"/>
+      <child link="castor"/>
+    </joint>
+  -->
     <!--Links for sensor integration-->
     <!--IMU link-->
@@ -203,39 +227,5 @@
     </link>
 -->
-    <!--JOINTS-->
-    <!--Joining base_link and dummy base-->
-    <joint name="base_footprint_joint" type="fixed">
-      <origin rpy="0 0 0" xyz="0 0 0.017"/>
-      <parent link="base_footprint"/>
-      <child link="base_link"/>
-    </joint>
     <!--Creating fixed joints for base link supports-->
-    <joint type="fixed" name="base_link_support_1_joint">
-      <origin rpy="0 0 0" xyz="0.26 0.26 0.575"/>
-      <parent link="base_link"/>
-      <child link="base_link_support_1"/>
-    </joint>
-    <joint type="fixed" name="base_link_support_2_joint">
-      <origin rpy="0 0 0" xyz="-0.26 0.26 0.575"/>
-      <parent link="base_link"/>
-      <child link="base_link_support_2"/>
-    </joint>
-    <joint type="fixed" name="base_link_support_3_joint">
-      <origin rpy="0 0 0" xyz="0 0.26 0.89"/>
-      <parent link="base_link"/>
-      <child link="base_link_support_3"/>
-    </joint>
-    <!--Creating joint for Castor Support-->
-    <joint type="fixed" name="castor_support_joint">
-      <origin rpy="0 0 0" xyz="0 0.375 -0.275"/>
-      <parent link="base_link"/>
-      <child link="castor_support"/>
-    </joint>
-    <!--Creating joint for CASTOR-->
-    <joint type="fixed" name="castor_joint">
-      <origin rpy="0 0 0" xyz="0 0.375 -0.325"/>
-      <parent link="base_link"/>
-      <child link="castor"/>
-    </joint>
     <!--Joint for IMU-->
    <!-- <joint name="IMU_sensor_joint" type="fixed">
@@ -298,7 +288,8 @@
 -->
     <!--  INSERT YOU MODEL HERE -->
-    <hokuyo_urg name="hokuyo_laser" parent="base_link" >
+   <!-- <hokuyo_urg name="hokuyo_laser" parent="base_link" >
       <origin xyz="0 0.375 -0.3" rpy="0 1 0"/>
     </hokuyo_urg>
+     -->
     <!-- Simulation sensors -->
     <!--<eklavya_sim_imu/>

File: eklavya_description/urdf/eklavya_wheel.xacro (robot description, xacro)
@@ -4,5 +4,4 @@
   xmlns:controller="http://playerstage.sourceforge.net/gazebo/xmlschema/#controller"
   xmlns:interface="http://playerstage.sourceforge.net/gazebo/xmlschema/#interface">
-  <include filename="$(find eklavya_description)/urdf/gazebo_segbot.xacro" />
   <macro name="eklavya_wheel" params="suffix parent *origin">
     <joint name="${parent}_${suffix}_wheel_joint" type="continuous">

File: eklavya_description/urdf/gazebo.urdf.xacro (robot description, xacro)
@@ -1,24 +1,3 @@
 <?xml version="1.0"?>
 <robot xmlns:controller="http://playerstage.sourceforge.net/gazebo/xmlschema/#controller" xmlns:interface="http://playerstage.sourceforge.net/gazebo/xmlschema/#interface" xmlns:sensor="http://playerstage.sourceforge.net/gazebo/xmlschema/#sensor" xmlns:xacro="http://ros.org/wiki/xacro" name="eklavya_gazebo">
-  <gazebo reference="left_wheel">
-    <mu1 value="10"/>
-    <mu2 value="10"/>
-    <kp value="100000000.0"/>
-    <kd value="10000.0"/>
-    <fdir value="1 0 0"/>
-  </gazebo>
-  <gazebo reference="right_wheel">
-    <mu1 value="10"/>
-    <mu2 value="10"/>
-    <kp value="100000000.0"/>
-    <kd value="10000.0"/>
-    <fdir value="1 0 0"/>
-  </gazebo>
-  <gazebo reference="castor">
-    <mu1 value="0"/>
-    <mu2 value="0"/>
-    <kp value="100000000.0"/>
-    <kd value="10000.0"/>
-    <fdir value="1 0 0"/>
-  </gazebo>
 </robot>

File: eklavya_description/urdf/gazebo_segbot_common.xacro (robot description, xacro)
@@ -4,5 +4,12 @@
   xmlns:controller="http://playerstage.sourceforge.net/gazebo/xmlschema/#controller"
   xmlns:interface="http://playerstage.sourceforge.net/gazebo/xmlschema/#interface">
-  <macro name="gazebo_segbot_base_link_surface">
+<gazebo reference="castor">
+    <mu1 value="0"/>
+    <mu2 value="0"/>
+    <kp value="100000000.0"/>
+    <kd value="10000.0"/>
+    <fdir value="1 0 0"/>
+  </gazebo>
+  <macro name="gazebo_eklavya_base_link_surface">
     <gazebo reference="base_link">
       <mu1 value="100.0" />
@@ -20,15 +27,11 @@
     </gazebo>
   </macro>
-  <macro name="segbot_base_link_mesh">
+  <macro name="eklavya_base_link_mesh">
     <origin xyz="0 0 0" rpy="0 0 0" />
     <geometry>
-      <mesh filename="package://eklavya_description/meshes/rmp50-base-link.dae" scale="0.0254 0.0254 0.0254"/>
+     <!-- <mesh filename="package://eklavya_description/meshes/rmp50-base-link.dae" scale="0.0254 0.0254 0.0254"/> -->
+    <box size=".55 .55 .55"/>
     </geometry>
-  </macro>
-  <macro name="segbot_base_link_cylinder">
-    <origin xyz="0 0 0" rpy="0 0 0" />
-    <geometry>
-      <cylinder length="0.4330" radius="0.6" />
-    </geometry>
+     <material name="GunMetalBrushedAluminum"/>
   </macro>
   <macro name="segbot_castor_wheel_link_mesh">

File: eklavya_description/urdf/gazebo_segbot_simple.xacro (robot description, xacro)
@@ -4,8 +4,8 @@
   <include filename="$(find eklavya_description)/urdf/gazebo_common.xacro" />
   <macro name="segbot_base_link_visual" >
-    <segbot_base_link_mesh />
+    <eklavya_base_link_mesh />
   </macro>
   <macro name="segbot_base_link_collision" >
-    <segbot_base_link_cylinder />
+    <eklavya_base_link_mesh />
   </macro>
   <macro name="segbot_castor_support_link_visual" >

Commit message: laser working too

File: eklavya_description/urdf/eklavya_body.urdf.xacro (robot description, xacro)
@@ -54,8 +54,8 @@
     </link>
     <eklavya_wheel suffix="left" parent="base_link">
-      <origin xyz="-0.2 0.335 -0.2239" rpy="0 0 0" />
+      <origin xyz="-0.2 0.335 -0.303" rpy="0 0 0" />
     </eklavya_wheel>
     <eklavya_wheel suffix="right" parent="base_link">
-      <origin xyz="-0.2 -0.335 -0.2239" rpy="0 0 0" />
+      <origin xyz="-0.2 -0.335 -0.303" rpy="0 0 0" />
     </eklavya_wheel>
     <joint type="fixed" name="base_link_support_left_joint">
@@ -128,28 +128,87 @@
       </visual>
     </link>
+  <joint type="fixed" name="castor_support_joint">
+	  <origin rpy="0 0 0" xyz="0.36 0 -0.255"/>
+      <parent link="base_link"/>
+      <child link="castor_support"/>
+    </joint>
+    <link name="castor_support">
+      <origin rpy="0 0 0" xyz="0 0 0"/>
+      <inertial>
+        <mass value="2.0001" />
+        <inertia ixx="1" ixy="0.0" ixz="0.0" iyy="1" iyz="0.0" izz="1"/>
+      </inertial>
+      <collision name='extrusion_collision'>
+        <geometry>
+          <box size=".2 .1 .02"/>
+        </geometry>
+      </collision>
+      <visual name='extrusion_visual'>
+        <geometry>
+          <box size=".2 .1 .02"/>
+        </geometry>
+        <material name="Blue"/>
+      </visual>
+    </link>
+ <joint name="base_caster_support_joint" type="continuous">
+      <origin xyz="0.36 0 -0.275" rpy="0 0 0" />
+      <parent link="base_link" />
+      <child link="base_caster_support_link"/>
+      <axis xyz="0 0 1" />
+      <anchor xyz="0.01 0 0" />
+      <limit effort="100" velocity="100" k_velocity="0" />
+      <joint_properties damping="0.0" friction="0.0" />
+    </joint>
+    <transmission type="pr2_mechanism_model/SimpleTransmission" name="base_caster_support_trans">
+      <actuator name="base_caster_support_motor" />
+      <joint name="base_caster_support_joint" />
+      <mechanicalReduction>1.0</mechanicalReduction>
+    </transmission>
+    <link name="base_caster_support_link">
+      <inertial>
+        <mass value="1"/>
+        <origin xyz="0 0 0" />
+        <inertia ixx="0.00375" ixy="0.0" ixz="0.0"
+          iyy="0.00375" iyz="0.0"
+          izz="0.00375" />
+      </inertial>
+      <visual>
+        <eklavya_castor_support_link_mesh />
+      </visual>
+      <collision>
+        <eklavya_castor_support_link_mesh />
+      </collision>
+    </link>
+<joint name="caster_wheel_joint" type="continuous">
+      <origin xyz="-0.0397 0 -0.0918" rpy="0 0 0" />
+      <parent link="base_caster_support_link" />
+      <child link="caster_wheel_link" />
+      <axis xyz="0 1 0" />
+      <anchor xyz="0 0 0" />
+      <limit effort="100" velocity="100" k_velocity="0" />
+      <joint_properties damping="0.0" friction="0.0" />
+    </joint>
+    <transmission type="pr2_mechanism_model/SimpleTransmission" name="caster_wheel_trans">
+      <actuator name="caster_wheel_motor" />
+      <joint name="caster_wheel_joint" />
+      <mechanicalReduction>1.0</mechanicalReduction>
+    </transmission>
+    <link name="caster_wheel_link">
+      <inertial>
+        <mass value="2" />
+        <origin xyz="0 0 0" rpy="0 0 0" />
+        <inertia  ixx="0.003" ixy="0.0" ixz="0.0"
+          iyy="0.00581" iyz="0.0"
+          izz="0.003" />
+      </inertial>
+      <visual>
+        <eklavya_castor_wheel_link_mesh />
+      </visual>
+      <collision>
+        <eklavya_castor_wheel_link_mesh />
+      </collision>
+    </link>
+    <gazebo_castor_wheel_link_surface />
     <!--
-    <link name="castor_support">
-      <origin rpy="0 0 0" xyz="0 0.375 -0.275"/>
-      <inertial>
-        <mass value="2.0001" />
-        <inertia ixx="1" ixy="0.0" ixz="0.0" iyy="1" iyz="0.0" izz="1"/>
-      </inertial>
-      <collision name='extrusion_collision'>
-        <geometry>
-          <box size=".1 .2 .02"/>
-        </geometry>
-      </collision>
-      <visual name='extrusion_visual'>
-        <geometry>
-          <box size=".1 .2 .02"/>
-        </geometry>
-        <material name="Blue"/>
-      </visual>
-    </link>
-        <joint type="fixed" name="castor_support_joint">
-      <origin rpy="0 0 0" xyz="0 0.375 -0.275"/>
-      <parent link="base_link"/>
-      <child link="castor_support"/>
-    </joint>
     <link name="castor">
    	  <origin rpy="0 0 0" xyz="0 0.375 -0.325"/>
@@ -279,22 +338,18 @@
       <turnGravityOff>false</turnGravityOff>
     </gazebo>-->
-    <!-- try  try try-->
     <!--Joint for GPS-->
-   <!-- <joint name="GPS_sensor_joint" type="fixed">
+    <!--
+    <joint name="GPS_sensor_joint" type="fixed">
       <origin xyz="-0.26 0.26 0.275" rpy="0 0 -1.0" />
       <parent link="base_link"/>
       <child link="GPS_sensor_link" />
-    </joint>
--->
+    </joint> -->
     <!--  INSERT YOU MODEL HERE -->
-   <!-- <hokuyo_urg name="hokuyo_laser" parent="base_link" >
-      <origin xyz="0 0.375 -0.3" rpy="0 1 0"/>
+    <hokuyo_urg name="hokuyo_laser" parent="base_link" >
+      <origin rpy="0 0 0" xyz="0.36 0 -0.245"/>
     </hokuyo_urg>
-     -->
     <!-- Simulation sensors -->
     <!--<eklavya_sim_imu/>
-    <eklavya_sim_laser/>
-    <eklavya_sim_create/>
-    <eklavya_sim_wall_sensors/>-->
+      -->
   </xacro:macro>
 </robot>

File: eklavya_description/urdf/gazebo_segbot_common.xacro (robot description, xacro)
@@ -35,5 +35,5 @@
      <material name="GunMetalBrushedAluminum"/>
   </macro>
-  <macro name="segbot_castor_wheel_link_mesh">
+  <macro name="eklavya_castor_wheel_link_mesh">
     <origin xyz="0 0 0" rpy="0 0 0" />
     <geometry>
@@ -47,5 +47,5 @@
     </geometry>
   </macro>
-  <macro name="segbot_castor_support_link_mesh">
+  <macro name="eklavya_castor_support_link_mesh">
     <origin xyz="0 0 0" rpy="0 0 0" />
     <geometry>
@@ -56,5 +56,5 @@
     <origin xyz="0 0 0" rpy="0 0 0" />
     <geometry>
-      <mesh filename="package://eklavya_description/meshes/rmp50-${suffix}-wheel.dae" scale="0.0254 0.0254 0.0254"/>
+      <mesh filename="package://eklavya_description/meshes/rmp50-${suffix}-wheel.dae" scale="0.0150 0.0150 0.0150"/>
     </geometry>
   </macro>
