Commit message: Bot moving in Gazebo with Teleop

File: eklavya_description/urdf/eklavya_body.urdf.xacro (robot description, xacro)
@@ -1,7 +1,17 @@
 <?xml version="1.0"?>
 <robot name="eklavya_hardware" xmlns:xacro="http://ros.org/wiki/xacro">
+<!-- Properties (Constants) -->
+    <property name="M_PI" value="3.14159"/>
+    <property name="base_size_x" value="0.217" />
+    <property name="base_size_y" value="0.280" />
+    <property name="base_size_z" value="0.155" />
+    <property name="top_size_x" value="0.3937" />
+    <property name="top_size_y" value="0.3556" />
+    <property name="top_size_z" value="0.0020" />
+    <property name="wheel_radius" value="0.0346" />
+    <property name="wheel_length" value="0.02" />
+    <property name="caster_wheel_offset_y" value="0.27" />
   <!-- Macro for eklavya body. Including Gazebo extensions, but does not include Kinect -->
   <include filename="$(find eklavya_description)/urdf/gazebo.urdf.xacro"/>
-  <include filename="$(find eklavya_description)/urdf/gazebo_segbot.xacro" />
   <include filename="$(find eklavya_description)/urdf/materials.urdf.xacro"/>
   <include filename="$(find eklavya_description)/urdf/eklavya_wheel.xacro"/>
@@ -345,5 +355,5 @@
       <child link="GPS_sensor_link" />
     </joint> -->
-    <!--  INSERT YOU MODEL HERE -->
+    <gazebo_segbot_drive_plugin2 />
     <hokuyo_urg name="hokuyo_laser" parent="base_link" >
       <origin rpy="0 0 0" xyz="0.36 0 -0.245"/>

File: eklavya_description/urdf/eklavya_wheel.xacro (robot description, xacro)
@@ -23,8 +23,8 @@
       </inertial>
       <visual>
-        <segbot_wheel_visual suffix="${suffix}" />
+        <segbot_wheel_mesh suffix="${suffix}" />
       </visual>
       <collision>
-        <segbot_wheel_collision suffix="${suffix}" />
+        <segbot_wheel_mesh suffix="${suffix}" />
       </collision>
     </link>

File: eklavya_description/urdf/gazebo.urdf.xacro (robot description, xacro)
@@ -1,3 +1,137 @@
 <?xml version="1.0"?>
-<robot xmlns:controller="http://playerstage.sourceforge.net/gazebo/xmlschema/#controller" xmlns:interface="http://playerstage.sourceforge.net/gazebo/xmlschema/#interface" xmlns:sensor="http://playerstage.sourceforge.net/gazebo/xmlschema/#sensor" xmlns:xacro="http://ros.org/wiki/xacro" name="eklavya_gazebo">
+<robot
+  xmlns:sensor="http://playerstage.sourceforge.net/gazebo/xmlschema/#sensor"
+  xmlns:controller="http://playerstage.sourceforge.net/gazebo/xmlschema/#controller"
+  xmlns:interface="http://playerstage.sourceforge.net/gazebo/xmlschema/#interface">
+<gazebo reference="castor">
+    <mu1 value="0"/>
+    <mu2 value="0"/>
+    <kp value="100000000.0"/>
+    <kd value="10000.0"/>
+    <fdir value="1 0 0"/>
+  </gazebo>
+  <macro name="gazebo_eklavya_base_link_surface">
+    <gazebo reference="base_link">
+      <mu1 value="100.0" />
+      <mu2 value="100.0" />
+      <kp  value="1000000.0" />
+      <kd  value="1.0" />
+    </gazebo>
+  </macro>
+  <macro name="gazebo_segbot_castor_wheel_link_surface">
+    <gazebo reference="caster_wheel_link">
+      <mu1 value="10.0" />
+      <mu2 value="10.0" />
+      <kp  value="1000000.0" />
+      <kd  value="1.0" />
+    </gazebo>
+  </macro>
+  <macro name="eklavya_base_link_mesh">
+    <origin xyz="0 0 0" rpy="0 0 0" />
+    <geometry>
+     <!-- <mesh filename="package://eklavya_description/meshes/rmp50-base-link.dae" scale="0.0254 0.0254 0.0254"/> -->
+    <box size=".55 .55 .55"/>
+    </geometry>
+     <material name="GunMetalBrushedAluminum"/>
+  </macro>
+  <macro name="eklavya_castor_wheel_link_mesh">
+    <origin xyz="0 0 0" rpy="0 0 0" />
+    <geometry>
+      <mesh filename="package://eklavya_description/meshes/rmp50-castor-wheel.dae" scale="0.0254 0.0254 0.0254"/>
+    </geometry>
+  </macro>
+  <macro name="segbot_collision_none">
+    <origin xyz="0 0 0" rpy="0 0 0" />
+    <geometry>
+      <box size="0.01 0.01 0.01" />
+    </geometry>
+  </macro>
+  <macro name="eklavya_castor_support_link_mesh">
+    <origin xyz="0 0 0" rpy="0 0 0" />
+    <geometry>
+      <mesh filename="package://eklavya_description/meshes/rmp50-castor-link.dae" scale="0.0254 0.0254 0.0254"/>
+    </geometry>
+  </macro>
+  <macro name="segbot_wheel_mesh" params="suffix">
+    <origin xyz="0 0 0" rpy="0 0 0" />
+    <geometry>
+      <mesh filename="package://eklavya_description/meshes/rmp50-${suffix}-wheel.dae" scale="0.0150 0.0150 0.0150"/>
+    </geometry>
+  </macro>
+  <macro name="gazebo_segbot_wheel_surface">
+    <gazebo reference="${parent}_${suffix}_wheel_link" >
+      <mu1 value="10.0" />
+      <mu2 value="10.0" />
+      <kp  value="1000000.0" />
+      <kd  value="1.0" />
+    </gazebo>
+  </macro>
+  <macro name="gazebo_segbot_controllers_common">
+    <canonicalBody>base_footprint</canonicalBody>
+    <controller:gazebo_ros_controller_manager name="gazebo_ros_controller_manager" plugin="libgazebo_ros_controller_manager.so">
+      <alwaysOn>true</alwaysOn>
+      <updateRate>5.0</updateRate>
+      <interface:audio name="gazebo_ros_controller_manager_dummy_iface" />
+    </controller:gazebo_ros_controller_manager>
+  </macro>
+  <macro name="gazebo_segbot_drive_parameters">
+    <alwaysOn>true</alwaysOn>
+    <update>100</update>
+    <updateRate>100.0</updateRate>
+    <leftJoint>base_link_right_wheel_joint</leftJoint>
+    <rightJoint>base_link_left_wheel_joint</rightJoint>
+    <wheelSeparation>0.5380</wheelSeparation>
+    <wheelDiameter>0.2410</wheelDiameter>
+    <torque>20</torque>
+    <interface:position name="position_iface_0"/>
+    <topicName>cmd_vel</topicName>
+  </macro>
+  <macro name="gazebo_segbot_simple_drive_plugin">
+    <controller:segbotsimpledrive_plugin name="differential_drive_controller" plugin="libsegbotsimpledrive_plugin.so">
+      <gazebo_segbot_drive_parameters />
+    </controller:segbotsimpledrive_plugin>
+  </macro>
+  <macro name="gazebo_segbot_drive_plugin">
+    <controller:segbotdrive_plugin name="differential_drive_controller" plugin="libsegbotdrive_plugin.so">
+      <gazebo_segbot_drive_parameters />
+    </controller:segbotdrive_plugin>
+   </macro>
+ <!-- CONTROLLERS -->
+ <macro name="gazebo_segbot_drive_plugin2">
+        <gazebo>
+            <controller:diffdrive_plugin name="differential_drive_controller" plugin="libdiffdrive_plugin.so">
+                <alwaysOn>true</alwaysOn>
+                <update>100</update>
+                <updateRate>100.0</updateRate>
+                <leftJoint>base_link_right_wheel_joint</leftJoint>
+                <rightJoint>base_link_left_wheel_joint</rightJoint>
+                <wheelSeparation>${caster_wheel_offset_y*2}</wheelSeparation>
+                <wheelDiameter>${wheel_radius*2}</wheelDiameter>
+                <torque>50</torque>
+                <interface:position name="position_iface_0"/>
+                <robotNamespace>/</robotNamespace>
+                <topicName>cmd_vel</topicName>
+            </controller:diffdrive_plugin>
+            <controller:gazebo_ros_p3d name="p3d_base_controller" plugin="libgazebo_ros_p3d.so">
+                <alwaysOn>true</alwaysOn>
+                <updateRate>100.0</updateRate>
+                <bodyName>base_link</bodyName>
+                <topicName>base_pose_ground_truth</topicName>
+                <gaussianNoise>0.01</gaussianNoise>
+                <frameName>map</frameName>
+                <xyzOffsets>0 0 0</xyzOffsets>
+                <rpyOffsets>0 0 0</rpyOffsets>
+                <interface:position name="p3d_base_position"/>
+            </controller:gazebo_ros_p3d>
+            <canonicalBody>base_footprint</canonicalBody>
+            <!-- this publishes empty joint_states due to no transmission, but
+             triggering robot_state_publisher to publish tf between fixed joints in create,
+             (e.g. base_laser_link for the base_scan frame) -->
+            <controller:gazebo_ros_controller_manager name="gazebo_ros_controller_manager" plugin="libgazebo_ros_controller_manager.so">
+                <alwaysOn>true</alwaysOn>
+                <updateRate>100.0</updateRate>
+                <interface:audio name="gazebo_ros_controller_manager_dummy_iface" />
+            </controller:gazebo_ros_controller_manager>
+        </gazebo>
+  </macro>
 </robot>

Commit message: updating xacros

File: eklavya_description/urdf/eklavya_body.urdf.xacro (robot description, xacro)
@@ -15,4 +15,5 @@
   <include filename="$(find eklavya_description)/urdf/gazebo.urdf.xacro"/>
   <include filename="$(find eklavya_description)/urdf/materials.urdf.xacro"/>
+  <include filename="$(find eklavya_description)/urdf/eklavya_hardware.xacro.xacro"/>
   <include filename="$(find eklavya_description)/urdf/eklavya_wheel.xacro"/>
   <include filename="$(find eklavya_description)/urdf/hokuyo_urg.xacro"/>
@@ -69,190 +70,22 @@
       <origin xyz="-0.2 -0.335 -0.303" rpy="0 0 0" />
     </eklavya_wheel>
-    <joint type="fixed" name="base_link_support_left_joint">
+	<eklavya_bar suffix="left" parent="base_link">
       <origin rpy="0 0 0" xyz="0.26 0.26 0.575"/>
-      <parent link="base_link"/>
-      <child link="base_link_support_left"/>
-    </joint>
-    <link name="base_link_support_left">
-      <origin rpy="0 0 0" xyz="0 0 0"/>
-      <inertial>
-        <mass value="2.0001" />
-        <inertia ixx="1" ixy="0.0" ixz="0.0" iyy="1" iyz="0.0" izz="1"/>
-      </inertial>
-      <collision name='sc1'>
-        <geometry>
-          <box size=".03 .03 .6"/>
-        </geometry>
-      </collision>
-      <visual name='sv1'>
-        <geometry>
-          <box size=".03 .03 .6"/>
-        </geometry>
-        <material name="Black"/>
-      </visual>
-    </link>
-     <joint type="fixed" name="base_link_support_right_joint">
+	</eklavya_bar>
+	<eklavya_bar suffix="right" parent="base_link">
       <origin rpy="0 0 0" xyz="0.26 -0.26 0.575"/>
-      <parent link="base_link"/>
-      <child link="base_link_support_right"/>
-    </joint>
-    <link name="base_link_support_right">
-      <origin rpy="0 0 0" xyz="0 0 0"/>
-      <inertial>
-        <mass value="2.0001" />
-        <inertia ixx="1" ixy="0.0" ixz="0.0" iyy="1" iyz="0.0" izz="1"/>
-      </inertial>
-      <collision name='sc2'>
-        <geometry>
-          <box size=".03 .03 .6"/>
-        </geometry>
-      </collision>
-      <visual name='sv2'>
-        <geometry>
-          <box size=".03 .03 .6"/>
-        </geometry>
-        <material name="White"/>
-      </visual>
-    </link>
-    <joint type="fixed" name="base_link_support_top_joint">
+	</eklavya_bar>
+	<eklavya_bar suffix="top" parent="base_link">
       <origin rpy="0 0  ${M_PI/2}" xyz="0.26 0 0.89"/>
-      <parent link="base_link"/>
-      <child link="base_link_support_top"/>
-    </joint>
-    <link name="base_link_support_top">
-      <origin rpy="0 0 0" xyz="0 0 0"/>
-      <inertial>
-        <mass value="2.0001" />
-        <inertia ixx="1" ixy="0.0" ixz="0.0" iyy="1" iyz="0.0" izz="1"/>
-      </inertial>
-      <collision name='sc3'>
-        <geometry>
-          <box size=".55 .03 .03"/>
-        </geometry>
-      </collision>
-      <visual name='sv3'>
-        <geometry>
-          <box size=".55 .03 .03"/>
-        </geometry>
-        <material name="Red"/>
-      </visual>
-    </link>
-  <joint type="fixed" name="castor_support_joint">
-	  <origin rpy="0 0 0" xyz="0.36 0 -0.255"/>
-      <parent link="base_link"/>
-      <child link="castor_support"/>
-    </joint>
-    <link name="castor_support">
-      <origin rpy="0 0 0" xyz="0 0 0"/>
-      <inertial>
-        <mass value="2.0001" />
-        <inertia ixx="1" ixy="0.0" ixz="0.0" iyy="1" iyz="0.0" izz="1"/>
-      </inertial>
-      <collision name='extrusion_collision'>
-        <geometry>
-          <box size=".2 .1 .02"/>
-        </geometry>
-      </collision>
-      <visual name='extrusion_visual'>
-        <geometry>
-          <box size=".2 .1 .02"/>
-        </geometry>
-        <material name="Blue"/>
-      </visual>
-    </link>
- <joint name="base_caster_support_joint" type="continuous">
+	</eklavya_bar>
+    <castor_support suffix="front" parent="base_link">
+      <origin rpy="0 0 0" xyz="0.36 0 -0.255"/>
+	</castor_support>
+	<caster_support_hinge suffix="front" parent="base_link">
       <origin xyz="0.36 0 -0.275" rpy="0 0 0" />
-      <parent link="base_link" />
-      <child link="base_caster_support_link"/>
-      <axis xyz="0 0 1" />
-      <anchor xyz="0.01 0 0" />
-      <limit effort="100" velocity="100" k_velocity="0" />
-      <joint_properties damping="0.0" friction="0.0" />
-    </joint>
-    <transmission type="pr2_mechanism_model/SimpleTransmission" name="base_caster_support_trans">
-      <actuator name="base_caster_support_motor" />
-      <joint name="base_caster_support_joint" />
-      <mechanicalReduction>1.0</mechanicalReduction>
-    </transmission>
-    <link name="base_caster_support_link">
-      <inertial>
-        <mass value="1"/>
-        <origin xyz="0 0 0" />
-        <inertia ixx="0.00375" ixy="0.0" ixz="0.0"
-          iyy="0.00375" iyz="0.0"
-          izz="0.00375" />
-      </inertial>
-      <visual>
-        <eklavya_castor_support_link_mesh />
-      </visual>
-      <collision>
-        <eklavya_castor_support_link_mesh />
-      </collision>
-    </link>
-<joint name="caster_wheel_joint" type="continuous">
+	</caster_support_hinge>
+    <caster_wheel suffix="front" parent="base_link">
       <origin xyz="-0.0397 0 -0.0918" rpy="0 0 0" />
-      <parent link="base_caster_support_link" />
-      <child link="caster_wheel_link" />
-      <axis xyz="0 1 0" />
-      <anchor xyz="0 0 0" />
-      <limit effort="100" velocity="100" k_velocity="0" />
-      <joint_properties damping="0.0" friction="0.0" />
-    </joint>
-    <transmission type="pr2_mechanism_model/SimpleTransmission" name="caster_wheel_trans">
-      <actuator name="caster_wheel_motor" />
-      <joint name="caster_wheel_joint" />
-      <mechanicalReduction>1.0</mechanicalReduction>
-    </transmission>
-    <link name="caster_wheel_link">
-      <inertial>
-        <mass value="2" />
-        <origin xyz="0 0 0" rpy="0 0 0" />
-        <inertia  ixx="0.003" ixy="0.0" ixz="0.0"
-          iyy="0.00581" iyz="0.0"
-          izz="0.003" />
-      </inertial>
-      <visual>
-        <eklavya_castor_wheel_link_mesh />
-      </visual>
-      <collision>
-        <eklavya_castor_wheel_link_mesh />
-      </collision>
-    </link>
-    <gazebo_castor_wheel_link_surface />
-    <!--
-    <link name="castor">
-   	  <origin rpy="0 0 0" xyz="0 0.375 -0.325"/>
-      <inertial>
-        <mass value="2.0001" />
-        <inertia ixx="1" ixy="0.0" ixz="0.0" iyy="1" iyz="0.0" izz="1"/>
-      </inertial>
-      <collision name='caster_collision'>
-        <geometry>
-          <sphere radius=".05"/>
-        </geometry>
-        <surface>
-          <friction>
-            <ode>
-              <mu>0</mu>
-              <mu2>0</mu2>
-              <slip1>1.0</slip1>
-              <slip2>1.0</slip2>
-            </ode>
-          </friction>
-        </surface>
-      </collision>
-      <visual name='caster_visual'>
-        <geometry>
-          <sphere radius=".05"/>
-        </geometry>
-        <material name="Green"/>
-      </visual>
-    </link>
-     <joint type="fixed" name="castor_joint">
-      <origin rpy="0 0 0" xyz="0 0.375 -0.325"/>
-      <parent link="base_link"/>
-      <child link="castor"/>
-    </joint>
-  -->
+	</caster_wheel>
     <!--Links for sensor integration-->
     <!--IMU link-->
@@ -296,5 +129,4 @@
     </link>
 -->
-    <!--Creating fixed joints for base link supports-->
     <!--Joint for IMU-->
    <!-- <joint name="IMU_sensor_joint" type="fixed">
@@ -318,34 +150,4 @@
     </joint>
 -->
-    <!-- try  try try-->
-  <!--  <joint name="hokuyo_laser_box_joint" type="fixed">
-      <origin xyz="0 0 0" rpy="0 0 0"/>
-      <parent link="LIDAR_sensor_link"/>
-      <child link="hokuyo_laser_box_link"/>
-    </joint>
-    <link name="hokuyo_laser_box_link">
-      <inertial>
-        <mass value="0.01"/>
-        <origin xyz="0 0 0"/>
-        <inertia ixx="0.001" ixy="0.0" ixz="0.0" iyy="0.001" iyz="0.0" izz="0.001"/>
-      </inertial>
-      <visual>
-        <origin xyz="0 0 0" rpy="0 0 0"/>
-        <geometry>-->
-        <!-- box size="0.05 0.05 0.1" / -->
-        <!--<mesh filename="package://meshes/collada/hokuyo_urg.dae" scale="0.5 0.5 0.5"/>
-        </geometry>
-      </visual>
-      <collision>
-        <origin xyz="0 0 0" rpy="0 0 0"/>
-        <geometry>
-          <box size="0.05 0.05 0.1"/>
-        </geometry>
-      </collision>
-    </link>
-    <gazebo reference="hokuyo_laser_box_link">
-      <material>Gazebo/Magenta</material>
-      <turnGravityOff>false</turnGravityOff>
-    </gazebo>-->
     <!--Joint for GPS-->
     <!--

File: eklavya_description/urdf/eklavya_wheel.xacro (robot description, xacro)
@@ -23,11 +23,11 @@
       </inertial>
       <visual>
-        <segbot_wheel_mesh suffix="${suffix}" />
+        <eklavya_wheel_mesh suffix="${suffix}" />
       </visual>
       <collision>
-        <segbot_wheel_mesh suffix="${suffix}" />
+        <eklavya_wheel_mesh suffix="${suffix}" />
       </collision>
     </link>
-    <gazebo_segbot_wheel_surface />
+    <eklavya_segbot_wheel_surface suffix="${suffix}" parent="${parent}" />
     <transmission type="pr2_mechanism_model/SimpleTransmission" name="${parent}_${suffix}_wheel_trans">
       <actuator name="${parent}_${suffix}_wheel_motor" />

File: eklavya_description/urdf/gazebo.urdf.xacro (robot description, xacro)
@@ -19,6 +19,6 @@
     </gazebo>
   </macro>
-  <macro name="gazebo_segbot_castor_wheel_link_surface">
-    <gazebo reference="caster_wheel_link">
+  <macro name="gazebo_eklavya_castor_wheel_link_surface" params="suffix parent">
+    <gazebo reference="${parent}_caster_wheel_${suffix}_link">
       <mu1 value="10.0" />
       <mu2 value="10.0" />
@@ -41,5 +41,5 @@
     </geometry>
   </macro>
-  <macro name="segbot_collision_none">
+  <macro name="eklavya_collision_none">
     <origin xyz="0 0 0" rpy="0 0 0" />
     <geometry>
@@ -53,5 +53,5 @@
     </geometry>
   </macro>
-  <macro name="segbot_wheel_mesh" params="suffix">
+  <macro name="eklavya_wheel_mesh" params="suffix">
     <origin xyz="0 0 0" rpy="0 0 0" />
     <geometry>
@@ -59,5 +59,5 @@
     </geometry>
   </macro>
-  <macro name="gazebo_segbot_wheel_surface">
+  <macro name="eklavya_segbot_wheel_surface" params="suffix parent">
     <gazebo reference="${parent}_${suffix}_wheel_link" >
       <mu1 value="10.0" />

Commit message: updating xacros

File: eklavya_description/urdf/eklavya_body.urdf.xacro (robot description, xacro)
@@ -15,5 +15,5 @@
   <include filename="$(find eklavya_description)/urdf/gazebo.urdf.xacro"/>
   <include filename="$(find eklavya_description)/urdf/materials.urdf.xacro"/>
-  <include filename="$(find eklavya_description)/urdf/eklavya_hardware.xacro.xacro"/>
+  <include filename="$(find eklavya_description)/urdf/eklavya_hardware.xacro"/>
   <include filename="$(find eklavya_description)/urdf/eklavya_wheel.xacro"/>
   <include filename="$(find eklavya_description)/urdf/hokuyo_urg.xacro"/>

File: eklavya_description/urdf/eklavya_hardware.xacro (robot description, xacro)
@@ -65,5 +65,5 @@
     </joint>
     <transmission type="pr2_mechanism_model/SimpleTransmission" name="base_caster_support_trans">
-      <actuator name="base_caster_support_motor" />
+      <actuator name="${parent}_caster_support_hinge_${suffix}_motor" />
       <joint name="${parent}_caster_support_hinge_${suffix}_joint" />
       <mechanicalReduction>1.0</mechanicalReduction>
@@ -86,9 +86,8 @@
 </macro>
 <macro name="caster_wheel" params="suffix parent *origin">
-	<joint type="fixed" name="${parent}_castor_support_${suffix}_joint">
-	  <joint name="caster_wheel_joint" type="continuous">
+	  <joint name="${parent}_caster_wheel_${suffix}_joint" type="continuous">
       <insert_block name="origin" />
       <parent link="${parent}_caster_support_hinge_${suffix}_link" />
-      <child link="caster_wheel_link" />
+      <child link="${parent}_caster_wheel_${suffix}_link" />
       <axis xyz="0 1 0" />
       <anchor xyz="0 0 0" />
@@ -97,9 +96,9 @@
     </joint>
     <transmission type="pr2_mechanism_model/SimpleTransmission" name="caster_wheel_trans">
-      <actuator name="caster_wheel_motor" />
-      <joint name="caster_wheel_joint" />
+      <actuator name="${parent}_caster_wheel_${suffix}_motor" />
+      <joint name="${parent}_caster_wheel_${suffix}_joint" />
       <mechanicalReduction>1.0</mechanicalReduction>
     </transmission>
-    <link name="caster_wheel_link">
+    <link name="${parent}_caster_wheel_${suffix}_link">
       <inertial>
         <mass value="2" />
@@ -116,5 +115,5 @@
       </collision>
     </link>
-    <gazebo_castor_wheel_link_surface />
+    <gazebo_eklavya_castor_wheel_link_surface suffix="${suffix}" parent="${parent}" />
 </macro>
 </robot>
