Commit message: xacrofied

File: eklavya_description/urdf/eklavya_body.urdf.xacro (robot description, xacro)
@@ -70,12 +70,12 @@
       <origin xyz="-0.2 -0.335 -0.303" rpy="0 0 0" />
     </eklavya_wheel>
-	<eklavya_bar suffix="left" parent="base_link">
+	<eklavya_bar suffix="left" parent="base_link" length="0.6">
       <origin rpy="0 0 0" xyz="0.26 0.26 0.575"/>
 	</eklavya_bar>
-	<eklavya_bar suffix="right" parent="base_link">
+	<eklavya_bar suffix="right" parent="base_link" length="0.6">
       <origin rpy="0 0 0" xyz="0.26 -0.26 0.575"/>
 	</eklavya_bar>
-	<eklavya_bar suffix="top" parent="base_link">
-      <origin rpy="0 0  ${M_PI/2}" xyz="0.26 0 0.89"/>
+	<eklavya_bar suffix="top" parent="base_link" length="0.55">
+      <origin rpy="${M_PI/2} 0 0" xyz="0.26 0 0.89"/>
 	</eklavya_bar>
     <castor_support suffix="front" parent="base_link">

File: eklavya_description/urdf/eklavya_hardware.xacro (robot description, xacro)
@@ -4,6 +4,6 @@
   xmlns:controller="http://playerstage.sourceforge.net/gazebo/xmlschema/#controller"
   xmlns:interface="http://playerstage.sourceforge.net/gazebo/xmlschema/#interface">
-  <macro name="eklavya_bar" params="suffix parent *origin">
-	<joint type="fixed" name="${parent}_support_${suffix}joint">
+  <macro name="eklavya_bar" params="suffix parent length *origin">
+	<joint type="fixed" name="${parent}_support_${suffix}_joint">
       <insert_block name="origin" />
       <parent link="${parent}"/>
@@ -13,15 +13,15 @@
       <origin rpy="0 0 0" xyz="0 0 0"/>
       <inertial>
-        <mass value="0.01" />
+        <mass value="2.01" />
         <inertia ixx="1" ixy="0.0" ixz="0.0" iyy="1" iyz="0.0" izz="1"/>
       </inertial>
-      <collision name='sc1'>
+      <collision >
         <geometry>
-          <box size=".03 .03 .6"/>
+          <box size=".03 .03 ${length}"/>
         </geometry>
       </collision>
-      <visual name='sv1'>
-        <geometry>
-          <box size=".03 .03 .6"/>
+      <visual >
+	    <geometry>
+          <box size=".03 .03 ${length}"/>
         </geometry>
         <material name="White"/>
@@ -38,5 +38,5 @@
       <origin rpy="0 0 0" xyz="0 0 0"/>
       <inertial>
-        <mass value="2.0001" />
+        <mass value="0.01" />
         <inertia ixx="1" ixy="0.0" ixz="0.0" iyy="1" iyz="0.0" izz="1"/>
       </inertial>
@@ -102,5 +102,5 @@
     <link name="${parent}_caster_wheel_${suffix}_link">
       <inertial>
-        <mass value="2" />
+        <mass value="1" />
         <origin xyz="0 0 0" rpy="0 0 0" />
         <inertia  ixx="0.003" ixy="0.0" ixz="0.0"

Commit message: 

File: eklavya_description/urdf/eklavya_body.urdf.xacro (robot description, xacro)
@@ -64,13 +64,13 @@
       <origin xyz="-0.2 -0.335 -0.303" rpy="0 0 0" />
     </eklavya_wheel>
-	<eklavya_bar suffix="left" parent="base_link" length="0.6">
+	<eklavya_support_bar suffix="left" parent="base_link" length="0.6">
       <origin rpy="0 0 0" xyz="0.26 0.26 0.575"/>
-	</eklavya_bar>
-	<eklavya_bar suffix="right" parent="base_link" length="0.6">
+	</eklavya_support_bar>
+	<eklavya_support_bar suffix="right" parent="base_link" length="0.6">
       <origin rpy="0 0 0" xyz="0.26 -0.26 0.575"/>
-	</eklavya_bar>
-	<eklavya_bar suffix="top" parent="base_link" length="0.55">
+	</eklavya_support_bar>
+	<eklavya_support_bar suffix="top" parent="base_link" length="0.55">
       <origin rpy="${M_PI/2} 0 0" xyz="0.26 0 0.89"/>
-	</eklavya_bar>
+	</eklavya_support_bar>
     <castor_support suffix="front" parent="base_link">
       <origin rpy="0 0 0" xyz="0.36 0 -0.255"/>
@@ -152,13 +152,14 @@
     </joint> -->
    <!-- <gazebo_eklavya_simple_drive_plugin />    -->
-    <gazebo_eklavya_drive_plugin_diffdrive />
-  <!--  <gazebo_eklavya_p3d_plugin /> -->
-   <!--   <eklavya_segbot_controllers_common />-->
+    <gazebo_eklavya_drive_plugin_diffdrive /><!-- cmd_vel movement -->
+    <gazebo_eklavya_p3d_plugin /> <!-- Ground Truth-->
+    <eklavya_controllers_common />
     <hokuyo_urg name="hokuyo_laser" parent="base_link" >
       <origin rpy="0 0 0" xyz="0.36 0 -0.245"/>
     </hokuyo_urg>
     <!-- Simulation sensors -->
-    <!--<eklavya_sim_imu/>
-      -->
+    <!--<eklavya_sim_imu/> -->
+    <!-- Kinect frames and mounting (includes simulation) -->
+  <turtlebot_kinect/>
   </xacro:macro>
 </robot>

File: eklavya_description/urdf/eklavya_hardware.xacro (robot description, xacro)
@@ -4,11 +4,11 @@
   xmlns:controller="http://playerstage.sourceforge.net/gazebo/xmlschema/#controller"
   xmlns:interface="http://playerstage.sourceforge.net/gazebo/xmlschema/#interface">
-  <macro name="eklavya_bar" params="suffix parent length *origin">
-	<joint type="fixed" name="${parent}_support_${suffix}_joint">
+  <macro name="eklavya_support_bar" params="suffix parent length *origin">
+	<joint type="fixed" name="${parent}_support_bar_${suffix}_joint">
       <insert_block name="origin" />
       <parent link="${parent}"/>
-      <child link="${parent}_support_${suffix}"/>
+      <child link="${parent}_support_bar_${suffix}"/>
     </joint>
-    <link name="${parent}_support_${suffix}">
+    <link name="${parent}_support_bar_${suffix}">
       <origin rpy="0 0 0" xyz="0 0 0"/>
       <inertial>

File: eklavya_description/urdf/eklavya_wheel.xacro (robot description, xacro)
@@ -29,5 +29,5 @@
       </collision>
     </link>
-    <eklavya_segbot_wheel_surface suffix="${suffix}" parent="${parent}" />
+    <eklavya_wheel_surface suffix="${suffix}" parent="${parent}" />
     <transmission type="pr2_mechanism_model/SimpleTransmission" name="${parent}_${suffix}_wheel_trans">
       <actuator name="${parent}_${suffix}_wheel_motor" />

File: eklavya_description/urdf/gazebo.urdf.xacro (robot description, xacro)
@@ -4,11 +4,4 @@
   xmlns:controller="http://playerstage.sourceforge.net/gazebo/xmlschema/#controller"
   xmlns:interface="http://playerstage.sourceforge.net/gazebo/xmlschema/#interface">
-<gazebo reference="castor">
-    <mu1 value="0"/>
-    <mu2 value="0"/>
-    <kp value="100000000.0"/>
-    <kd value="10000.0"/>
-    <fdir value="1 0 0"/>
-  </gazebo>
   <macro name="gazebo_eklavya_base_link_surface">
     <gazebo reference="base_link">
@@ -59,5 +52,5 @@
     </geometry>
   </macro>
-  <macro name="eklavya_segbot_wheel_surface" params="suffix parent">
+  <macro name="eklavya_wheel_surface" params="suffix parent">
     <gazebo reference="${parent}_${suffix}_wheel_link" >
       <mu1 value="10.0" />
@@ -65,12 +58,12 @@
       <kp  value="1000000.0" />
       <kd  value="1.0" />
+       <fdir value="1 0 0"/>
     </gazebo>
   </macro>
  <!-- CONTROLLERS -->
-        <!-- this publishes empty joint_states due to no transmission, but
+  <macro name="eklavya_controllers_common">
+ <!-- this publishes empty joint_states due to no transmission, but
              triggering robot_state_publisher to publish tf between fixed joints in eklavya,
              (e.g. base_laser_link for the base_scan frame) -->
- <!--
-  <macro name="eklavya_segbot_controllers_common">
     <controller:gazebo_ros_controller_manager name="gazebo_ros_controller_manager" plugin="libgazebo_ros_controller_manager.so">
       <alwaysOn>true</alwaysOn>
@@ -80,6 +73,5 @@
     <canonicalBody>base_footprint</canonicalBody>
   </macro>
-  -->
-  <macro name="eklavya_segbot_drive_parameters">
+  <macro name="eklavya_drive_parameters">
     <alwaysOn>true</alwaysOn>
     <update>100</update>
@@ -95,17 +87,17 @@
   <macro name="gazebo_eklavya_simple_drive_plugin">
 	  <gazebo>
-    <controller:segbotsimpledrive_plugin name="differential_drive_controller" plugin="libeklavya_simple_drive_plugin.so">
-      <eklavya_segbot_drive_parameters />
-    </controller:segbotsimpledrive_plugin>
+    <controller:eklavya_simple_drive_plugin name="differential_drive_controller" plugin="libeklavya_simple_drive_plugin.so">
+      <eklavya_drive_parameters />
+    </controller:eklavya_simple_drive_plugin>
      </gazebo>
   </macro>
   <macro name="gazebo_eklavya_drive_plugin">
 	<gazebo>
-    <controller:segbotdrive_plugin name="differential_drive_controller" plugin="libeklavya_drive_plugin.so">
-      <eklavya_segbot_drive_parameters />
-    </controller:segbotdrive_plugin>
+    <controller:eklavya_drive_plugin name="differential_drive_controller" plugin="libeklavya_drive_plugin.so">
+      <eklavya_drive_parameters />
+    </controller:eklavya_drive_plugin>
      </gazebo>
    </macro>
- <macro name="gazebo_eklavya_drive_plugin_diffdrive">
+	<macro name="gazebo_eklavya_drive_plugin_diffdrive">
         <gazebo>
             <controller:diffdrive_plugin name="differential_drive_controller" plugin="libdiffdrive_plugin.so">
@@ -124,6 +116,5 @@
          </gazebo>
     </macro>
-    <!--
-<macro name="gazebo_eklavya_p3d_plugin">
+	<macro name="gazebo_eklavya_p3d_plugin">
 		 <gazebo>
             <controller:gazebo_ros_p3d name="p3d_base_controller" plugin="libgazebo_ros_p3d.so">
@@ -139,4 +130,4 @@
             </controller:gazebo_ros_p3d>
         </gazebo>
-  </macro>  -->
+  </macro>
 </robot>

Commit message: sensors working

File: eklavya_description/urdf/eklavya_body.urdf.xacro (robot description, xacro)
@@ -12,4 +12,6 @@
   <include filename="$(find eklavya_description)/urdf/eklavya_wheel.xacro"/>
   <include filename="$(find eklavya_description)/urdf/hokuyo_urg.xacro"/>
+  <include filename="$(find eklavya_description)/urdf/microstrain_3dmgx3_imu.urdf.xacro"/>
+  <include filename="$(find eklavya_description)/urdf/eklavya_kinect.urdf.xacro"/>
   <xacro:macro name="eklavya_body">
     <!--Dummy base without INERTIA because base_link is not supposed to have inertia-->
@@ -82,84 +84,18 @@
       <origin xyz="-0.0397 0 -0.0918" rpy="0 0 0" />
 	</caster_wheel>
-    <!--Links for sensor integration-->
-    <!--IMU link-->
-   <!-- <link name="IMU_sensor_link">
-      <inertial>
-        <mass value="0.01" />
-        <origin xyz="0 0 0"/>
-        <inertia ixx="0.001" ixy="0.0" ixz="0.0"
-                  iyy="0.001" iyz="0.0" izz="0.001" />
-      </inertial>
-    </link>
--->
-    <!--BumbleBee link-->
-   <!-- <link name="BumbleBee_sensor_link">
-      <inertial>
-        <mass value="0.01" />
-        <origin xyz="0 0 0"/>
-        <inertia ixx="0.001" ixy="0.0" ixz="0.0"
-                 iyy="0.001" iyz="0.0" izz="0.001" />
-      </inertial>
-    </link>
- -->
-    <!--LIDAR link-->
-    <!--<link name="LIDAR_sensor_link">
-      <inertial>
-        <mass value="0.01" />
-        <origin xyz="0 0 0"/>
-        <inertia ixx="0.001" ixy="0.0" ixz="0.0"
-                 iyy="0.001" iyz="0.0" izz="0.001" />
-      </inertial>
-    </link>
--->
-    <!--GPS link-->
-   <!-- <link name="GPS_sensor_link">
-      <inertial>
-        <mass value="0.01" />
-        <origin xyz="0 0 0"/>
-        <inertia ixx="0.001" ixy="0.0" ixz="0.0"
-                 iyy="0.001" iyz="0.0" izz="0.001" />
-      </inertial>
-    </link>
--->
-    <!--Joint for IMU-->
-   <!-- <joint name="IMU_sensor_joint" type="fixed">
-      <origin xyz="0.26 0.26 0.275" rpy="0 0 -1.0" />
-      <parent link="base_link"/>
-      <child link="IMU_sensor_link" />
-    </joint>
--->
-    <!--Joint for BumbleBee Sterio Camera-->
-   <!-- <joint name="BumbleBee_sensor_joint" type="fixed">
-      <origin rpy="0 0 0" xyz="0 0.26 0.89"/>
-      <parent link="base_link"/>
-      <child link="BumbleBee_sensor_link" />
-    </joint>
--->
-    <!--Joint for LIDAR-->
-   <!-- <joint name="LIDAR_sensor_joint" type="fixed">
-      <origin xyz="0 0.375 -0.3" rpy="0 0 -1.0" />
-      <parent link="base_link"/>
-      <child link="LIDAR_sensor_link" />
-    </joint>
--->
-    <!--Joint for GPS-->
-    <!--
-    <joint name="GPS_sensor_joint" type="fixed">
-      <origin xyz="-0.26 0.26 0.275" rpy="0 0 -1.0" />
-      <parent link="base_link"/>
-      <child link="GPS_sensor_link" />
-    </joint> -->
+	<!-- Controllers -->
    <!-- <gazebo_eklavya_simple_drive_plugin />    -->
     <gazebo_eklavya_drive_plugin_diffdrive /><!-- cmd_vel movement -->
     <gazebo_eklavya_p3d_plugin /> <!-- Ground Truth-->
-    <eklavya_controllers_common />
-    <hokuyo_urg name="hokuyo_laser" parent="base_link" >
+     <eklavya_controllers_common />
+    <!-- Simulation sensors -->
+	<hokuyo_urg name="hokuyo_laser" parent="base_link" >
       <origin rpy="0 0 0" xyz="0.36 0 -0.245"/>
     </hokuyo_urg>
-    <!-- Simulation sensors -->
-    <!--<eklavya_sim_imu/> -->
+	<microstrain_imu name="eklavya_sim_imu" parent="base_link" imu_topic="imu/data" update_rate="30" stdevNoise="0.0017">
+		<origin rpy="0 0 0" xyz="0.26 0.20 0.575"/>
+	</microstrain_imu>
     <!-- Kinect frames and mounting (includes simulation) -->
-  <turtlebot_kinect/>
+   <eklavya_kinect/>
   </xacro:macro>
 </robot>

File: eklavya_description/urdf/eklavya_calibration.xacro (robot description, xacro)
@@ -1,10 +1,10 @@
 <?xml version="1.0"?>
 <robot>
-  <property name="eklavya_calib_cam_x" value="-0.0844382" />
-  <property name="eklavya_calib_cam_y" value="0" />
-  <property name="eklavya_calib_cam_z" value="0.1047496" />
+  <property name="eklavya_calib_cam_x" value="${-0.0844382+0.36}" />
+  <property name="eklavya_calib_cam_y" value="${0+ 0}" />
+  <property name="eklavya_calib_cam_z" value="${0.1047496+0.22}" />
   <property name="eklavya_calib_cam_rr" value="0" />
   <property name="eklavya_calib_cam_rp" value="0" />
   <property name="eklavya_calib_cam_ry" value="0" />
-  <property name="eklavya_camera_parent_name" value="base_link_support_bar_top" />
+  <property name="eklavya_camera_parent_name" value="base_link" />
 </robot>

File: eklavya_description/urdf/eklavya_kinect.urdf.xacro (robot description, xacro)
@@ -1,8 +1,37 @@
 <?xml version="1.0"?>
-<robot name="eklavya_hardware" xmlns:xacro="http://ros.org/wiki/xacro">
+<robot name="eklavya_hardware" xmlns:xacro="http://ros.org/wiki/xacro"
+		xmlns:sensor="http://playerstage.sourceforge.net/gazebo/xmlschema/#sensor"
+       xmlns:controller="http://playerstage.sourceforge.net/gazebo/xmlschema/#controller"
+       xmlns:interface="http://playerstage.sourceforge.net/gazebo/xmlschema/#interface">
   <property name="M_PI" value="3.14159"/>
   <include filename="$(find eklavya_description)/urdf/gazebo.urdf.xacro"/>
   <include filename="$(find eklavya_description)/urdf/eklavya_calibration.xacro" />
-<xacro:macro name="eklavya_kinect">
+<xacro:macro name="eklavya_sim_kinect">
+  <gazebo reference="camera_link">
+    <sensor:camera name="camera">
+      <imageFormat>R8G8B8</imageFormat>
+      <imageSize>640 480</imageSize>
+      <hfov>60</hfov>
+      <nearClip>0.05</nearClip>
+      <farClip>3</farClip>
+      <updateRate>20</updateRate>
+      <baseline>0.1</baseline>
+      <controller:gazebo_ros_openni_kinect name="kinect_camera_controller" plugin="libgazebo_ros_openni_kinect.so">
+        <alwaysOn>true</alwaysOn>
+        <updateRate>20</updateRate>
+        <imageTopicName>/camera/image_raw</imageTopicName>
+        <pointCloudTopicName>/camera/depth/points</pointCloudTopicName>
+        <cameraInfoTopicName>/camera/camera_info</cameraInfoTopicName>
+        <frameName>camera_depth_optical_frame</frameName>
+        <distortion_k1>0.0</distortion_k1>
+        <distortion_k2>0.0</distortion_k2>
+        <distortion_k3>0.0</distortion_k3>
+        <distortion_t1>0.0</distortion_t1>
+        <distortion_t2>0.0</distortion_t2>
+      </controller:gazebo_ros_openni_kinect>
+    </sensor:camera>
+  </gazebo>
+</xacro:macro>
+<xacro:macro name="eklavya_kinect" >
   <joint name="base_camera_joint" type="fixed">
     <origin xyz="${eklavya_calib_cam_x} ${eklavya_calib_cam_y} ${eklavya_calib_cam_z}"

File: eklavya_description/urdf/microstrain_3dmgx3_imu.urdf.xacro (robot description, xacro)
@@ -1,6 +1,22 @@
 <?xml version="1.0"?>
-<robot xmlns:xacro="http://ros.org/wiki/xacro">
-  <include filename="$(find wubble_description)/urdf/microstrain_3dmgx3_imu.gazebo.xacro" />
-  <xacro:macro name="microstrain_3dmgx3_imu_v0" params="name parent *origin imu_topic update_rate stdev">
+<robot xmlns:xacro="http://ros.org/wiki/xacro"
+       xmlns:sensor="http://playerstage.sourceforge.net/gazebo/xmlschema/#sensor"
+       xmlns:controller="http://playerstage.sourceforge.net/gazebo/xmlschema/#controller"
+       xmlns:interface="http://playerstage.sourceforge.net/gazebo/xmlschema/#interface">
+   <xacro:macro name="microstrain_imu_gazebo" params="name imu_topic update_rate stdevNoise">
+    <gazebo>
+      <controller:gazebo_ros_imu name="imu_controller" plugin="libgazebo_ros_imu.so">
+        <alwaysOn>true</alwaysOn>
+        <updateRate>${update_rate}</updateRate>
+        <bodyName>${name}_link</bodyName>
+        <topicName>${imu_topic}</topicName>
+        <gaussianNoise>${stdevNoise*stdevNoise}</gaussianNoise>
+        <xyzOffsets>0 0 0</xyzOffsets>
+        <rpyOffsets>0 0 0</rpyOffsets>
+        <interface:position name="imu_position"/>
+      </controller:gazebo_ros_imu>
+    </gazebo>
+  </xacro:macro>
+  <xacro:macro name="microstrain_imu" params="name parent *origin imu_topic update_rate stdevNoise">
     <joint name="${name}_joint" type="fixed">
       <axis xyz="0 1 0" />
@@ -17,5 +33,5 @@
     </link>
     <!-- gazebo extensions -->
-    <xacro:microstrain_3dmgx2_imu_gazebo_v0 name="${name}" imu_topic="${imu_topic}" update_rate="${update_rate}" stdev="${stdev}" />
+    <xacro:microstrain_imu_gazebo name="${name}" imu_topic="${imu_topic}" update_rate="${update_rate}" stdevNoise="${stdevNoise}" />
   </xacro:macro>
 </robot>

Commit message: testing sick lidar simulation.. rviz body hav to be fixed

File: eklavya_description/urdf/eklavya_body.urdf.xacro (robot description, xacro)
@@ -11,5 +11,6 @@
   <include filename="$(find eklavya_description)/urdf/eklavya_hardware.xacro"/>
   <include filename="$(find eklavya_description)/urdf/eklavya_wheel.xacro"/>
-  <include filename="$(find eklavya_description)/urdf/hokuyo_urg.xacro"/>
+  <!--  <include filename="$(find eklavya_description)/urdf/hokuyo_urg.xacro"/>-->
+ <include filename="$(find eklavya_description)/urdf/sick_lms100_200.urdf.xacro"/>
   <include filename="$(find eklavya_description)/urdf/microstrain_3dmgx3_imu.urdf.xacro"/>
   <include filename="$(find eklavya_description)/urdf/eklavya_kinect.urdf.xacro"/>
@@ -18,12 +19,18 @@
     <link name="base_footprint">
       <visual>
-        <origin xyz="0 0 0" rpy="0 0 0" />
+        <origin xyz="0 0 0.0" rpy="0 0 0" />
         <geometry>
           <box size="0.001 0.001 0.001" />
         </geometry>
       </visual>
+      <collision>
+		<origin xyz="0 0 0.817" rpy="0 0 0" />
+	      <geometry>
+			<box size="0.001 0.001 0.001" />
+	      </geometry>
+		</collision>
     </link>
     <joint name="base_footprint_joint" type="fixed">
-      <origin xyz="0.0 0 0.5" rpy="0 0 0" />
+      <origin xyz="0.0 0 0.97" rpy="0 0 0" />
       <parent link="base_footprint"/>
       <child link="base_link" />
@@ -91,5 +98,6 @@
     <!-- Simulation sensors -->
 	<hokuyo_urg name="hokuyo_laser" parent="base_link" >
-      <origin rpy="0 0 0" xyz="0.36 0 -0.245"/>
+      <origin rpy="0 0 0" xyz="0.36 0 -0.190"/>
+       <!--<origin rpy="0 0 0" xyz="0.36 0 -0.245"/>-->
     </hokuyo_urg>
 	<microstrain_imu name="eklavya_sim_imu" parent="base_link" imu_topic="imu/data" update_rate="30" stdevNoise="0.0017">

File: eklavya_description/urdf/eklavya_hardware.xacro (robot description, xacro)
@@ -51,5 +51,5 @@
           <box size=".2 .1 .02"/>
         </geometry>
-        <material name="Blue"/>
+        <material name="GunMetalBrushedAluminum"/>
       </visual>
     </link>

File: eklavya_description/urdf/gazebo.urdf.xacro (robot description, xacro)
@@ -21,5 +21,5 @@
   </macro>
   <macro name="eklavya_base_link_mesh">
-    <origin xyz="0 0 0" rpy="0 0 0" />
+    <origin xyz="0 0 0.0308" rpy="0 0 0" />
     <geometry>
      <!-- <mesh filename="package://eklavya_description/meshes/rmp50-base-link.dae" scale="0.0254 0.0254 0.0254"/> -->
@@ -121,5 +121,5 @@
                 <alwaysOn>true</alwaysOn>
                 <updateRate>100.0</updateRate>
-                <bodyName>base_link</bodyName>
+                <bodyName>base_footprint</bodyName>
                 <topicName>base_pose_ground_truth</topicName>
                 <gaussianNoise>0.01</gaussianNoise>

File: eklavya_description/urdf/materials.urdf.xacro (robot description, xacro)
@@ -23,5 +23,5 @@
     </material>
     <material name="GunMetalBrushedAluminum">
-        <texture filename="package://eklavya_gazebo/textures/gun_metal_brushed_aluminum.jpg" />
+        <texture filename="package://eklavya_gazebo/Media/materials/textures/gun_metal_brushed_aluminum.jpg" />
     </material>
 </robot>

Commit message: test model change

File: eklavya_description/urdf/eklavya_body.urdf.xacro (robot description, xacro)
@@ -97,8 +97,10 @@
      <eklavya_controllers_common />
     <!-- Simulation sensors -->
-	<hokuyo_urg name="hokuyo_laser" parent="base_link" >
-      <origin rpy="0 0 0" xyz="0.36 0 -0.190"/>
-       <!--<origin rpy="0 0 0" xyz="0.36 0 -0.245"/>-->
-    </hokuyo_urg>
+	<!--<hokuyo_urg name="hokuyo_laser" parent="base_link" >
+       <origin rpy="0 0 0" xyz="0.36 0 -0.245"/>
+    </hokuyo_urg> -->
+    <sick_lms100_200 name="sick_laser" parent="base_link" >
+      <origin rpy="0 0 0" xyz="0.39 0 -0.185"/>
+    </sick_lms100_200>
 	<microstrain_imu name="eklavya_sim_imu" parent="base_link" imu_topic="imu/data" update_rate="30" stdevNoise="0.0017">
 		<origin rpy="0 0 0" xyz="0.26 0.20 0.575"/>

File: eklavya_description/urdf/sick_lms100_200.urdf.xacro (robot description, xacro)
@@ -8,5 +8,5 @@
   <property name="laser_mass" value="1.1" />
   <include filename="$(find eklavya_description)/urdf/common.xacro"/>
-    <macro name="hokuyo_urg" params="name parent *origin" >
+    <macro name="sick_lms100_200" params="name parent *origin" >
         <joint name="${name}_mount_joint" type="fixed">
             <insert_block name="origin" />
