Commit message: wheeks and color

File: eklavya_description/urdf/eklavya_body.urdf.xacro (robot description, xacro)
@@ -11,5 +11,5 @@
   <include filename="$(find eklavya_description)/urdf/eklavya_hardware.xacro"/>
   <include filename="$(find eklavya_description)/urdf/eklavya_wheel.xacro"/>
-  <!--  <include filename="$(find eklavya_description)/urdf/hokuyo_urg.xacro"/>-->
+  <include filename="$(find eklavya_description)/urdf/hokuyo_urg.xacro"/>
  <include filename="$(find eklavya_description)/urdf/sick_lms100_200.urdf.xacro"/>
   <include filename="$(find eklavya_description)/urdf/microstrain_3dmgx3_imu.urdf.xacro"/>
@@ -67,10 +67,23 @@
       </inertial>
     </link>
+	 <!-- WHEEL macros -->
     <eklavya_wheel suffix="left" parent="base_link">
-      <origin xyz="-0.2 0.335 -0.303" rpy="0 0 0" />
+      <origin xyz="${ -1*base_x_origin_to_wheel_origin} ${base_y_origin_to_wheel_origin} ${ -1*base_z_origin_to_wheel_origin}" rpy="0 0 0" />
     </eklavya_wheel>
     <eklavya_wheel suffix="right" parent="base_link">
-      <origin xyz="-0.2 -0.335 -0.303" rpy="0 0 0" />
+      <origin xyz="${ -1*base_x_origin_to_wheel_origin} ${-1*base_y_origin_to_wheel_origin} ${ -1*base_z_origin_to_wheel_origin}" rpy="0 0 0" />
     </eklavya_wheel>
+    <!-- Castor -->
+    <castor_support suffix="front" parent="base_link">
+      <origin rpy="0 0 0" xyz="0.36 0 -0.255"/>
+	</castor_support>
+	<caster_support_hinge suffix="front" parent="base_link">
+      <origin xyz="0.36 0 -0.275" rpy="0 0 0" />
+	</caster_support_hinge>
+    <caster_wheel suffix="front" parent="base_link">
+      <origin xyz="-0.0397 0 -0.0918" rpy="0 0 0" />
+	</caster_wheel>
+     <!-- DECORATIONS -->
+     <!-- Bars -->
 	<eklavya_support_bar suffix="left" parent="base_link" length="0.6">
       <origin rpy="0 0 0" xyz="0.26 0.26 0.575"/>
@@ -82,13 +95,4 @@
       <origin rpy="${M_PI/2} 0 0" xyz="0.26 0 0.89"/>
 	</eklavya_support_bar>
-    <castor_support suffix="front" parent="base_link">
-      <origin rpy="0 0 0" xyz="0.36 0 -0.255"/>
-	</castor_support>
-	<caster_support_hinge suffix="front" parent="base_link">
-      <origin xyz="0.36 0 -0.275" rpy="0 0 0" />
-	</caster_support_hinge>
-    <caster_wheel suffix="front" parent="base_link">
-      <origin xyz="-0.0397 0 -0.0918" rpy="0 0 0" />
-	</caster_wheel>
 	<!-- Controllers -->
    <!-- <gazebo_eklavya_simple_drive_plugin />    -->
@@ -97,10 +101,10 @@
      <eklavya_controllers_common />
     <!-- Simulation sensors -->
-	<!--<hokuyo_urg name="hokuyo_laser" parent="base_link" >
+	<hokuyo_urg name="hokuyo_laser" parent="base_link" >
        <origin rpy="0 0 0" xyz="0.36 0 -0.245"/>
-    </hokuyo_urg> -->
-    <sick_lms100_200 name="sick_laser" parent="base_link" >
+    </hokuyo_urg>
+   <!-- <sick_lms100_200 name="sick_laser" parent="base_link" >
       <origin rpy="0 0 0" xyz="0.39 0 -0.185"/>
-    </sick_lms100_200>
+    </sick_lms100_200> -->
 	<microstrain_imu name="eklavya_sim_imu" parent="base_link" imu_topic="imu/data" update_rate="30" stdevNoise="0.0017">
 		<origin rpy="0 0 0" xyz="0.26 0.20 0.575"/>

File: eklavya_description/urdf/eklavya_wheel.xacro (robot description, xacro)
@@ -4,4 +4,21 @@
   xmlns:controller="http://playerstage.sourceforge.net/gazebo/xmlschema/#controller"
   xmlns:interface="http://playerstage.sourceforge.net/gazebo/xmlschema/#interface">
+    <property name="wheel_x_com" value="0.00000000" /> <!-- com : center of mass -->
+	<property name="wheel_y_com" value="0.00000000" /> <!-- com : center of mass -->
+	<property name="wheel_z_com" value="0.00019000" /> <!-- com : center of mass -->
+	<property name="wheel_x_size" value="0.35550000" />
+	<property name="wheel_y_size" value="0.35550000" />
+	<property name="wheel_z_size" value="0.11430000" />
+	<property name="wheel_mass" value="2.63657000" /> <!-- in kg-->
+	<property name="wheel_ixx_com_cs" value="0.02466885" /> <!-- at center of mass aligned with coordinate system, kg*m^2-->
+	<property name="wheel_ixy_com_cs" value="0.00000000" /> <!-- at center of mass aligned with coordinate system, kg*m^2-->
+	<property name="wheel_ixz_com_cs" value="0.00000000" /> <!-- at center of mass aligned with coordinate system, kg*m^2-->
+	<property name="wheel_iyy_com_cs" value="0.02466885" /> <!-- at center of mass aligned with coordinate system, kg*m^2-->
+	<property name="wheel_iyz_com_cs" value="0.00000000" /> <!-- at center of mass aligned with coordinate system, kg*m^2-->
+	<property name="wheel_izz_com_cs" value="0.04410576" /> <!-- at center of mass aligned with coordinate system, kg*m^2-->
+	<property name="base_x_origin_to_wheel_origin" value="0.2" />
+	<property name="base_y_origin_to_wheel_origin" value="0.355" />
+	<property name="base_z_origin_to_wheel_origin" value="0.303" />
+	<property name="base_z_origin_offset" value="0.00317500" /> <!-- origin is offset in + z direction by 3.175mm, so need to bring it back down for visual and collision-->
   <macro name="eklavya_wheel" params="suffix parent *origin">
     <joint name="${parent}_${suffix}_wheel_joint" type="continuous">
@@ -16,12 +33,12 @@
     <link name="${parent}_${suffix}_wheel_link">
       <inertial>
-        <mass value="5" />
-        <origin xyz=" 0 0 0 " />
-        <inertia  ixx="0.076" ixy="0.0" ixz="0.0"
-          iyy="0.144" iyz="0.0"
-          izz="0.076" />
-      </inertial>
+			<mass value="${wheel_mass}" />
+			<origin xyz="${wheel_x_com} ${wheel_y_com} ${wheel_z_com}" />
+			<inertia  ixx="${wheel_ixx_com_cs}" ixy="${wheel_ixy_com_cs}" ixz="${wheel_ixz_com_cs}"
+				iyy="${wheel_iyy_com_cs}" iyz="${wheel_iyz_com_cs}" izz="${wheel_izz_com_cs}" />
+		</inertial>
       <visual>
         <eklavya_wheel_mesh suffix="${suffix}" />
+		<!--<material name="DarkGray" />-->
       </visual>
       <collision>
@@ -30,8 +47,10 @@
     </link>
     <eklavya_wheel_surface suffix="${suffix}" parent="${parent}" />
+    <!-- Transmission is important to link the joints and the controller -->
     <transmission type="pr2_mechanism_model/SimpleTransmission" name="${parent}_${suffix}_wheel_trans">
       <actuator name="${parent}_${suffix}_wheel_motor" />
       <joint name="${parent}_${suffix}_wheel_joint" />
       <mechanicalReduction>1.0</mechanicalReduction>
+      <motorTorqueConstant>1</motorTorqueConstant>
     </transmission>
   </macro>

File: eklavya_description/urdf/gazebo.urdf.xacro (robot description, xacro)
@@ -10,4 +10,6 @@
       <kp  value="1000000.0" />
       <kd  value="1.0" />
+      <!--material name="Eklavya/GunMetalBrushedAluminum   Gazebo/Blue" />-->
+    <material>Eklavya/GunMetalBrushedAluminum</material>
     </gazebo>
   </macro>
@@ -21,5 +23,5 @@
   </macro>
   <macro name="eklavya_base_link_mesh">
-    <origin xyz="0 0 0.0308" rpy="0 0 0" />
+    <origin xyz="0 0 0" rpy="0 0 0" />
     <geometry>
      <!-- <mesh filename="package://eklavya_description/meshes/rmp50-base-link.dae" scale="0.0254 0.0254 0.0254"/> -->
@@ -49,14 +51,18 @@
     <origin xyz="0 0 0" rpy="0 0 0" />
     <geometry>
-      <mesh filename="package://eklavya_description/meshes/rmp50-${suffix}-wheel.dae" scale="0.0150 0.0150 0.0150"/>
+     <!-- <mesh filename="package://eklavya_description/meshes/rmp50-${suffix}-wheel.dae" scale="0.0150 0.0150 0.0150"/>-->
+      <mesh filename="package://eklavya_description/meshes/wheel.stl" />
     </geometry>
+    <material name="DarkGray" />
   </macro>
   <macro name="eklavya_wheel_surface" params="suffix parent">
     <gazebo reference="${parent}_${suffix}_wheel_link" >
-      <mu1 value="10.0" />
-      <mu2 value="10.0" />
-      <kp  value="1000000.0" />
-      <kd  value="1.0" />
-       <fdir value="1 0 0"/>
+		<mu1 value="75.0"/>
+		<mu2 value="1.5"/>
+		<kp  value="1000000.0" />
+		<kd  value="1.0" />
+		<fdir value="1 0 0"/>
+		<material>Gazebo/Grey</material>
+		<turnGravityOff>false</turnGravityOff>
     </gazebo>
   </macro>
@@ -121,5 +127,5 @@
                 <alwaysOn>true</alwaysOn>
                 <updateRate>100.0</updateRate>
-                <bodyName>base_footprint</bodyName>
+                <bodyName>base_link</bodyName>
                 <topicName>base_pose_ground_truth</topicName>
                 <gaussianNoise>0.01</gaussianNoise>

File: eklavya_description/urdf/materials.urdf.xacro (robot description, xacro)
@@ -22,4 +22,7 @@
         <color rgba="1.0 1.0 1.0 1.0"/>
     </material>
+	<material name="DarkGray">
+		<color rgba="0.3 0.3 0.3 1.0"/>
+	</material>
     <material name="GunMetalBrushedAluminum">
         <texture filename="package://eklavya_gazebo/Media/materials/textures/gun_metal_brushed_aluminum.jpg" />
