Commit message: model fixed+ more todo.. vibrating

File: eklavya_description/urdf/eklavya_body.urdf.xacro (robot description, xacro)
@@ -1,9 +1,25 @@
 <?xml version="1.0"?>
 <robot name="eklavya_hardware" xmlns:xacro="http://ros.org/wiki/xacro">
-<!-- Properties (Constants) -->
-    <property name="M_PI" value="3.14159"/>
-    <property name="wheel_radius" value="0.0711" />
-    <property name="wheel_length" value="0.1423" />
-    <property name="caster_wheel_offset_y" value="-0.56" />
+    <!-- PROPERTY LIST -->
+    <!--All units in m-kg-s-radians unit system -->
+    <property name="M_PI" value="3.1415926535897931" />
+    <!-- Main Body-base-->
+    <!-- Location of com : center of mass -->
+    <property name="base_x_com" value="-0.04748000" />
+    <property name="base_y_com" value="-0.00000000" />
+    <property name="base_z_com" value="0.09947000" />
+    <!-- Size of the base-->
+    <property name="base_x_size" value="0.55000000" />
+    <property name="base_y_size" value="0.55000000" />
+    <property name="base_z_size" value="0.55000000" />
+    <!--Weight of the base-->
+    <property name="base_mass" value="33.45489000" /> <!-- in kg-->
+    <!--Inertial values for the base at center of mass, aligned with coordinate system. Units are kg*m^2-->
+    <property name="base_ixx_com_cs" value="0.60216370" />
+    <property name="base_ixy_com_cs" value="-0.02364198" />
+    <property name="base_ixz_com_cs" value="-0.11972132" />
+    <property name="base_iyy_com_cs" value="1.73859574" />
+    <property name="base_iyz_com_cs" value="-0.00154437" />
+    <property name="base_izz_com_cs" value="2.02955229" />
   <!-- Macro for eklavya body. Including Gazebo extensions, but does not include Kinect -->
   <include filename="$(find eklavya_description)/urdf/gazebo.urdf.xacro"/>
@@ -12,9 +28,11 @@
   <include filename="$(find eklavya_description)/urdf/eklavya_wheel.xacro"/>
   <include filename="$(find eklavya_description)/urdf/hokuyo_urg.xacro"/>
- <include filename="$(find eklavya_description)/urdf/sick_lms100_200.urdf.xacro"/>
+  <include filename="$(find eklavya_description)/urdf/sick_lms100_200.urdf.xacro"/>
   <include filename="$(find eklavya_description)/urdf/microstrain_3dmgx3_imu.urdf.xacro"/>
   <include filename="$(find eklavya_description)/urdf/eklavya_kinect.urdf.xacro"/>
   <xacro:macro name="eklavya_body">
     <!--Dummy base without INERTIA because base_link is not supposed to have inertia-->
+    <!-- BASE-FOOTPRINT -->
+    <!-- base_footprint is a fictitious link(frame) that is on the ground right below base_link origin, navigation stack depends on this frame -->
     <link name="base_footprint">
       <visual>
@@ -24,47 +42,54 @@
         </geometry>
       </visual>
-      <collision>
-		<origin xyz="0 0 0.817" rpy="0 0 0" />
-	      <geometry>
-			<box size="0.001 0.001 0.001" />
-	      </geometry>
-		</collision>
+      <inertial>
+            <mass value="0.0001" />
+            <origin xyz="0 0 0" />
+            <inertia ixx="0.0001" ixy="0.0" ixz="0.0"
+                iyy="0.0001" iyz="0.0"
+                izz="0.0001" />
+        </inertial>
+	<!--  <collision>
+          <origin xyz="0 0 0.0" rpy="0 0 0" />
+          <geometry>
+            <box size="0.001 0.001 0.001" />
+         </geometry>
+      </collision>-->
     </link>
+    <gazebo reference="base_footprint">
+        <material>Gazebo/Green</material>
+        <turnGravityOff>false</turnGravityOff>
+    </gazebo>
     <joint name="base_footprint_joint" type="fixed">
-      <origin xyz="0.0 0 0.97" rpy="0 0 0" />
+      <!-- <origin xyz="0.0 0 0.97" rpy="0 0 0" />-->
+      <origin xyz="0 0 ${wheel_x_size/2 - base_z_origin_to_wheel_origin}" rpy="0 0 0" />
       <parent link="base_footprint"/>
       <child link="base_link" />
     </joint>
-    <!-- Links and Joints (i.e., the robot) -->
+    <!-- BASE-LINK -->
+    <!--Actual body/chassis of the robot-->
     <link name="base_link">
-      <inertial>
-        <mass value="0.01" />
-        <origin xyz="0 0 0" />
-        <inertia ixx="1.0" ixy="0.0" ixz="0.0"
-          iyy="1.0" iyz="0.0"
-          izz="1.0" />
-      </inertial>
+	 <inertial>
+		<mass value="${base_mass}" />
+		<!--This is the pose of the inertial reference frame, relative to the link reference frame. The origin of the inertial reference frame needs to be at the center of gravity. The axes of the inertial reference frame do not need to be aligned with the principal axes of the inertia.-->
+		<origin xyz="${base_x_com} ${base_y_com} ${base_z_com}" />
+		<!--The 3x3 rotational inertia matrix. Because the rotational inertia matrix is symmetric, only 6 above-diagonal elements of this matrix are specified here, using the attributes ixx, ixy, ixz, iyy, iyz, izz.-->
+		<inertia ixx="${base_ixx_com_cs}" ixy="${base_ixy_com_cs}" ixz="${base_ixz_com_cs}"
+			iyy="${base_iyy_com_cs}" iyz="${base_iyz_com_cs}" izz="${base_izz_com_cs}" />
+	 </inertial>
       <visual>
-        <eklavya_base_link_mesh />
+        <eklavya_base_link_mesh>
+           <origin xyz="0 0 ${base_x_size/2}" rpy="0 0 0" />
+           <box size = "${base_x_size} ${base_y_size} ${base_z_size}"/>
+          <!-- <origin xyz="0 0 0" rpy="0 0 0" />-->
+        </eklavya_base_link_mesh>
       </visual>
       <collision>
-        <eklavya_base_link_mesh />
+        <eklavya_base_link_mesh>
+           <origin xyz="0 0 ${base_x_size/2 }" rpy="0 0 0 " />
+           <box size = "${base_x_size} ${base_y_size} ${base_z_size}"/> <!--making it slightly bigger in x and z direction-->
+        </eklavya_base_link_mesh>
       </collision>
     </link>
     <gazebo_eklavya_base_link_surface />
-    <joint name="base_center_of_mass_joint" type="fixed">
-      <origin xyz="-0.1 0 -0.075" rpy="0 0 0" />
-      <parent link="base_link"/>
-      <child link="base_center_of_mass_link" />
-    </joint>
-    <link name="base_center_of_mass_link">
-      <inertial>
-        <mass value="30" />
-        <origin xyz="0 0 0" />
-        <inertia ixx="1.0" ixy="0.0" ixz="0.0"
-          iyy="1.0" iyz="0.0"
-          izz="1.0" />
-      </inertial>
-    </link>
 	 <!-- WHEEL macros -->
     <eklavya_wheel suffix="left" parent="base_link">
@@ -75,23 +100,17 @@
     </eklavya_wheel>
     <!-- Castor -->
-    <castor_support suffix="front" parent="base_link">
-      <origin rpy="0 0 0" xyz="0.36 0 -0.255"/>
-	</castor_support>
-	<caster_support_hinge suffix="front" parent="base_link">
-      <origin xyz="0.36 0 -0.275" rpy="0 0 0" />
-	</caster_support_hinge>
-    <caster_wheel suffix="front" parent="base_link">
-      <origin xyz="-0.0397 0 -0.0918" rpy="0 0 0" />
-	</caster_wheel>
+    <castor_support suffix="front" parent="base_link" />
+	<caster_support_hinge suffix="front" parent="base_link" />
+    <caster_wheel suffix="front" parent="base_link" />
      <!-- DECORATIONS -->
      <!-- Bars -->
-	<eklavya_support_bar suffix="left" parent="base_link" length="0.6">
-      <origin rpy="0 0 0" xyz="0.26 0.26 0.575"/>
+	 <eklavya_support_bar suffix="left" parent="base_link" length="0.6">
+      <origin rpy="0 0 0" xyz="${base_x_size/2-0.03/2} ${(base_y_size/2-0.03/2)} ${base_z_size+0.6/2}"/>
 	</eklavya_support_bar>
 	<eklavya_support_bar suffix="right" parent="base_link" length="0.6">
-      <origin rpy="0 0 0" xyz="0.26 -0.26 0.575"/>
+     <origin rpy="0 0 0" xyz="${base_x_size/2-0.03/2} ${-1*(base_y_size/2+-0.03/2)} ${base_z_size+0.6/2}"/>
 	</eklavya_support_bar>
 	<eklavya_support_bar suffix="top" parent="base_link" length="0.55">
-      <origin rpy="${M_PI/2} 0 0" xyz="0.26 0 0.89"/>
+		<origin rpy="${M_PI/2} 0 0"  xyz="${base_x_size/2-0.03/2} 0 ${base_z_size+0.6+0.03/2}"/>
 	</eklavya_support_bar>
 	<!-- Controllers -->
@@ -102,14 +121,14 @@
     <!-- Simulation sensors -->
 	<hokuyo_urg name="hokuyo_laser" parent="base_link" >
-       <origin rpy="0 0 0" xyz="0.36 0 -0.245"/>
+      <origin rpy="0 0 0" xyz="${base_x_size/2+0.05} 0  0.021"/>
     </hokuyo_urg>
    <!-- <sick_lms100_200 name="sick_laser" parent="base_link" >
       <origin rpy="0 0 0" xyz="0.39 0 -0.185"/>
     </sick_lms100_200> -->
-	<microstrain_imu name="eklavya_sim_imu" parent="base_link" imu_topic="imu/data" update_rate="30" stdevNoise="0.0017">
-		<origin rpy="0 0 0" xyz="0.26 0.20 0.575"/>
+	 <microstrain_imu name="eklavya_sim_imu" parent="base_link" imu_topic="imu/data" update_rate="30" stdevNoise="0.0017">
+		 <origin rpy="0 0 0" xyz="${base_x_size/2-0.03/2} ${base_y_size/4} ${base_z_size}"/>
 	</microstrain_imu>
     <!-- Kinect frames and mounting (includes simulation) -->
-   <eklavya_kinect/>
+    <eklavya_kinect/>
   </xacro:macro>
 </robot>

File: eklavya_description/urdf/eklavya_calibration.xacro (robot description, xacro)
@@ -3,5 +3,5 @@
   <property name="eklavya_calib_cam_x" value="${-0.0844382+0.36}" />
   <property name="eklavya_calib_cam_y" value="${0+ 0}" />
-  <property name="eklavya_calib_cam_z" value="${0.1047496+0.22}" />
+  <property name="eklavya_calib_cam_z" value="${0.05+0.55}" />
   <property name="eklavya_calib_cam_rr" value="0" />
   <property name="eklavya_calib_cam_rp" value="0" />

File: eklavya_description/urdf/eklavya_hardware.xacro (robot description, xacro)
@@ -30,7 +30,7 @@
     </link>
  </macro>
- <macro name="castor_support" params="suffix parent *origin">
+ <macro name="castor_support" params="suffix parent">
 	<joint type="fixed" name="${parent}_castor_support_${suffix}_joint">
-	  <insert_block name="origin" />
+	  <origin rpy="0 0 0" xyz="${base_x_size/2+0.1} 0 ${0.02/2}"/>
       <parent link="${parent}"/>
       <child link="${parent}_castor_support_${suffix}_link"/>
@@ -55,7 +55,7 @@
     </link>
  </macro>
- <macro name="caster_support_hinge" params="suffix parent *origin">
+ <macro name="caster_support_hinge" params="suffix parent">
 	<joint name="${parent}_caster_support_hinge_${suffix}_joint" type="continuous">
-      <insert_block name="origin" />
+      <origin rpy="0 0 0" xyz="${base_x_size/2+0.1} 0 ${0.02-0.02}"/>
       <parent link="${parent}" />
       <child link="${parent}_caster_support_hinge_${suffix}_link"/>
@@ -86,7 +86,7 @@
     </link>
 </macro>
-<macro name="caster_wheel" params="suffix parent *origin">
+<macro name="caster_wheel" params="suffix parent">
 	  <joint name="${parent}_caster_wheel_${suffix}_joint" type="continuous">
-      <insert_block name="origin" />
+      <origin rpy="0 0 0" xyz="${-0.036} 0 ${-0.0818}" />
       <parent link="${parent}_caster_support_hinge_${suffix}_link" />
       <child link="${parent}_caster_wheel_${suffix}_link" />

File: eklavya_description/urdf/eklavya_wheel.xacro (robot description, xacro)
@@ -7,6 +7,6 @@
 	<property name="wheel_y_com" value="0.00000000" /> <!-- com : center of mass -->
 	<property name="wheel_z_com" value="0.00019000" /> <!-- com : center of mass -->
-	<property name="wheel_x_size" value="0.35550000" />
-	<property name="wheel_y_size" value="0.35550000" />
+	<property name="wheel_x_size" value="0.30550000" />
+	<property name="wheel_y_size" value="0.30550000" />
 	<property name="wheel_z_size" value="0.11430000" />
 	<property name="wheel_mass" value="2.63657000" /> <!-- in kg-->
@@ -17,8 +17,7 @@
 	<property name="wheel_iyz_com_cs" value="0.00000000" /> <!-- at center of mass aligned with coordinate system, kg*m^2-->
 	<property name="wheel_izz_com_cs" value="0.04410576" /> <!-- at center of mass aligned with coordinate system, kg*m^2-->
-	<property name="base_x_origin_to_wheel_origin" value="0.2" />
-	<property name="base_y_origin_to_wheel_origin" value="0.355" />
-	<property name="base_z_origin_to_wheel_origin" value="0.303" />
-	<property name="base_z_origin_offset" value="0.00317500" /> <!-- origin is offset in + z direction by 3.175mm, so need to bring it back down for visual and collision-->
+	<property name="base_x_origin_to_wheel_origin" value="0.20" />
+	<property name="base_y_origin_to_wheel_origin" value="0.350" />
+	<property name="base_z_origin_to_wheel_origin" value="-0.0262508" />
   <macro name="eklavya_wheel" params="suffix parent *origin">
     <joint name="${parent}_${suffix}_wheel_joint" type="continuous">

File: eklavya_description/urdf/gazebo.urdf.xacro (robot description, xacro)
@@ -6,8 +6,8 @@
   <macro name="gazebo_eklavya_base_link_surface">
     <gazebo reference="base_link">
-      <mu1 value="100.0" />
+      <!--<mu1 value="100.0" />
       <mu2 value="100.0" />
       <kp  value="1000000.0" />
-      <kd  value="1.0" />
+      <kd  value="1.0" />-->
       <!--material name="Eklavya/GunMetalBrushedAluminum   Gazebo/Blue" />-->
     <material>Eklavya/GunMetalBrushedAluminum</material>
@@ -22,9 +22,9 @@
     </gazebo>
   </macro>
-  <macro name="eklavya_base_link_mesh">
-    <origin xyz="0 0 0" rpy="0 0 0" />
+  <macro name="eklavya_base_link_mesh"  params="*origin *box" >
+	  <insert_block name="origin" />
     <geometry>
      <!-- <mesh filename="package://eklavya_description/meshes/rmp50-base-link.dae" scale="0.0254 0.0254 0.0254"/> -->
-    <box size=".55 .55 .55"/>
+    <insert_block name="box" />
     </geometry>
      <material name="GunMetalBrushedAluminum"/>
@@ -33,5 +33,5 @@
     <origin xyz="0 0 0" rpy="0 0 0" />
     <geometry>
-      <mesh filename="package://eklavya_description/meshes/rmp50-castor-wheel.dae" scale="0.0254 0.0254 0.0254"/>
+      <mesh filename="package://eklavya_description/meshes/rmp50-castor-wheel.dae" scale="0.0220 0.0220 0.0220"/>
     </geometry>
   </macro>
@@ -45,5 +45,5 @@
     <origin xyz="0 0 0" rpy="0 0 0" />
     <geometry>
-      <mesh filename="package://eklavya_description/meshes/rmp50-castor-link.dae" scale="0.0254 0.0254 0.0254"/>
+      <mesh filename="package://eklavya_description/meshes/rmp50-castor-link.dae" scale="0.0220 0.0220 0.0220"/>
     </geometry>
   </macro>
@@ -85,6 +85,6 @@
     <leftJoint>base_link_right_wheel_joint</leftJoint>
     <rightJoint>base_link_left_wheel_joint</rightJoint>
-    <wheelSeparation>${caster_wheel_offset_y*2}</wheelSeparation>
-    <wheelDiameter>${wheel_radius}</wheelDiameter>
+    <wheelSeparation>${base_y_size}</wheelSeparation>
+    <wheelDiameter>${wheel_x_size/2}</wheelDiameter>
     <torque>30</torque>
     <interface:position name="position_iface_0"/>
@@ -113,7 +113,7 @@
                 <leftJoint>base_link_right_wheel_joint</leftJoint>
                 <rightJoint>base_link_left_wheel_joint</rightJoint>
-                <wheelSeparation>${caster_wheel_offset_y*2}</wheelSeparation>
-                <wheelDiameter>${wheel_radius*2}</wheelDiameter>
-                <torque>30</torque>
+                <wheelSeparation>${base_y_size}</wheelSeparation>
+                <wheelDiameter>${wheel_x_size}</wheelDiameter>
+                <torque>35</torque>
                 <interface:position name="position_iface_0"/>
                 <robotNamespace>/</robotNamespace>

Commit message: using sick Laser

File: eklavya_description/urdf/eklavya_body.urdf.xacro (robot description, xacro)
@@ -120,10 +120,10 @@
      <eklavya_controllers_common />
     <!-- Simulation sensors -->
-	<hokuyo_urg name="hokuyo_laser" parent="base_link" >
+	<!-- <hokuyo_urg name="hokuyo_laser" parent="base_link" >
       <origin rpy="0 0 0" xyz="${base_x_size/2+0.05} 0  0.021"/>
-    </hokuyo_urg>
-   <!-- <sick_lms100_200 name="sick_laser" parent="base_link" >
-      <origin rpy="0 0 0" xyz="0.39 0 -0.185"/>
-    </sick_lms100_200> -->
+    </hokuyo_urg> -->
+    <sick_lms100_200 name="sick_laser" parent="base_link" >
+      <origin rpy="0 0 0" xyz="${base_x_size/2+0.12} 0  0.080"/>
+    </sick_lms100_200>
 	 <microstrain_imu name="eklavya_sim_imu" parent="base_link" imu_topic="imu/data" update_rate="30" stdevNoise="0.0017">
 		 <origin rpy="0 0 0" xyz="${base_x_size/2-0.03/2} ${base_y_size/4} ${base_z_size}"/>

File: eklavya_description/urdf/sick_lms100_200.urdf.xacro (robot description, xacro)
@@ -43,5 +43,5 @@
         </link>
         <joint name="${name}_joint" type="fixed">
-            <origin xyz="0 0 0.06" rpy="0 0 0" />
+            <origin xyz="0.08 0 0.01" rpy="0 0 0" />
             <parent link="${name}_mount_link" />
             <child link="${name}_link" />
@@ -71,18 +71,18 @@
         </link>
         <gazebo reference="${name}_mount_link">
-            <material value="Erratic/Black" />
+            <material value="Erratic/Blue" />
         </gazebo>
         <gazebo reference="${name}_link">
-            <material value="Erratic/Black" />
+            <material value="Erratic/Blue" />
         </gazebo>
         <gazebo reference="${name}_link">
             <sensor:ray name="laser">
-                <rayCount>1080</rayCount>
-                <rangeCount>1080</rangeCount>
+                <rayCount>1000</rayCount>
+                <rangeCount>1000</rangeCount>
                 <laserCount>1</laserCount>
                 <origin>0.0 0.0 0.0</origin>
                 <displayRays>false</displayRays>
-                <minAngle>-120</minAngle>
-                <maxAngle> 120</maxAngle>
+                <minAngle>-100</minAngle>
+                <maxAngle> 100</maxAngle>
                 <minRange>0.05</minRange>
                 <maxRange>6.0</maxRange>

Commit message: good mapping

File: eklavya_description/urdf/eklavya_body.urdf.xacro (robot description, xacro)
@@ -61,5 +61,4 @@
     </gazebo>
     <joint name="base_footprint_joint" type="fixed">
-      <!-- <origin xyz="0.0 0 0.97" rpy="0 0 0" />-->
       <origin xyz="0 0 ${wheel_x_size/2 - base_z_origin_to_wheel_origin}" rpy="0 0 0" />
       <parent link="base_footprint"/>
@@ -79,12 +78,13 @@
       <visual>
         <eklavya_base_link_mesh>
-           <origin xyz="0 0 ${base_x_size/2}" rpy="0 0 0" />
+          <origin xyz="0 0 ${base_x_size/2}" rpy="0 0 0" />
+           <!--  <origin xyz="-0.33 0 0.69" rpy="0 0 0" /> -->
            <box size = "${base_x_size} ${base_y_size} ${base_z_size}"/>
-          <!-- <origin xyz="0 0 0" rpy="0 0 0" />-->
         </eklavya_base_link_mesh>
       </visual>
       <collision>
         <eklavya_base_link_mesh>
-           <origin xyz="0 0 ${base_x_size/2 }" rpy="0 0 0 " />
+	   <origin xyz="0 0 0" rpy="0 0 0" />
+            <!-- <origin xyz="0 0 ${base_x_size/2 }" rpy="0 0 0 " /> -->
            <box size = "${base_x_size} ${base_y_size} ${base_z_size}"/> <!--making it slightly bigger in x and z direction-->
         </eklavya_base_link_mesh>
@@ -94,5 +94,5 @@
 	 <!-- WHEEL macros -->
     <eklavya_wheel suffix="left" parent="base_link">
-      <origin xyz="${ -1*base_x_origin_to_wheel_origin} ${base_y_origin_to_wheel_origin} ${ -1*base_z_origin_to_wheel_origin}" rpy="0 0 0" />
+      <origin xyz="${ -1*base_x_origin_to_wheel_origin} ${base_y_origin_to_wheel_origin} ${ -1*base_z_origin_to_wheel_origin}" rpy="${M_PI} 0 0" />
     </eklavya_wheel>
     <eklavya_wheel suffix="right" parent="base_link">

File: eklavya_description/urdf/gazebo.urdf.xacro (robot description, xacro)
@@ -24,7 +24,8 @@
   <macro name="eklavya_base_link_mesh"  params="*origin *box" >
 	  <insert_block name="origin" />
-    <geometry>
-     <!-- <mesh filename="package://eklavya_description/meshes/rmp50-base-link.dae" scale="0.0254 0.0254 0.0254"/> -->
-    <insert_block name="box" />
+     <geometry>
+    <!--<mesh filename="package://eklavya_description/meshes/rmp50-base-link.dae" scale="0.0254 0.0254 0.0254"/> -->
+    <!-- <mesh filename="package://eklavya_description/meshes/body.dae" />-->
+  	<insert_block name="box" />
     </geometry>
      <material name="GunMetalBrushedAluminum"/>
@@ -53,4 +54,5 @@
      <!-- <mesh filename="package://eklavya_description/meshes/rmp50-${suffix}-wheel.dae" scale="0.0150 0.0150 0.0150"/>-->
       <mesh filename="package://eklavya_description/meshes/wheel.stl" />
+    <!--  <mesh filename="package://eklavya_description/meshes/wheel.dae" />-->
     </geometry>
     <material name="DarkGray" />
