Commit message: Eklavya 2.0 model integrated as main and the only model

File: eklavya_description/urdf/eklavya_body.urdf.xacro (robot description, xacro)
@@ -6,7 +6,7 @@
     <!-- Main Body-base-->
     <!-- Location of com : center of mass -->
-    <property name="base_x_com" value="-0.04748000" />
-    <property name="base_y_com" value="-0.00000000" />
-    <property name="base_z_com" value="0.09947000" />
+    <property name="base_x_com" value="0" />
+    <property name="base_y_com" value="0" />
+    <property name="base_z_com" value="0" />
     <!-- Size of the base-->
     <property name="base_x_size" value="0.55000000" />
@@ -37,7 +37,7 @@
     <link name="base_footprint">
       <visual>
-        <origin xyz="0 0 0.0" rpy="0 0 0" />
+        <origin xyz="0 0 0" rpy="0 0 0" />
         <geometry>
-          <box size="0.001 0.001 0.001" />
+          <box size="0.1 0.1 0.01" />
         </geometry>
       </visual>
@@ -78,13 +78,12 @@
       <visual>
         <eklavya_base_link_mesh>
-          <origin xyz="0 0 ${base_x_size/2}" rpy="0 0 0" />
-           <!--  <origin xyz="-0.33 0 0.69" rpy="0 0 0" /> -->
-           <box size = "${base_x_size} ${base_y_size} ${base_z_size}"/>
+           <!--<origin xyz="0 0 ${base_x_size/2}" rpy="0 0 0" />-->
+            <origin xyz="0 0 0" rpy="0 0 0" />
+           <box size = "0.001 0.001 0.001"/>
         </eklavya_base_link_mesh>
       </visual>
       <collision>
         <eklavya_base_link_mesh>
-	   <origin xyz="0 0 0" rpy="0 0 0" />
-            <!-- <origin xyz="0 0 ${base_x_size/2 }" rpy="0 0 0 " /> -->
+            <origin xyz="0 0 0" rpy="0 0 0" />
            <box size = "${base_x_size} ${base_y_size} ${base_z_size}"/> <!--making it slightly bigger in x and z direction-->
         </eklavya_base_link_mesh>
@@ -93,5 +92,5 @@
     <gazebo_eklavya_base_link_surface />
 	 <!-- WHEEL macros -->
-    <eklavya_wheel suffix="left" parent="base_link">
+   <eklavya_wheel suffix="left" parent="base_link">
       <origin xyz="${ -1*base_x_origin_to_wheel_origin} ${base_y_origin_to_wheel_origin} ${ -1*base_z_origin_to_wheel_origin}" rpy="${M_PI} 0 0" />
     </eklavya_wheel>
@@ -103,32 +102,23 @@
 	<caster_support_hinge suffix="front" parent="base_link" />
     <caster_wheel suffix="front" parent="base_link" />
-     <!-- DECORATIONS -->
-     <!-- Bars -->
-	 <eklavya_support_bar suffix="left" parent="base_link" length="0.6">
-      <origin rpy="0 0 0" xyz="${base_x_size/2-0.03/2} ${(base_y_size/2-0.03/2)} ${base_z_size+0.6/2}"/>
-	</eklavya_support_bar>
-	<eklavya_support_bar suffix="right" parent="base_link" length="0.6">
-     <origin rpy="0 0 0" xyz="${base_x_size/2-0.03/2} ${-1*(base_y_size/2+-0.03/2)} ${base_z_size+0.6/2}"/>
-	</eklavya_support_bar>
-	<eklavya_support_bar suffix="top" parent="base_link" length="0.55">
-		<origin rpy="${M_PI/2} 0 0"  xyz="${base_x_size/2-0.03/2} 0 ${base_z_size+0.6+0.03/2}"/>
-	</eklavya_support_bar>
 	<!-- Controllers -->
-   <!-- <gazebo_eklavya_simple_drive_plugin />    -->
-    <gazebo_eklavya_drive_plugin_diffdrive /><!-- cmd_vel movement -->
-    <gazebo_eklavya_p3d_plugin /> <!-- Ground Truth-->
-     <eklavya_controllers_common />
+	<!-- <gazebo_eklavya_simple_drive_plugin />    -->
+	<!--  <gazebo_eklavya_drive_plugin_diffdrive /> --><!-- cmd_vel movement -->
+	<gazebo_eklavya_p3d_plugin /> <!-- Ground Truth-->
+	<eklavya_controllers_common />
     <!-- Simulation sensors -->
-	<hokuyo_urg name="hokuyo_laser" parent="base_link" >
-      <origin rpy="0 0 0" xyz="${base_x_size/2+0.05} 0  0.021"/>
+    <hokuyo_urg name="hokuyo_laser" parent="base_link" >
+      <origin rpy="0 0 ${M_PI}" xyz="${-base_x_size/2} 0  0.33"/>
     </hokuyo_urg>
-    <!-- <sick_lms100_200 name="sick_laser" parent="base_link" >
-      <origin rpy="0 0 0" xyz="${base_x_size/2+0.12} 0  0.080"/>
-    </sick_lms100_200>   -->
+	<!--<sick_lms100_200 name="sick_laser" parent="base_link" >
+		<origin rpy="0 0 0" xyz="${base_x_size/2+0.12} 0  0.080"/>
+	</sick_lms100_200>   -->
 	 <microstrain_imu name="eklavya_sim_imu" parent="base_link" imu_topic="imu/data" update_rate="30" stdevNoise="0.0017">
-		 <origin rpy="0 0 0" xyz="${base_x_size/2-0.03/2} ${base_y_size/4} ${base_z_size}"/>
+		 <origin rpy="0 0 0" xyz="0 0 0"/>
 	</microstrain_imu>
     <!-- Kinect frames and mounting (includes simulation) -->
-    <eklavya_kinect/>
+    <eklavya_kinect>
+	  <!--origin rpy="0 0 ${M_PI/2}" xyz="${-base_x_size/2-0.05} 0  0.6"/-->
+	</eklavya_kinect>
   </xacro:macro>
 </robot>

File: eklavya_description/urdf/gazebo.urdf.xacro (robot description, xacro)
@@ -25,7 +25,7 @@
 	  <insert_block name="origin" />
      <geometry>
-    <!--<mesh filename="package://eklavya_description/meshes/rmp50-base-link.dae" scale="0.0254 0.0254 0.0254"/> -->
-    <!-- <mesh filename="package://eklavya_description/meshes/body.dae" />-->
-  	<insert_block name="box" />
+    <!-- mesh filename="package://eklavya_description/meshes/rmp50-base-link.dae" scale="0.0254 0.0254 0.0254"/ -->
+    <mesh filename="package://eklavya_description/meshes/body.dae" />
+  	<!-- <insert_block name="box" /> -->
     </geometry>
      <material name="GunMetalBrushedAluminum"/>
@@ -34,5 +34,6 @@
     <origin xyz="0 0 0" rpy="0 0 0" />
     <geometry>
-      <mesh filename="package://eklavya_description/meshes/rmp50-castor-wheel.dae" scale="0.0220 0.0220 0.0220"/>
+      <!--mesh filename="package://eklavya_description/meshes/rmp50-castor-wheel.dae"/-->
+      <mesh filename="package://eklavya_description/meshes/castorWheel.dae" scale="2 2 2"/>
     </geometry>
   </macro>
@@ -46,13 +47,14 @@
     <origin xyz="0 0 0" rpy="0 0 0" />
     <geometry>
-      <mesh filename="package://eklavya_description/meshes/rmp50-castor-link.dae" scale="0.0220 0.0220 0.0220"/>
+      <!--mesh filename="package://eklavya_description/meshes/rmp50-castor-link.dae" scale="0.0220 0.0220 0.0220"/-->
+      <mesh filename="package://eklavya_description/meshes/wheelhub.dae"/> <!-- scale="0.0220 0.0220 0.0220"-->
     </geometry>
   </macro>
   <macro name="eklavya_wheel_mesh" params="suffix">
-    <origin xyz="0 0 0" rpy="0 0 0" />
+    <origin xyz="0 0 0" rpy="0 0 1.570796327" />
     <geometry>
      <!-- <mesh filename="package://eklavya_description/meshes/rmp50-${suffix}-wheel.dae" scale="0.0150 0.0150 0.0150"/>-->
-      <mesh filename="package://eklavya_description/meshes/wheel.stl" />
-    <!--  <mesh filename="package://eklavya_description/meshes/wheel.dae" />-->
+     <!-- <mesh filename="package://eklavya_description/meshes/wheel.stl" /> -->
+    <mesh filename="package://eklavya_description/meshes/wheel.dae" />
     </geometry>
     <material name="DarkGray" />

Commit message: With some vibrations on model, the model has been configured to run properly except castor

File: eklavya_description/urdf/eklavya_body.urdf.xacro (robot description, xacro)
@@ -79,5 +79,5 @@
         <eklavya_base_link_mesh>
            <!--<origin xyz="0 0 ${base_x_size/2}" rpy="0 0 0" />-->
-            <origin xyz="0 0 0" rpy="0 0 0" />
+            <origin xyz="0 0 0" rpy="0 0 3.1415926535897932384626" />
            <box size = "0.001 0.001 0.001"/>
         </eklavya_base_link_mesh>
@@ -93,8 +93,8 @@
 	 <!-- WHEEL macros -->
    <eklavya_wheel suffix="left" parent="base_link">
-      <origin xyz="${ -1*base_x_origin_to_wheel_origin} ${base_y_origin_to_wheel_origin} ${ -1*base_z_origin_to_wheel_origin}" rpy="${M_PI} 0 0" />
+      <origin xyz="${-1*base_x_origin_to_wheel_origin} ${-1*base_y_origin_to_wheel_origin} ${ -1*base_z_origin_to_wheel_origin}" rpy="${M_PI} 0 ${M_PI}" />
     </eklavya_wheel>
     <eklavya_wheel suffix="right" parent="base_link">
-      <origin xyz="${ -1*base_x_origin_to_wheel_origin} ${-1*base_y_origin_to_wheel_origin} ${ -1*base_z_origin_to_wheel_origin}" rpy="0 0 0" />
+      <origin xyz="${-1*base_x_origin_to_wheel_origin} ${base_y_origin_to_wheel_origin} ${ -1*base_z_origin_to_wheel_origin}" rpy="0 0 ${M_PI}" />
     </eklavya_wheel>
     <!-- Castor -->
@@ -103,6 +103,6 @@
     <caster_wheel suffix="front" parent="base_link" />
 	<!-- Controllers -->
-	<!-- <gazebo_eklavya_simple_drive_plugin />    -->
-	<!--  <gazebo_eklavya_drive_plugin_diffdrive /> --><!-- cmd_vel movement -->
+	<!--gazebo_eklavya_simple_drive_plugin /-->
+	<gazebo_eklavya_drive_plugin_diffdrive /><!-- cmd_vel movement -->
 	<gazebo_eklavya_p3d_plugin /> <!-- Ground Truth-->
 	<eklavya_controllers_common />

File: eklavya_description/urdf/eklavya_hardware.xacro (robot description, xacro)
@@ -32,5 +32,5 @@
  <macro name="castor_support" params="suffix parent">
 	<joint type="fixed" name="${parent}_castor_support_${suffix}_joint">
-	  <origin rpy="0 0 0" xyz="${base_x_size/2} 0 0.058"/>
+	  <origin rpy="0 0 0" xyz="${base_x_size/2-0.5} 0 0.058"/>
       <parent link="${parent}"/>
       <child link="${parent}_castor_support_${suffix}_link"/>
@@ -57,5 +57,5 @@
  <macro name="caster_support_hinge" params="suffix parent">
 	<joint name="${parent}_caster_support_hinge_${suffix}_joint" type="continuous">
-      <origin rpy="0 0 0" xyz="${base_x_size/2} 0 0.058"/>
+      <origin rpy="0 0 ${M_PI}" xyz="${base_x_size/2-0.5} 0 0.058"/>
       <parent link="${parent}" />
       <child link="${parent}_caster_support_hinge_${suffix}_link"/>
@@ -88,5 +88,5 @@
 <macro name="caster_wheel" params="suffix parent">
 	  <joint name="${parent}_caster_wheel_${suffix}_joint" type="continuous">
-      <origin rpy="0 0 0" xyz="0.066 0 -0.085" />
+      <origin rpy="0 0 0" xyz="${0.066} 0 -0.085" />
       <parent link="${parent}_caster_support_hinge_${suffix}_link" />
       <child link="${parent}_caster_wheel_${suffix}_link" />

File: eklavya_description/urdf/eklavya_wheel.xacro (robot description, xacro)
@@ -19,5 +19,5 @@
 	<property name="wheel_iyz_com_cs" value="0.00000000" /> <!-- at center of mass aligned with coordinate system, kg*m^2-->
 	<property name="wheel_izz_com_cs" value="0.04410576" /> <!-- at center of mass aligned with coordinate system, kg*m^2-->
-	<property name="base_x_origin_to_wheel_origin" value="0.15" />
+	<property name="base_x_origin_to_wheel_origin" value="-0.18" />
 	<property name="base_y_origin_to_wheel_origin" value="0.225" />
 	<property name="base_z_origin_to_wheel_origin" value="0" />

File: eklavya_description/urdf/gazebo.urdf.xacro (robot description, xacro)
@@ -102,11 +102,11 @@
      </gazebo>
   </macro>
-  <macro name="gazebo_eklavya_drive_plugin">
-	<gazebo>
-    <controller:eklavya_drive_plugin name="differential_drive_controller" plugin="libeklavya_drive_plugin.so">
-      <eklavya_drive_parameters />
-    </controller:eklavya_drive_plugin>
-     </gazebo>
-   </macro>
+	<macro name="gazebo_eklavya_drive_plugin">
+		<gazebo>
+			<controller:eklavya_drive_plugin name="differential_drive_controller" plugin="libeklavya_drive_plugin.so">
+				<eklavya_drive_parameters />
+			</controller:eklavya_drive_plugin>
+		</gazebo>
+	</macro>
 	<macro name="gazebo_eklavya_drive_plugin_diffdrive">
         <gazebo>

Commit message: Collision model of main body reversed

File: eklavya_description/urdf/eklavya_body.urdf.xacro (robot description, xacro)
@@ -85,5 +85,5 @@
       <collision>
         <eklavya_base_link_mesh>
-            <origin xyz="0 0 0" rpy="0 0 0" />
+            <origin xyz="0 0 0" rpy="0 0 3.1415926535897932384626" />
            <box size = "${base_x_size} ${base_y_size} ${base_z_size}"/> <!--making it slightly bigger in x and z direction-->
         </eklavya_base_link_mesh>

File: eklavya_description/urdf/eklavya_hardware.xacro (robot description, xacro)
@@ -61,5 +61,5 @@
       <child link="${parent}_caster_support_hinge_${suffix}_link"/>
       <axis xyz="0 0 1" />
-      <anchor xyz="0.01 0 0" />
+      <anchor xyz="0 0 0" />
       <limit effort="100" velocity="100" k_velocity="0" />
       <joint_properties damping="0.0" friction="0.0" />
