Commit message: fixing model

File: eklavya_description/urdf/common.xacro (robot description, xacro)
@@ -24,4 +24,13 @@
     </inertial>
   </macro>
+ <macro name="cylinder_inertial_with_origin_wheel" params="radius length mass origin">
+    <inertial>
+      <mass value="${mass}" />
+      <origin xyz="${origin}" />
+      <inertia ixx="${0.0833333 * mass * (3 * radius * radius + length * length)}" ixy="0.0" ixz="0.0"
+        iyy="${0.0833333 * mass * (3 * radius * radius + length * length)}" iyz="0.0"
+        izz="${0.5 * mass * radius * radius}" />
+    </inertial>
+  </macro>
   <macro name="box_inertial" params="x y z mass">
     <inertial>

File: eklavya_description/urdf/eklavya_body.urdf.xacro (robot description, xacro)
@@ -4,23 +4,6 @@
     <!--All units in m-kg-s-radians unit system -->
     <property name="M_PI" value="3.1415926535897931" />
-    <!-- Main Body-base-->
-    <!-- Location of com : center of mass -->
-    <property name="base_x_com" value="0" />
-    <property name="base_y_com" value="0" />
-    <property name="base_z_com" value="0" />
-    <!-- Size of the base-->
-    <property name="base_x_size" value="0.55000000" />
-    <property name="base_y_size" value="0.55000000" />
-    <property name="base_z_size" value="0.55000000" />
-    <!--Weight of the base-->
-    <property name="base_mass" value="33.45489000" /> <!-- in kg-->
-    <!--Inertial values for the base at center of mass, aligned with coordinate system. Units are kg*m^2-->
-    <property name="base_ixx_com_cs" value="0.60216370" />
-    <property name="base_ixy_com_cs" value="-0.02364198" />
-    <property name="base_ixz_com_cs" value="-0.11972132" />
-    <property name="base_iyy_com_cs" value="1.73859574" />
-    <property name="base_iyz_com_cs" value="-0.00154437" />
-    <property name="base_izz_com_cs" value="2.02955229" />
   <!-- Macro for eklavya body. Including Gazebo extensions, but does not include Kinect -->
+  <include filename="$(find eklavya_description)/urdf/params.xacro"/>
   <include filename="$(find eklavya_description)/urdf/gazebo.urdf.xacro"/>
   <include filename="$(find eklavya_description)/urdf/materials.urdf.xacro"/>
@@ -68,57 +51,49 @@
     <!--Actual body/chassis of the robot-->
     <link name="base_link">
-	 <inertial>
-		<mass value="${base_mass}" />
-		<!--This is the pose of the inertial reference frame, relative to the link reference frame. The origin of the inertial reference frame needs to be at the center of gravity. The axes of the inertial reference frame do not need to be aligned with the principal axes of the inertia.-->
-		<origin xyz="${base_x_com} ${base_y_com} ${base_z_com}" />
-		<!--The 3x3 rotational inertia matrix. Because the rotational inertia matrix is symmetric, only 6 above-diagonal elements of this matrix are specified here, using the attributes ixx, ixy, ixz, iyy, iyz, izz.-->
-		<inertia ixx="${base_ixx_com_cs}" ixy="${base_ixy_com_cs}" ixz="${base_ixz_com_cs}"
-			iyy="${base_iyy_com_cs}" iyz="${base_iyz_com_cs}" izz="${base_izz_com_cs}" />
-	 </inertial>
+	<box_inertial_with_origin x="${base_x_size}" y="${base_y_size}" z="${base_z_size}" mass="${base_mass}" origin="0 0 ${base_z_size/2}" />
       <visual>
         <eklavya_base_link_mesh>
-           <!--<origin xyz="0 0 ${base_x_size/2}" rpy="0 0 0" />-->
-            <origin xyz="0 0 0" rpy="0 0 3.1415926535897932384626" />
-           <box size = "0.001 0.001 0.001"/>
+           <origin xyz="0 0 ${base_z_size/2}" rpy="0 0 0" />
+           <box size="${base_x_size} ${base_y_size} ${base_z_size}" />
         </eklavya_base_link_mesh>
       </visual>
       <collision>
-        <eklavya_base_link_mesh>
-            <origin xyz="0 0 0" rpy="0 0 3.1415926535897932384626" />
-           <box size = "${base_x_size} ${base_y_size} ${base_z_size}"/> <!--making it slightly bigger in x and z direction-->
-        </eklavya_base_link_mesh>
+         <origin xyz="0 0 ${base_z_size/2}" rpy="0 0 0" />
+         <geometry>
+            <box size = "${base_x_size+0.02} ${base_y_size} ${base_z_size+0.02}"/>--> <!--making it slightly bigger in x and z direction-->
+         </geometry>
       </collision>
     </link>
     <gazebo_eklavya_base_link_surface />
 	 <!-- WHEEL macros -->
-   <eklavya_wheel suffix="left" parent="base_link">
-      <origin xyz="${-1*base_x_origin_to_wheel_origin} ${-1*base_y_origin_to_wheel_origin} ${ -1*base_z_origin_to_wheel_origin}" rpy="${M_PI} 0 ${M_PI}" />
+    <eklavya_wheel suffix="left" parent="base_link">
+      <origin xyz="${-1*base_x_origin_to_wheel_origin} ${-1*base_y_origin_to_wheel_origin} ${ -1*base_z_origin_to_wheel_origin}" rpy="${M_PI} 0 0" />
     </eklavya_wheel>
     <eklavya_wheel suffix="right" parent="base_link">
-      <origin xyz="${-1*base_x_origin_to_wheel_origin} ${base_y_origin_to_wheel_origin} ${ -1*base_z_origin_to_wheel_origin}" rpy="0 0 ${M_PI}" />
+      <origin xyz="${-1*base_x_origin_to_wheel_origin} ${base_y_origin_to_wheel_origin} ${ -1*base_z_origin_to_wheel_origin}" rpy="0 0 0" />
     </eklavya_wheel>
     <!-- Castor -->
-    <castor_support suffix="front" parent="base_link" />
 	<caster_support_hinge suffix="front" parent="base_link" />
     <caster_wheel suffix="front" parent="base_link" />
 	<!-- Controllers -->
-	<!--gazebo_eklavya_simple_drive_plugin /-->
-	<gazebo_eklavya_drive_plugin_diffdrive /><!-- cmd_vel movement -->
-	<gazebo_eklavya_p3d_plugin /> <!-- Ground Truth-->
-	<eklavya_controllers_common />
+	<!--<gazebo_eklavya_simple_drive_plugin />-->
+	<!--<gazebo_eklavya_drive_plugin /> -->
+	   <gazebo_eklavya_drive_plugin_diffdrive />  <!-- cmd_vel movement -->
+	 <!-- <gazebo_eklavya_p3d_plugin />--> <!-- Ground Truth-->
+	 <!-- <eklavya_controllers_common /> -->
     <!-- Simulation sensors -->
-    <hokuyo_urg name="hokuyo_laser" parent="base_link" >
+   <!-- <hokuyo_urg name="hokuyo_laser" parent="base_link" >
       <origin rpy="0 0 ${M_PI}" xyz="${-base_x_size/2} 0  0.33"/>
-    </hokuyo_urg>
+    </hokuyo_urg> -->
 	<!--<sick_lms100_200 name="sick_laser" parent="base_link" >
 		<origin rpy="0 0 0" xyz="${base_x_size/2+0.12} 0  0.080"/>
 	</sick_lms100_200>   -->
-	 <microstrain_imu name="eklavya_sim_imu" parent="base_link" imu_topic="imu/data" update_rate="30" stdevNoise="0.0017">
+	<!-- <microstrain_imu name="eklavya_sim_imu" parent="base_link" imu_topic="imu/data" update_rate="30" stdevNoise="0.0017">
 		 <origin rpy="0 0 0" xyz="0 0 0"/>
-	</microstrain_imu>
+	</microstrain_imu> -->
     <!-- Kinect frames and mounting (includes simulation) -->
-    <eklavya_kinect>
+   <!-- <eklavya_kinect> -->
 	  <!--origin rpy="0 0 ${M_PI/2}" xyz="${-base_x_size/2-0.05} 0  0.6"/-->
-	</eklavya_kinect>
+	<!--</eklavya_kinect> -->
   </xacro:macro>
 </robot>

File: eklavya_description/urdf/eklavya_hardware.xacro (robot description, xacro)
@@ -4,62 +4,12 @@
   xmlns:controller="http://playerstage.sourceforge.net/gazebo/xmlschema/#controller"
   xmlns:interface="http://playerstage.sourceforge.net/gazebo/xmlschema/#interface">
-  <macro name="eklavya_support_bar" params="suffix parent length *origin">
-	<joint type="fixed" name="${parent}_support_bar_${suffix}_joint">
-      <insert_block name="origin" />
-      <parent link="${parent}"/>
-      <child link="${parent}_support_bar_${suffix}"/>
-    </joint>
-    <link name="${parent}_support_bar_${suffix}">
-      <origin rpy="0 0 0" xyz="0 0 0"/>
-      <inertial>
-        <mass value="2.01" />
-        <inertia ixx="1" ixy="0.0" ixz="0.0" iyy="1" iyz="0.0" izz="1"/>
-      </inertial>
-      <collision >
-        <geometry>
-          <box size=".03 .03 ${length}"/>
-        </geometry>
-      </collision>
-      <visual >
-	    <geometry>
-          <box size=".03 .03 ${length}"/>
-        </geometry>
-        <!--<material name="White"/>-->
-        <material name="GunMetalBrushedAluminum"/>
-      </visual>
-    </link>
- </macro>
- <macro name="castor_support" params="suffix parent">
-	<joint type="fixed" name="${parent}_castor_support_${suffix}_joint">
-	  <origin rpy="0 0 0" xyz="${base_x_size/2-0.5} 0 0.058"/>
-      <parent link="${parent}"/>
-      <child link="${parent}_castor_support_${suffix}_link"/>
-    </joint>
-    <link name="${parent}_castor_support_${suffix}_link">
-      <origin rpy="0 0 0" xyz="0 0 0"/>
-      <inertial>
-        <mass value="0.01" />
-        <inertia ixx="1" ixy="0.0" ixz="0.0" iyy="1" iyz="0.0" izz="1"/>
-      </inertial>
-      <collision name='extrusion_collision'>
-        <geometry>
-          <box size="0 0 0"/>
-        </geometry>
-      </collision>
-      <visual name='extrusion_visual'>
-        <geometry>
-          <box size="0 0 0"/>
-        </geometry>
-        <material name="GunMetalBrushedAluminum"/>
-      </visual>
-    </link>
- </macro>
+    <include filename="$(find eklavya_description)/urdf/params.xacro"/>
  <macro name="caster_support_hinge" params="suffix parent">
 	<joint name="${parent}_caster_support_hinge_${suffix}_joint" type="continuous">
-      <origin rpy="0 0 ${M_PI}" xyz="${base_x_size/2-0.5} 0 0.058"/>
+      <origin rpy="0 0 0" xyz="${base_x_size/2-0.5} 0 ${caster_support_hinge_z_offset}"/>
       <parent link="${parent}" />
       <child link="${parent}_caster_support_hinge_${suffix}_link"/>
       <axis xyz="0 0 1" />
-      <anchor xyz="0 0 0" />
+      <anchor xyz="0 0 ${M_PI}" />
       <limit effort="100" velocity="100" k_velocity="0" />
       <joint_properties damping="0.0" friction="0.0" />
@@ -82,11 +32,11 @@
       </visual>
       <collision>
-        <eklavya_castor_support_link_mesh />
+        <eklavya_collision_none />
       </collision>
     </link>
 </macro>
 <macro name="caster_wheel" params="suffix parent">
-	  <joint name="${parent}_caster_wheel_${suffix}_joint" type="continuous">
-      <origin rpy="0 0 0" xyz="${0.066} 0 -0.085" />
+	 <joint name="${parent}_caster_wheel_${suffix}_joint" type="continuous">
+      <origin rpy="0 0 0" xyz="${base_x_origin_to_caster_wheel_origin} ${base_y_origin_to_caster_wheel_origin} ${base_z_origin_to_caster_wheel_origin } " />
       <parent link="${parent}_caster_support_hinge_${suffix}_link" />
       <child link="${parent}_caster_wheel_${suffix}_link" />
@@ -102,16 +52,14 @@
     </transmission>
     <link name="${parent}_caster_wheel_${suffix}_link">
-      <inertial>
-        <mass value="1" />
-        <origin xyz="0 0 0" rpy="0 0 0" />
-        <inertia  ixx="0.003" ixy="0.0" ixz="0.0"
-          iyy="0.00581" iyz="0.0"
-          izz="0.003" />
-      </inertial>
+	<cylinder_inertial_with_origin_wheel radius="${castor_x_size/2}" length="${castor_z_size}" mass="1" origin="0 0 0" />
       <visual>
         <eklavya_castor_wheel_link_mesh />
       </visual>
       <collision>
-        <eklavya_castor_wheel_link_mesh />
+		<origin xyz="0 0 0" rpy="1.570796327 0 0" />
+		<!--<origin xyz="0 0 0" rpy="0 0 0" /> -->
+		<geometry>
+			<cylinder radius="${castor_x_size/2}" length="${castor_z_size}"/>
+		</geometry>
       </collision>
     </link>

File: eklavya_description/urdf/eklavya_wheel.xacro (robot description, xacro)
@@ -4,22 +4,6 @@
   xmlns:controller="http://playerstage.sourceforge.net/gazebo/xmlschema/#controller"
   xmlns:interface="http://playerstage.sourceforge.net/gazebo/xmlschema/#interface">
-    <property name="wheel_x_com" value="0.00000000" /> <!-- com : center of mass -->
-	<property name="wheel_y_com" value="0.00000000" /> <!-- com : center of mass -->
-	<property name="wheel_z_com" value="0.00019000" /> <!-- com : center of mass -->
-	<!--property name="wheel_x_size" value="0.30550000" /-->
-	<!--property name="wheel_y_size" value="0.30550000" /-->
-	<property name="wheel_x_size" value="0.22" />
-	<property name="wheel_y_size" value="0.22" />
-	<property name="wheel_z_size" value="0.11430000" />
+    <include filename="$(find eklavya_description)/urdf/params.xacro"/>
 	<property name="wheel_mass" value="2.63657000" /> <!-- in kg-->
-	<property name="wheel_ixx_com_cs" value="0.02466885" /> <!-- at center of mass aligned with coordinate system, kg*m^2-->
-	<property name="wheel_ixy_com_cs" value="0.00000000" /> <!-- at center of mass aligned with coordinate system, kg*m^2-->
-	<property name="wheel_ixz_com_cs" value="0.00000000" /> <!-- at center of mass aligned with coordinate system, kg*m^2-->
-	<property name="wheel_iyy_com_cs" value="0.02466885" /> <!-- at center of mass aligned with coordinate system, kg*m^2-->
-	<property name="wheel_iyz_com_cs" value="0.00000000" /> <!-- at center of mass aligned with coordinate system, kg*m^2-->
-	<property name="wheel_izz_com_cs" value="0.04410576" /> <!-- at center of mass aligned with coordinate system, kg*m^2-->
-	<property name="base_x_origin_to_wheel_origin" value="-0.18" />
-	<property name="base_y_origin_to_wheel_origin" value="0.225" />
-	<property name="base_z_origin_to_wheel_origin" value="0" />
   <macro name="eklavya_wheel" params="suffix parent *origin">
     <joint name="${parent}_${suffix}_wheel_joint" type="continuous">
@@ -33,16 +17,14 @@
     </joint>
     <link name="${parent}_${suffix}_wheel_link">
-      <inertial>
-			<mass value="${wheel_mass}" />
-			<origin xyz="${wheel_x_com} ${wheel_y_com} ${wheel_z_com}" />
-			<inertia  ixx="${wheel_ixx_com_cs}" ixy="${wheel_ixy_com_cs}" ixz="${wheel_ixz_com_cs}"
-				iyy="${wheel_iyy_com_cs}" iyz="${wheel_iyz_com_cs}" izz="${wheel_izz_com_cs}" />
-		</inertial>
-      <visual>
+      <cylinder_inertial_with_origin_wheel radius="${wheel_x_size/2}" length="${wheel_z_size}" mass="${wheel_mass}" origin="0 0 0" />
+	  <visual>
         <eklavya_wheel_mesh suffix="${suffix}" />
 		<material name="Red" />
       </visual>
       <collision>
-        <eklavya_wheel_mesh suffix="${suffix}" />
+		  <origin xyz="0 0 0" rpy="1.570796327 0 0" />
+		  <geometry>
+			 <cylinder radius="${wheel_x_size/2}" length="0.09"/>
+	      </geometry>
       </collision>
     </link>

File: eklavya_description/urdf/gazebo.urdf.xacro (robot description, xacro)
@@ -4,4 +4,5 @@
   xmlns:controller="http://playerstage.sourceforge.net/gazebo/xmlschema/#controller"
   xmlns:interface="http://playerstage.sourceforge.net/gazebo/xmlschema/#interface">
+  <include filename="$(find eklavya_description)/urdf/params.xacro"/>
   <macro name="gazebo_eklavya_base_link_surface">
     <gazebo reference="base_link">
@@ -11,5 +12,5 @@
       <kd  value="1.0" />-->
       <!--material name="Eklavya/GunMetalBrushedAluminum   Gazebo/Blue" />-->
-    <material>Eklavya/GunMetalBrushedAluminum</material>
+    <!--<material>Eklavya/GunMetalBrushedAluminum</material>-->
     </gazebo>
   </macro>
@@ -25,16 +26,33 @@
 	  <insert_block name="origin" />
      <geometry>
-    <!-- mesh filename="package://eklavya_description/meshes/rmp50-base-link.dae" scale="0.0254 0.0254 0.0254"/ -->
-    <mesh filename="package://eklavya_description/meshes/body.dae" />
-  	<!-- <insert_block name="box" /> -->
+     <mesh filename="package://eklavya_description/meshes/body.dae" />
+      <!--   <box size="${base_x_size} ${base_y_size} ${base_z_size}" />  -->
+  	 <!-- <insert_block name="box" /> -->
     </geometry>
      <material name="GunMetalBrushedAluminum"/>
   </macro>
+  <macro name="eklavya_castor_support_link_mesh">
+    <origin xyz="0 0 0" rpy="0 0 ${M_PI}" />
+    <geometry>
+      <mesh filename="package://eklavya_description/meshes/wheelhub.dae"/>
+     <!--  <box size="0.14715 0.12074 0.12065" /> -->
+    </geometry>
+     <material name="Blue"/>
+  </macro>
   <macro name="eklavya_castor_wheel_link_mesh">
-    <origin xyz="0 0 0" rpy="0 0 0" />
+	  <origin xyz="0 0 0" rpy="1.570796327 0 0" />
+    <!--<origin xyz="0 0 0" rpy="0 0 0" /> -->
     <geometry>
-      <!--mesh filename="package://eklavya_description/meshes/rmp50-castor-wheel.dae"/-->
-      <mesh filename="package://eklavya_description/meshes/castorWheel.dae" scale="2 2 2"/>
+      <mesh filename="package://eklavya_description/meshes/castorWheel.dae" />
+      <!-- <cylinder radius="${castor_x_size/2}" length="${castor_z_size}"/>  -->
     </geometry>
+  </macro>
+ <macro name="eklavya_wheel_mesh" params="suffix">
+    <origin xyz="0 0 0" rpy="1.570796327 0 0" />
+    <geometry>
+      <mesh filename="package://eklavya_description/meshes/wheel.dae" />
+    <!-- <cylinder radius="${wheel_x_size/2}" length="${wheel_z_size}" />-->
+    </geometry>
+    <material name="DarkGray" />
   </macro>
   <macro name="eklavya_collision_none">
@@ -43,20 +61,4 @@
       <box size="0.01 0.01 0.01" />
     </geometry>
-  </macro>
-  <macro name="eklavya_castor_support_link_mesh">
-    <origin xyz="0 0 0" rpy="0 0 0" />
-    <geometry>
-      <!--mesh filename="package://eklavya_description/meshes/rmp50-castor-link.dae" scale="0.0220 0.0220 0.0220"/-->
-      <mesh filename="package://eklavya_description/meshes/wheelhub.dae"/> <!-- scale="0.0220 0.0220 0.0220"-->
-    </geometry>
-  </macro>
-  <macro name="eklavya_wheel_mesh" params="suffix">
-    <origin xyz="0 0 0" rpy="0 0 1.570796327" />
-    <geometry>
-     <!-- <mesh filename="package://eklavya_description/meshes/rmp50-${suffix}-wheel.dae" scale="0.0150 0.0150 0.0150"/>-->
-     <!-- <mesh filename="package://eklavya_description/meshes/wheel.stl" /> -->
-    <mesh filename="package://eklavya_description/meshes/wheel.dae" />
-    </geometry>
-    <material name="DarkGray" />
   </macro>
   <macro name="eklavya_wheel_surface" params="suffix parent">
@@ -87,6 +89,6 @@
     <update>100</update>
     <updateRate>100.0</updateRate>
-    <leftJoint>base_link_right_wheel_joint</leftJoint>
-    <rightJoint>base_link_left_wheel_joint</rightJoint>
+    <leftJoint>base_link_left_wheel_joint</leftJoint>
+    <rightJoint>base_link_right_wheel_joint</rightJoint>
     <wheelSeparation>${base_y_size}</wheelSeparation>
     <wheelDiameter>${wheel_x_size/2}</wheelDiameter>
@@ -115,9 +117,9 @@
                 <update>100</update>
                 <updateRate>100.0</updateRate>
-                <leftJoint>base_link_right_wheel_joint</leftJoint>
-                <rightJoint>base_link_left_wheel_joint</rightJoint>
+                <leftJoint>base_link_left_wheel_joint</leftJoint>
+                <rightJoint>base_link_right_wheel_joint</rightJoint>
                 <wheelSeparation>${base_y_size}</wheelSeparation>
                 <wheelDiameter>${wheel_x_size}</wheelDiameter>
-                <torque>35</torque>
+                <torque>30</torque>
                 <interface:position name="position_iface_0"/>
                 <robotNamespace>/</robotNamespace>

Commit message: model stable, to do controller

File: eklavya_description/urdf/common.xacro (robot description, xacro)
@@ -29,6 +29,6 @@
       <origin xyz="${origin}" />
       <inertia ixx="${0.0833333 * mass * (3 * radius * radius + length * length)}" ixy="0.0" ixz="0.0"
-        iyy="${0.0833333 * mass * (3 * radius * radius + length * length)}" iyz="0.0"
-        izz="${0.5 * mass * radius * radius}" />
+        iyy="${0.5 * mass * radius * radius}" iyz="0.0"
+        izz="${0.0833333 * mass * (3 * radius * radius + length * length)}" />
     </inertial>
   </macro>

File: eklavya_description/urdf/eklavya_hardware.xacro (robot description, xacro)
@@ -7,9 +7,9 @@
  <macro name="caster_support_hinge" params="suffix parent">
 	<joint name="${parent}_caster_support_hinge_${suffix}_joint" type="continuous">
-      <origin rpy="0 0 0" xyz="${base_x_size/2-0.5} 0 ${caster_support_hinge_z_offset}"/>
+      <origin  rpy="0 0 ${M_PI}" xyz="${-base_x_size/2 +wheelhub_x_size/2} 0 ${castor_x_size/2 -wheel_x_size/2 -base_z_origin_to_caster_wheel_origin}"/>
       <parent link="${parent}" />
       <child link="${parent}_caster_support_hinge_${suffix}_link"/>
       <axis xyz="0 0 1" />
-      <anchor xyz="0 0 ${M_PI}" />
+      <anchor xyz="0.01 0 0" />
       <limit effort="100" velocity="100" k_velocity="0" />
       <joint_properties damping="0.0" friction="0.0" />
@@ -23,5 +23,5 @@
       <inertial>
         <mass value="1"/>
-        <origin xyz="0 0 0" />
+        <origin xyz="0 0 0"/>
         <inertia ixx="0.00375" ixy="0.0" ixz="0.0"
           iyy="0.00375" iyz="0.0"
@@ -38,5 +38,5 @@
 <macro name="caster_wheel" params="suffix parent">
 	 <joint name="${parent}_caster_wheel_${suffix}_joint" type="continuous">
-      <origin rpy="0 0 0" xyz="${base_x_origin_to_caster_wheel_origin} ${base_y_origin_to_caster_wheel_origin} ${base_z_origin_to_caster_wheel_origin } " />
+      <origin rpy="0 0 0" xyz="${base_x_origin_to_caster_wheel_origin} ${base_y_origin_to_caster_wheel_origin} ${base_z_origin_to_caster_wheel_origin} " />
       <parent link="${parent}_caster_support_hinge_${suffix}_link" />
       <child link="${parent}_caster_wheel_${suffix}_link" />

File: eklavya_description/urdf/gazebo.urdf.xacro (robot description, xacro)
@@ -121,5 +121,5 @@
                 <wheelSeparation>${base_y_size}</wheelSeparation>
                 <wheelDiameter>${wheel_x_size}</wheelDiameter>
-                <torque>30</torque>
+                <torque>20</torque>
                 <interface:position name="position_iface_0"/>
                 <robotNamespace>/</robotNamespace>

File: eklavya_description/urdf/params.xacro (robot description, xacro)
@@ -31,4 +31,4 @@
 	<property name="wheelhub_y_size" value="0.12000000" />
 	<property name="wheelhub_z_size" value="0.12000000" />
-	<property name="caster_support_hinge_z_offset" value="0.05325" /> <!-- 0.06275 0.05325 .058-->
+	<property name="caster_support_hinge_z_offset" value="0.0325" /> <!-- 0.06275 0.05325 .058-->
 </robot>
